File: AF_amp.kicad_sch (KiCad schematic)
At the start: 24 parts, among them J3 SPK, Q1 2N3904, U5 LM386

Commit message: Continue Migration from D612
Changed lines of the file:
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@@
-    )
-  )
-  (global_label "RX12V" (shape output) (at 187.96 73.025 90) (fields_autoplaced)
-    (effects (font (size 1.27 1.27)) (justify left))
-    (property "Intersheet References" "${INTERSHEET_REFS}" (id 0) (at 187.8806 64.6248 90)
-      (effects (font (size 1.27 1.27)) (justify left) hide)
     )
   )
@@
     (pin "8")
   )
-  (symbol (lib_id "power:PWR_FLAG") (at 187.96 73.025 180) (unit 1)
-    (in_bom yes) (on_board yes) (fields_autoplaced)
-    (property "Reference" "#FLG0101" (id 0) (at 187.96 74.93 0)
-      (effects (font (size 1.27 1.27)) hide)
-    )
-    (property "Value" "PWR_FLAG" (id 1) (at 187.96 77.47 0))
-    (property "Footprint" "" (id 2) (at 187.96 73.025 0)
-      (effects (font (size 1.27 1.27)) hide)
-    )
-    (property "Datasheet" "~" (id 3) (at 187.96 73.025 0)
-      (effects (font (size 1.27 1.27)) hide)
-    )
-    (pin "1")
-  )
   (symbol (lib_id "Device:C_Polarized") (at 101.6 115.57 90) (unit 1)
     (in_bom yes) (on_board yes)
@@
   (symbol (lib_id "power:GND") (at 68.58 111.76 0) (unit 1)
     (in_bom yes) (on_board yes)
-    (property "Reference" "#PWR027" (id 0) (at 68.58 118.11 0)
+    (property "Reference" "#PWR019" (id 0) (at 68.58 118.11 0)
       (effects (font (size 1.27 1.27)) hide)
     )
@@
   (symbol (lib_id "power:PWR_FLAG") (at 157.48 87.63 0) (unit 1)
     (in_bom yes) (on_board yes) (fields_autoplaced)
-    (property "Reference" "#FLG0102" (id 0) (at 157.48 85.725 0)
+    (property "Reference" "#FLG04" (id 0) (at 157.48 85.725 0)
       (effects (font (size 1.27 1.27)) hide)
     )
@@
   (symbol (lib_id "power:GND") (at 157.48 99.06 0) (unit 1)
     (in_bom yes) (on_board yes)
-    (property "Reference" "#PWR034" (id 0) (at 157.48 105.41 0)
+    (property "Reference" "#PWR026" (id 0) (at 157.48 105.41 0)
       (effects (font (size 1.27 1.27)) hide)
     )
@@
   (symbol (lib_id "power:GND") (at 90.17 142.24 0) (unit 1)
     (in_bom yes) (on_board yes)
-    (property "Reference" "#PWR029" (id 0) (at 90.17 148.59 0)
+    (property "Reference" "#PWR021" (id 0) (at 90.17 148.59 0)
       (effects (font (size 1.27 1.27)) hide)
     )
@@
   (symbol (lib_id "power:GND") (at 137.16 113.03 0) (unit 1)
     (in_bom yes) (on_board yes)
-    (property "Reference" "#PWR031" (id 0) (at 137.16 119.38 0)
+    (property "Reference" "#PWR023" (id 0) (at 137.16 119.38 0)
       (effects (font (size 1.27 1.27)) hide)
     )
@@
   (symbol (lib_id "power:GND") (at 76.2 134.62 0) (unit 1)
     (in_bom yes) (on_board yes)
-    (property "Reference" "#PWR028" (id 0) (at 76.2 140.97 0)
+    (property "Reference" "#PWR020" (id 0) (at 76.2 140.97 0)
       (effects (font (size 1.27 1.27)) hide)
     )
@@
   (symbol (lib_id "power:GND") (at 140.97 97.155 0) (unit 1)
     (in_bom yes) (on_board yes)
-    (property "Reference" "#PWR032" (id 0) (at 140.97 103.505 0)
+    (property "Reference" "#PWR024" (id 0) (at 140.97 103.505 0)
       (effects (font (size 1.27 1.27)) hide)
     )
@@
   (symbol (lib_id "power:GND") (at 179.07 119.38 0) (unit 1)
     (in_bom yes) (on_board yes)
-    (property "Reference" "#PWR036" (id 0) (at 179.07 125.73 0)
+    (property "Reference" "#PWR028" (id 0) (at 179.07 125.73 0)
       (effects (font (size 1.27 1.27)) hide)
     )
@@
   (symbol (lib_id "power:GND") (at 165.735 133.35 0) (unit 1)
     (in_bom yes) (on_board yes) (fields_autoplaced)
-    (property "Reference" "#PWR035" (id 0) (at 165.735 139.7 0)
+    (property "Reference" "#PWR027" (id 0) (at 165.735 139.7 0)
       (effects (font (size 1.27 1.27)) hide)
     )
@@
   (symbol (lib_id "power:GND") (at 130.81 134.62 0) (unit 1)
     (in_bom yes) (on_board yes)
-    (property "Reference" "#PWR030" (id 0) (at 130.81 140.97 0)
+    (property "Reference" "#PWR022" (id 0) (at 130.81 140.97 0)
       (effects (font (size 1.27 1.27)) hide)
     )
@@
   (symbol (lib_id "power:PWR_FLAG") (at 90.17 101.6 0) (unit 1)
     (in_bom yes) (on_board yes) (fields_autoplaced)
-    (property "Reference" "#FLG0105" (id 0) (at 90.17 99.695 0)
+    (property "Reference" "#FLG03" (id 0) (at 90.17 99.695 0)
       (effects (font (size 1.27 1.27)) hide)
     )
@@
   (symbol (lib_id "power:GND") (at 144.78 124.46 0) (unit 1)
     (in_bom yes) (on_board yes)
-    (property "Reference" "#PWR033" (id 0) (at 144.78 130.81 0)
-      (effects (font (size 1.27 1.27)) hide)
-    )
+    (property "Reference" "#PWR025" (id 0) (at 144.78 130.81 0)
+      (effects (font (size 1.27 1.27)) hide)
+    )

Commit message: Update
Parts:
- renumbered C28 to C29, C29 to C30, C30 to C31, C31 to C32, C32 to C33, C33 to C34, C34 to C35, C35 to C36, C36 to C37, C37 to C38, C38 to C39, C39 to C40, J3 to J4
Changed lines of the file:
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@@
   (symbol (lib_id "Device:C_Polarized") (at 101.6 115.57 90) (unit 1)
     (in_bom yes) (on_board yes)
-    (property "Reference" "C30" (id 0) (at 97.79 119.38 0)
+    (property "Reference" "C31" (id 0) (at 97.79 119.38 0)
       (effects (font (size 1.27 1.27)) (justify left))
     )
@@
   (symbol (lib_id "Device:C") (at 147.32 101.6 180) (unit 1)
     (in_bom yes) (on_board yes)
-    (property "Reference" "C33" (id 0) (at 146.05 104.14 0)
+    (property "Reference" "C34" (id 0) (at 146.05 104.14 0)
       (effects (font (size 1.27 1.27)) (justify left))
     )
@@
   (symbol (lib_id "Device:C_Polarized") (at 68.58 107.95 0) (unit 1)
     (in_bom yes) (on_board yes)
-    (property "Reference" "C28" (id 0) (at 64.77 104.14 0)
+    (property "Reference" "C29" (id 0) (at 64.77 104.14 0)
       (effects (font (size 1.27 1.27)) (justify left))
     )
@@
   (symbol (lib_id "power:GND") (at 68.58 111.76 0) (unit 1)
     (in_bom yes) (on_board yes)
-    (property "Reference" "#PWR019" (id 0) (at 68.58 118.11 0)
+    (property "Reference" "#PWR021" (id 0) (at 68.58 118.11 0)
       (effects (font (size 1.27 1.27)) hide)
     )
@@
   (symbol (lib_id "Device:C_Polarized") (at 151.13 125.095 90) (unit 1)
     (in_bom yes) (on_board yes)
-    (property "Reference" "C35" (id 0) (at 148.59 122.555 0)
+    (property "Reference" "C36" (id 0) (at 148.59 122.555 0)
       (effects (font (size 1.27 1.27)) (justify left))
     )
@@
   (symbol (lib_id "Device:C_Polarized") (at 175.26 113.03 90) (unit 1)
     (in_bom yes) (on_board yes)
-    (property "Reference" "C39" (id 0) (at 172.72 110.49 0)
+    (property "Reference" "C40" (id 0) (at 172.72 110.49 0)
       (effects (font (size 1.27 1.27)) (justify left))
     )
@@
   (symbol (lib_id "power:GND") (at 157.48 99.06 0) (unit 1)
     (in_bom yes) (on_board yes)
-    (property "Reference" "#PWR026" (id 0) (at 157.48 105.41 0)
+    (property "Reference" "#PWR028" (id 0) (at 157.48 105.41 0)
       (effects (font (size 1.27 1.27)) hide)
     )
@@
   (symbol (lib_id "power:GND") (at 90.17 142.24 0) (unit 1)
     (in_bom yes) (on_board yes)
-    (property "Reference" "#PWR021" (id 0) (at 90.17 148.59 0)
+    (property "Reference" "#PWR023" (id 0) (at 90.17 148.59 0)
       (effects (font (size 1.27 1.27)) hide)
     )
@@
   (symbol (lib_id "power:GND") (at 137.16 113.03 0) (unit 1)
     (in_bom yes) (on_board yes)
-    (property "Reference" "#PWR023" (id 0) (at 137.16 119.38 0)
+    (property "Reference" "#PWR025" (id 0) (at 137.16 119.38 0)
       (effects (font (size 1.27 1.27)) hide)
     )
@@
   (symbol (lib_id "power:GND") (at 76.2 134.62 0) (unit 1)
     (in_bom yes) (on_board yes)
-    (property "Reference" "#PWR020" (id 0) (at 76.2 140.97 0)
+    (property "Reference" "#PWR022" (id 0) (at 76.2 140.97 0)
       (effects (font (size 1.27 1.27)) hide)
     )
@@
   (symbol (lib_id "power:GND") (at 140.97 97.155 0) (unit 1)
     (in_bom yes) (on_board yes)
-    (property "Reference" "#PWR024" (id 0) (at 140.97 103.505 0)
+    (property "Reference" "#PWR026" (id 0) (at 140.97 103.505 0)
       (effects (font (size 1.27 1.27)) hide)
     )
@@
   (symbol (lib_id "Device:C_Polarized") (at 163.83 92.71 0) (unit 1)
     (in_bom yes) (on_board yes)
-    (property "Reference" "C37" (id 0) (at 166.37 90.17 0)
+    (property "Reference" "C38" (id 0) (at 166.37 90.17 0)
       (effects (font (size 1.27 1.27)) (justify left))
     )
@@
   (symbol (lib_id "Device:C_Polarized") (at 70.485 121.92 90) (unit 1)
     (in_bom yes) (on_board yes)
-    (property "Reference" "C29" (id 0) (at 66.675 125.73 0)
+    (property "Reference" "C30" (id 0) (at 66.675 125.73 0)
       (effects (font (size 1.27 1.27)) (justify left))
     )
@@
   (symbol (lib_id "Device:C") (at 151.13 92.71 0) (unit 1)
     (in_bom yes) (on_board yes)
-    (property "Reference" "C34" (id 0) (at 152.4 90.17 0)
+    (property "Reference" "C35" (id 0) (at 152.4 90.17 0)
       (effects (font (size 1.27 1.27)) (justify left))
     )
@@
   (symbol (lib_id "Device:C") (at 116.84 121.92 0) (unit 1)
     (in_bom yes) (on_board yes)
-    (property "Reference" "C32" (id 0) (at 118.11 124.46 90))
+    (property "Reference" "C33" (id 0) (at 118.11 124.46 90))
     (property "Value" "10n" (id 1) (at 114.3 125.73 90))
     (property "Footprint" "Capacitor_THT:C_Disc_D3.4mm_W2.1mm_P2.50mm" (id 2) (at 117.8052 125.73 0)
@@
   (symbol (lib_id "Connector_Generic:Conn_01x02") (at 186.69 113.03 0) (unit 1)
     (in_bom yes) (on_board yes) (fields_autoplaced)
-    (property "Reference" "J3" (id 0) (at 189.23 113.0299 0)
+    (property "Reference" "J4" (id 0) (at 189.23 113.0299 0)
       (effects (font (size 1.27 1.27)) (justify left))
     )
@@
   (symbol (lib_id "power:GND") (at 179.07 119.38 0) (unit 1)
     (in_bom yes) (on_board yes)
-    (property "Reference" "#PWR028" (id 0) (at 179.07 125.73 0)
+    (property "Reference" "#PWR030" (id 0) (at 179.07 125.73 0)
       (effects (font (size 1.27 1.27)) hide)
     )
@@
   (symbol (lib_id "power:GND") (at 165.735 133.35 0) (unit 1)
     (in_bom yes) (on_board yes) (fields_autoplaced)
-    (property "Reference" "#PWR027" (id 0) (at 165.735 139.7 0)
+    (property "Reference" "#PWR029" (id 0) (at 165.735 139.7 0)
       (effects (font (size 1.27 1.27)) hide)
     )
@@
   (symbol (lib_id "Device:C") (at 165.735 118.11 0) (unit 1)
     (in_bom yes) (on_board yes) (fields_autoplaced)
-    (property "Reference" "C38" (id 0) (at 168.91 116.8399 0)
+    (property "Reference" "C39" (id 0) (at 168.91 116.8399 0)
       (effects (font (size 1.27 1.27)) (justify left))
     )
@@
   (symbol (lib_id "Device:C") (at 157.48 92.71 0) (unit 1)
     (in_bom yes) (on_board yes)
-    (property "Reference" "C36" (id 0) (at 158.75 90.17 0)
+    (property "Reference" "C37" (id 0) (at 158.75 90.17 0)
       (effects (font (size 1.27 1.27)) (justify left))
     )
@@
   (symbol (lib_id "power:GND") (at 130.81 134.62 0) (unit 1)
     (in_bom yes) (on_board yes)
-    (property "Reference" "#PWR022" (id 0) (at 130.81 140.97 0)
+    (property "Reference" "#PWR024" (id 0) (at 130.81 140.97 0)
       (effects (font (size 1.27 1.27)) hide)
     )
@@
   (symbol (lib_id "Device:C_Polarized") (at 102.87 133.35 0) (unit 1)
     (in_bom yes) (on_board yes)
-    (property "Reference" "C31" (id 0) (at 99.06 129.54 0)
+    (property "Reference" "C32" (id 0) (at 99.06 129.54 0)
       (effects (font (size 1.27 1.27)) (justify left))
     )
@@
   (symbol (lib_id "power:GND") (at 144.78 124.46 0) (unit 1)
     (in_bom yes) (on_board yes)
-    (property "Reference" "#PWR025" (id 0) (at 144.78 130.81 0)
-      (effects (font (size 1.27 1.27)) hide)
-    )
+    (property "Reference" "#PWR027" (id 0) (at 144.78 130.81 0)
+      (effects (font (size 1.27 1.27)) hide)
+    )
