File: AntSwitch.kicad_sch (KiCad schematic)
At the start: 17 parts, among them J10 Rev, J8 ANT, J9 Fwd, K4 G5V-2, T4 FT37-43 (1:10), T5 FT37-43 (1:10)

Commit message: Update
Parts:
- added J10: ANT_OUT, Connector_Coaxial:SMA_Amphenol_901-144_Vertical, symbol Connector:Conn_Coaxial
- added J12: PA_OUT, Connector_Coaxial:SMA_Amphenol_901-144_Vertical, symbol Connector:Conn_Coaxial
- added J9: ANT_IN, Connector_Coaxial:SMA_Amphenol_901-144_Vertical, symbol Connector:Conn_Coaxial
- renumbered C63 to C61, C64 to C62, C65 to C63, J8 to J11, J9 to J13, J10 to J14
Connections:
- net ANT_IN is gone; now on an unnamed net: K4.11
- net ANT_OUT: no longer K4.8
- net GND: now also J10.2 (Ext), J12.2 (Ext), J9.2 (Ext)
- net PA_OUT: now also J12.1 (In)
- net at K4.6: now also J9.1 (In)
- net at K4.9: now also K4.8, J10.1 (In)
- no-connect marks 2 -> 0
