File: IF_stage.kicad_sch (KiCad schematic)
At the start: 41 parts, among them J1 LO/BFO, J2 BFO/LO, K1 G5V-2, K2 G5V-2, T2 FT50-75 (18:7), T3 FT50-75 (7:18), U3 SA612, U4 SA612, Y1 12 MHz, Y2 12 MHz, Y3 12 MHz, Y4 12 MHz

Commit message: Add AF Stage
Connections:
- net IFAFOUT: now also K2.11
- net IFPAOUT: now also K2.8
- no-connect marks 4 -> 8
Changed lines of the file:
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@@
   (no_connect (at 83.82 92.71))
   (no_connect (at 217.17 120.65))
+  (no_connect (at 236.22 154.94))
+  (no_connect (at 220.98 154.94))
+  (no_connect (at 29.21 81.28))
+  (no_connect (at 29.21 96.52))
   (no_connect (at 64.77 100.33))
   (wire (pts (xy 224.79 93.98) (xy 231.14 93.98))
@@
     )
   )
-  (global_label "IFPAOUT" (shape output) (at 200.66 165.1 0) (fields_autoplaced)
-    (effects (font (size 1.27 1.27)) (justify left))
-    (property "Intersheet References" "${INTERSHEET_REFS}" (id 0) (at 210.7536 165.0206 0)
-      (effects (font (size 1.27 1.27)) (justify left) hide)
+  (global_label "IFPAOUT" (shape output) (at 210.82 165.1 180) (fields_autoplaced)
+    (effects (font (size 1.27 1.27)) (justify right))
+    (property "Intersheet References" "${INTERSHEET_REFS}" (id 0) (at 200.7264 165.1794 0)
+      (effects (font (size 1.27 1.27)) (justify right) hide)
     )
   )
@@
     )
   )
-  (global_label "IFAFOUT" (shape output) (at 200.66 158.75 0) (fields_autoplaced)
-    (effects (font (size 1.27 1.27)) (justify left))
-    (property "Intersheet References" "${INTERSHEET_REFS}" (id 0) (at 210.5721 158.6706 0)
-      (effects (font (size 1.27 1.27)) (justify left) hide)
+  (global_label "IFAFOUT" (shape output) (at 210.82 158.75 180) (fields_autoplaced)
+    (effects (font (size 1.27 1.27)) (justify right))
+    (property "Intersheet References" "${INTERSHEET_REFS}" (id 0) (at 200.9079 158.8294 0)
+      (effects (font (size 1.27 1.27)) (justify right) hide)
     )
   )
@@
     (pin "1")
   )
-  (symbol (lib_id "power:GND") (at 231.14 40.64 0) (unit 1)
-    (in_bom yes) (on_board yes) (fields_autoplaced)
-    (property "Reference" "#PWR023" (id 0) (at 231.14 46.99 0)
-      (effects (font (size 1.27 1.27)) hide)
-    )
-    (property "Value" "GND" (id 1) (at 231.14 45.72 0))
-    (property "Footprint" "" (id 2) (at 231.14 40.64 0)
-      (effects (font (size 1.27 1.27)) hide)
-    )
-    (property "Datasheet" "" (id 3) (at 231.14 40.64 0)
+  (symbol (lib_id "power:GND") (at 248.285 27.305 0) (unit 1)
+    (in_bom yes) (on_board yes) (fields_autoplaced)
+    (property "Reference" "#PWR023" (id 0) (at 248.285 33.655 0)
+      (effects (font (size 1.27 1.27)) hide)
+    )
+    (property "Value" "GND" (id 1) (at 248.285 32.385 0))
+    (property "Footprint" "" (id 2) (at 248.285 27.305 0)
+      (effects (font (size 1.27 1.27)) hide)
+    )
+    (property "Datasheet" "" (id 3) (at 248.285 27.305 0)
       (effects (font (size 1.27 1.27)) hide)
     )
@@
     (pin "2")
   )
+  (symbol (lib_id "power:PWR_FLAG") (at 93.98 68.58 0) (unit 1)
+    (in_bom yes) (on_board yes) (fields_autoplaced)
+    (property "Reference" "#FLG0103" (id 0) (at 93.98 66.675 0)
+      (effects (font (size 1.27 1.27)) hide)
+    )
+    (property "Value" "PWR_FLAG" (id 1) (at 95.885 67.3099 0)
+      (effects (font (size 1.27 1.27)) (justify left))
+    )
+    (property "Footprint" "" (id 2) (at 93.98 68.58 0)
+      (effects (font (size 1.27 1.27)) hide)
+    )
+    (property "Datasheet" "~" (id 3) (at 93.98 68.58 0)
+      (effects (font (size 1.27 1.27)) hide)
+    )
+    (pin "1")
+  )
   (symbol (lib_id "power:GND") (at 256.54 137.16 90) (unit 1)
     (in_bom yes) (on_board yes) (fields_autoplaced)
@@
     (pin "2")
   )
+  (symbol (lib_id "power:PWR_FLAG") (at 231.14 93.98 0) (unit 1)
+    (in_bom yes) (on_board yes) (fields_autoplaced)
+    (property "Reference" "#FLG0104" (id 0) (at 231.14 92.075 0)
+      (effects (font (size 1.27 1.27)) hide)
+    )
+    (property "Value" "PWR_FLAG" (id 1) (at 233.045 92.7099 0)
+      (effects (font (size 1.27 1.27)) (justify left))
+    )
+    (property "Footprint" "" (id 2) (at 231.14 93.98 0)
+      (effects (font (size 1.27 1.27)) hide)
+    )
+    (property "Datasheet" "~" (id 3) (at 231.14 93.98 0)
+      (effects (font (size 1.27 1.27)) hide)
+    )
+    (pin "1")
+  )
   (symbol (lib_id "power:+8V") (at 231.14 27.94 0) (unit 1)
     (in_bom yes) (on_board yes)
@@
     (pin "2")
   )
-  (symbol (lib_id "power:PWR_FLAG") (at 231.14 40.64 0) (unit 1)
-    (in_bom yes) (on_board yes) (fields_autoplaced)
-    (property "Reference" "#FLG05" (id 0) (at 231.14 38.735 0)
-      (effects (font (size 1.27 1.27)) hide)
-    )
-    (property "Value" "PWR_FLAG" (id 1) (at 231.14 35.56 0))
-    (property "Footprint" "" (id 2) (at 231.14 40.64 0)
-      (effects (font (size 1.27 1.27)) hide)
-    )
-    (property "Datasheet" "~" (id 3) (at 231.14 40.64 0)
-      (effects (font (size 1.27 1.27)) hide)
-    )
+  (symbol (lib_id "power:PWR_FLAG") (at 248.285 27.305 0) (unit 1)
+    (in_bom yes) (on_board yes) (fields_autoplaced)
+    (property "Reference" "#FLG05" (id 0) (at 248.285 25.4 0)
+      (effects (font (size 1.27 1.27)) hide)
+    )
+    (property "Value" "PWR_FLAG" (id 1) (at 248.285 22.225 0))
+    (property "Footprint" "" (id 2) (at 248.285 27.305 0)
+      (effects (font (size 1.27 1.27)) hide)
+    )
+    (property "Datasheet" "~" (id 3) (at 248.285 27.305 0)
+      (effects (font (size 1.27 1.27)) hide)
+    )

Commit message: Continue Migration from D612
Connections:
- net +8V renamed 8V
Other:
- note added: "Can also be 5V for Less gain"
Changed lines of the file:
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@@
-    (stroke (width 0) (type default) (color 0 0 0 0))
-  )
-  (wire (pts (xy 212.09 26.67) (xy 212.09 29.21))
     (stroke (width 0) (type default) (color 0 0 0 0))
   )
@@
   (wire (pts (xy 252.73 137.16) (xy 256.54 137.16))
     (stroke (width 0) (type default) (color 0 0 0 0))
+  )
+  (text "Can also be 5V for Less gain" (at 71.12 41.275 0)
+    (effects (font (size 1.27 1.27)) (justify left bottom))
+  )
+  (global_label "8V" (shape output) (at 81.28 46.99 90) (fields_autoplaced)
+    (effects (font (size 1.27 1.27)) (justify left))
+    (property "Intersheet References" "${INTERSHEET_REFS}" (id 0) (at 81.2006 42.2788 90)
+      (effects (font (size 1.27 1.27)) (justify left) hide)
+    )
   )
   (global_label "IFRFIN" (shape input) (at 20.32 81.28 90) (fields_autoplaced)
@@
     )
   )
+  (global_label "8V" (shape output) (at 218.44 72.39 90) (fields_autoplaced)
+    (effects (font (size 1.27 1.27)) (justify left))
+    (property "Intersheet References" "${INTERSHEET_REFS}" (id 0) (at 218.3606 67.6788 90)
+      (effects (font (size 1.27 1.27)) (justify left) hide)
+    )
+  )
   (global_label "IFPAOUT" (shape output) (at 210.82 165.1 180) (fields_autoplaced)
     (effects (font (size 1.27 1.27)) (justify right))
@@
     )
   )
-  (global_label "TX12V" (shape input) (at 212.09 26.67 90) (fields_autoplaced)
-    (effects (font (size 1.27 1.27)) (justify left))
-    (property "Intersheet References" "${INTERSHEET_REFS}" (id 0) (at 212.1694 18.5721 90)
-      (effects (font (size 1.27 1.27)) (justify left) hide)
-    )
-  )
   (global_label "IFAFOUT" (shape output) (at 210.82 158.75 180) (fields_autoplaced)
     (effects (font (size 1.27 1.27)) (justify right))
@@
   (symbol (lib_id "power:GND") (at 190.5 134.62 0) (unit 1)
     (in_bom yes) (on_board yes) (fields_autoplaced)
-    (property "Reference" "#PWR020" (id 0) (at 190.5 140.97 0)
+    (property "Reference" "#PWR015" (id 0) (at 190.5 140.97 0)
       (effects (font (size 1.27 1.27)) hide)
     )
@@
   (symbol (lib_id "power:GND") (at 93.98 81.28 0) (unit 1)
     (in_bom yes) (on_board yes)
-    (property "Reference" "#PWR015" (id 0) (at 93.98 87.63 0)
+    (property "Reference" "#PWR010" (id 0) (at 93.98 87.63 0)
       (effects (font (size 1.27 1.27)) hide)
     )
@@
     (pin "1")
     (pin "2")
-  )
-  (symbol (lib_id "power:PWR_FLAG") (at 212.09 29.21 180) (unit 1)
-    (in_bom yes) (on_board yes) (fields_autoplaced)
-    (property "Reference" "#FLG03" (id 0) (at 212.09 31.115 0)
-      (effects (font (size 1.27 1.27)) hide)
-    )
-    (property "Value" "PWR_FLAG" (id 1) (at 214.63 30.4799 0)
-      (effects (font (size 1.27 1.27)) (justify right))
-    )
-    (property "Footprint" "" (id 2) (at 212.09 29.21 0)
-      (effects (font (size 1.27 1.27)) hide)
-    )
-    (property "Datasheet" "~" (id 3) (at 212.09 29.21 0)
-      (effects (font (size 1.27 1.27)) hide)
-    )
-    (pin "1")
   )
   (symbol (lib_id "Diode:1N914") (at 252.73 148.59 90) (unit 1)
@@
     (pin "2")
   )
-  (symbol (lib_id "power:+8V") (at 81.28 46.99 0) (unit 1)
-    (in_bom yes) (on_board yes)
-    (property "Reference" "#PWR014" (id 0) (at 81.28 50.8 0)
-      (effects (font (size 1.27 1.27)) hide)
-    )
-    (property "Value" "+8V" (id 1) (at 81.28 41.91 0))
-    (property "Footprint" "" (id 2) (at 81.28 46.99 0)
-      (effects (font (size 1.27 1.27)) hide)
-    )
-    (property "Datasheet" "" (id 3) (at 81.28 46.99 0)
-      (effects (font (size 1.27 1.27)) hide)
-    )
-    (pin "1")
-  )
   (symbol (lib_id "Device:R_US") (at 81.28 60.96 0) (unit 1)
     (in_bom yes) (on_board yes) (fields_autoplaced)
@@
     (pin "1")
     (pin "2")
-  )
-  (symbol (lib_id "power:+8V") (at 218.44 72.39 0) (unit 1)
-    (in_bom yes) (on_board yes)
-    (property "Reference" "#PWR021" (id 0) (at 218.44 76.2 0)
-      (effects (font (size 1.27 1.27)) hide)
-    )
-    (property "Value" "+8V" (id 1) (at 218.44 67.31 0))
-    (property "Footprint" "" (id 2) (at 218.44 72.39 0)
-      (effects (font (size 1.27 1.27)) hide)
-    )
-    (property "Datasheet" "" (id 3) (at 218.44 72.39 0)
-      (effects (font (size 1.27 1.27)) hide)
-    )
-    (pin "1")
-  )
-  (symbol (lib_id "power:GND") (at 248.285 27.305 0) (unit 1)
-    (in_bom yes) (on_board yes) (fields_autoplaced)
-    (property "Reference" "#PWR023" (id 0) (at 248.285 33.655 0)
-      (effects (font (size 1.27 1.27)) hide)
-    )
-    (property "Value" "GND" (id 1) (at 248.285 32.385 0))
-    (property "Footprint" "" (id 2) (at 248.285 27.305 0)
-      (effects (font (size 1.27 1.27)) hide)
-    )
-    (property "Datasheet" "" (id 3) (at 248.285 27.305 0)
-      (effects (font (size 1.27 1.27)) hide)
-    )
-    (pin "1")
   )
   (symbol (lib_id "Device:C") (at 147.32 104.14 0) (unit 1)
@@
   (symbol (lib_id "power:GND") (at 118.11 116.84 0) (unit 1)
     (in_bom yes) (on_board yes) (fields_autoplaced)
-    (property "Reference" "#PWR016" (id 0) (at 118.11 123.19 0)
+    (property "Reference" "#PWR011" (id 0) (at 118.11 123.19 0)
       (effects (font (size 1.27 1.27)) hide)
     )
@@
   (symbol (lib_id "power:PWR_FLAG") (at 93.98 68.58 0) (unit 1)
     (in_bom yes) (on_board yes) (fields_autoplaced)
-    (property "Reference" "#FLG0103" (id 0) (at 93.98 66.675 0)
+    (property "Reference" "#FLG01" (id 0) (at 93.98 66.675 0)
       (effects (font (size 1.27 1.27)) hide)
     )
@@
   (symbol (lib_id "power:GND") (at 256.54 137.16 90) (unit 1)
     (in_bom yes) (on_board yes) (fields_autoplaced)
-    (property "Reference" "#PWR026" (id 0) (at 262.89 137.16 0)
+    (property "Reference" "#PWR018" (id 0) (at 262.89 137.16 0)
       (effects (font (size 1.27 1.27)) hide)
     )
@@
   (symbol (lib_id "power:GND") (at 57.15 106.68 0) (unit 1)
     (in_bom yes) (on_board yes) (fields_autoplaced)
-    (property "Reference" "#PWR013" (id 0) (at 57.15 113.03 0)
+    (property "Reference" "#PWR09" (id 0) (at 57.15 113.03 0)
       (effects (font (size 1.27 1.27)) hide)
     )
@@
   (symbol (lib_id "power:PWR_FLAG") (at 231.14 93.98 0) (unit 1)
     (in_bom yes) (on_board yes) (fields_autoplaced)
-    (property "Reference" "#FLG0104" (id 0) (at 231.14 92.075 0)
+    (property "Reference" "#FLG02" (id 0) (at 231.14 92.075 0)
       (effects (font (size 1.27 1.27)) hide)
     )
@@
     )
     (property "Datasheet" "~" (id 3) (at 231.14 93.98 0)
-      (effects (font (size 1.27 1.27)) hide)
-    )
-    (pin "1")
-  )
-  (symbol (lib_id "power:+8V") (at 231.14 27.94 0) (unit 1)
-    (in_bom yes) (on_board yes)
-    (property "Reference" "#PWR022" (id 0) (at 231.14 31.75 0)
-      (effects (font (size 1.27 1.27)) hide)
-    )
-    (property "Value" "+8V" (id 1) (at 231.14 22.86 0))
-    (property "Footprint" "" (id 2) (at 231.14 27.94 0)
-      (effects (font (size 1.27 1.27)) hide)
-    )
-    (property "Datasheet" "" (id 3) (at 231.14 27.94 0)
-      (effects (font (size 1.27 1.27)) hide)
-    )
-    (pin "1")
-  )
-  (symbol (lib_id "power:PWR_FLAG") (at 231.14 27.94 180) (unit 1)
-    (in_bom yes) (on_board yes) (fields_autoplaced)
-    (property "Reference" "#FLG04" (id 0) (at 231.14 29.845 0)
-      (effects (font (size 1.27 1.27)) hide)
-    )
-    (property "Value" "PWR_FLAG" (id 1) (at 233.68 29.2099 0)
-      (effects (font (size 1.27 1.27)) (justify right))
-    )
-    (property "Footprint" "" (id 2) (at 231.14 27.94 0)
-      (effects (font (size 1.27 1.27)) hide)
-    )
-    (property "Datasheet" "~" (id 3) (at 231.14 27.94 0)
       (effects (font (size 1.27 1.27)) hide)
     )
@@
   (symbol (lib_id "power:GND") (at 246.38 116.84 0) (unit 1)
     (in_bom yes) (on_board yes)
-    (property "Reference" "#PWR025" (id 0) (at 246.38 123.19 0)
+    (property "Reference" "#PWR017" (id 0) (at 246.38 123.19 0)
       (effects (font (size 1.27 1.27)) hide)
     )
@@
   (symbol (lib_id "power:GND") (at 147.32 113.03 0) (unit 1)
     (in_bom yes) (on_board yes) (fields_autoplaced)
-    (property "Reference" "#PWR018" (id 0) (at 147.32 119.38 0)
+    (property "Reference" "#PWR013" (id 0) (at 147.32 119.38 0)
       (effects (font (size 1.27 1.27)) hide)
     )
@@
     (pin "2")
   )
-  (symbol (lib_id "power:PWR_FLAG") (at 248.285 27.305 0) (unit 1)
-    (in_bom yes) (on_board yes) (fields_autoplaced)
-    (property "Reference" "#FLG05" (id 0) (at 248.285 25.4 0)
-      (effects (font (size 1.27 1.27)) hide)
-    )
-    (property "Value" "PWR_FLAG" (id 1) (at 248.285 22.225 0))
-    (property "Footprint" "" (id 2) (at 248.285 27.305 0)
-      (effects (font (size 1.27 1.27)) hide)
-    )
-    (property "Datasheet" "~" (id 3) (at 248.285 27.305 0)
-      (effects (font (size 1.27 1.27)) hide)
-    )
-    (pin "1")
-  )
   (symbol (lib_id "Device:R_US") (at 20.32 119.38 0) (unit 1)
     (in_bom yes) (on_board yes) (fields_autoplaced)
@@
   (symbol (lib_id "power:GND") (at 161.29 129.54 0) (unit 1)
     (in_bom yes) (on_board yes) (fields_autoplaced)
-    (property "Reference" "#PWR019" (id 0) (at 161.29 135.89 0)
+    (property "Reference" "#PWR014" (id 0) (at 161.29 135.89 0)
       (effects (font (size 1.27 1.27)) hide)
     )
@@
   (symbol (lib_id "power:GND") (at 121.92 78.74 0) (unit 1)
     (in_bom yes) (on_board yes)
-    (property "Reference" "#PWR017" (id 0) (at 121.92 85.09 0)
+    (property "Reference" "#PWR012" (id 0) (at 121.92 85.09 0)
       (effects (font (size 1.27 1.27)) hide)
     )
@@
   (symbol (lib_id "power:GND") (at 231.14 106.68 0) (unit 1)
     (in_bom yes) (on_board yes)
-    (property "Reference" "#PWR024" (id 0) (at 231.14 113.03 0)
+    (property "Reference" "#PWR016" (id 0) (at 231.14 113.03 0)
       (effects (font (size 1.27 1.27)) hide)
     )
@@
   (symbol (lib_id "power:GND") (at 48.26 118.11 0) (unit 1)
     (in_bom yes) (on_board yes) (fields_autoplaced)
-    (property "Reference" "#PWR012" (id 0) (at 48.26 124.46 0)
-      (effects (font (size 1.27 1.27)) hide)
-    )
+    (property "Reference" "#PWR08" (id 0) (at 48.26 124.46 0)
+      (effects (font (size 1.27 1.27)) hide)
+    )

Commit message: Update
Parts:
- renumbered C9 to C10, C10 to C11, C11 to C12, C12 to C13, C13 to C14, C14 to C15, C15 to C16, C16 to C17, C17 to C18, C18 to C19, C19 to C20, C20 to C21, C21 to C22, C22 to C23, C23 to C24, C24 to C25, C25 to C26, C26 to C27, C27 to C28, C8 to C9, J1 to J2, J2 to J3
Connections:
- net IFAFOUT: now also K2.6
- net IFMICIN: now also K1.9
- net IFPAOUT: now also K2.9
- net IFRFIN: now also K1.6
- net 8V renamed RX5V
- no-connect marks 8 -> 4
