File: MicPreamp.kicad_sch (KiCad schematic)
At the start: 17 parts, among them J5 MICIN, Q2 2N3904

Commit message: Update
Parts:
- renumbered C46 to C47, C47 to C48, C48 to C49, C49 to C50, C50 to C51, C51 to C52, C52 to C53, J5 to J6
Changed lines of the file:
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@@
   (symbol (lib_id "Connector_Generic:Conn_01x02") (at 62.23 104.775 180) (unit 1)
     (in_bom yes) (on_board yes) (fields_autoplaced)
-    (property "Reference" "J5" (id 0) (at 62.23 95.25 0))
+    (property "Reference" "J6" (id 0) (at 62.23 95.25 0))
     (property "Value" "MICIN" (id 1) (at 62.23 97.79 0))
     (property "Footprint" "Connector_PinHeader_2.54mm:PinHeader_1x02_P2.54mm_Vertical" (id 2) (at 62.23 104.775 0)
@@
   (symbol (lib_id "power:GND") (at 67.31 107.315 0) (unit 1)
     (in_bom yes) (on_board yes)
-    (property "Reference" "#PWR037" (id 0) (at 67.31 113.665 0)
+    (property "Reference" "#PWR039" (id 0) (at 67.31 113.665 0)
       (effects (font (size 1.27 1.27)) hide)
     )
@@
   (symbol (lib_id "Device:C") (at 75.565 108.585 0) (unit 1)
     (in_bom yes) (on_board yes)
-    (property "Reference" "C47" (id 0) (at 76.835 111.125 90))
+    (property "Reference" "C48" (id 0) (at 76.835 111.125 90))
     (property "Value" "10n" (id 1) (at 73.66 111.76 90))
     (property "Footprint" "Capacitor_THT:C_Disc_D3.4mm_W2.1mm_P2.50mm" (id 2) (at 76.5302 112.395 0)
@@
   (symbol (lib_id "power:GND") (at 76.2 83.185 0) (unit 1)
     (in_bom yes) (on_board yes)
-    (property "Reference" "#PWR039" (id 0) (at 76.2 89.535 0)
+    (property "Reference" "#PWR041" (id 0) (at 76.2 89.535 0)
       (effects (font (size 1.27 1.27)) hide)
     )
@@
   (symbol (lib_id "Device:C") (at 150.495 97.155 0) (unit 1)
     (in_bom yes) (on_board yes) (fields_autoplaced)
-    (property "Reference" "C52" (id 0) (at 153.67 95.8849 0)
+    (property "Reference" "C53" (id 0) (at 153.67 95.8849 0)
       (effects (font (size 1.27 1.27)) (justify left))
     )
@@
   (symbol (lib_id "power:GND") (at 90.17 114.935 0) (unit 1)
     (in_bom yes) (on_board yes)
-    (property "Reference" "#PWR040" (id 0) (at 90.17 121.285 0)
+    (property "Reference" "#PWR042" (id 0) (at 90.17 121.285 0)
       (effects (font (size 1.27 1.27)) hide)
     )
@@
   (symbol (lib_id "Device:C_Polarized") (at 96.52 102.235 90) (unit 1)
     (in_bom yes) (on_board yes)
-    (property "Reference" "C50" (id 0) (at 93.98 99.695 0)
+    (property "Reference" "C51" (id 0) (at 93.98 99.695 0)
       (effects (font (size 1.27 1.27)) (justify left))
     )
@@
   (symbol (lib_id "power:GND") (at 142.24 99.06 0) (unit 1)
     (in_bom yes) (on_board yes)
-    (property "Reference" "#PWR042" (id 0) (at 142.24 105.41 0)
+    (property "Reference" "#PWR044" (id 0) (at 142.24 105.41 0)
       (effects (font (size 1.27 1.27)) hide)
     )
@@
   (symbol (lib_id "Device:C_Polarized") (at 82.55 76.835 0) (unit 1)
     (in_bom yes) (on_board yes)
-    (property "Reference" "C49" (id 0) (at 85.09 74.295 0)
+    (property "Reference" "C50" (id 0) (at 85.09 74.295 0)
       (effects (font (size 1.27 1.27)) (justify left))
     )
@@
   (symbol (lib_id "power:GND") (at 150.495 112.395 0) (unit 1)
     (in_bom yes) (on_board yes) (fields_autoplaced)
-    (property "Reference" "#PWR043" (id 0) (at 150.495 118.745 0)
+    (property "Reference" "#PWR045" (id 0) (at 150.495 118.745 0)
       (effects (font (size 1.27 1.27)) hide)
     )
@@
   (symbol (lib_id "power:GND") (at 113.03 111.125 0) (unit 1)
     (in_bom yes) (on_board yes)
-    (property "Reference" "#PWR041" (id 0) (at 113.03 117.475 0)
+    (property "Reference" "#PWR043" (id 0) (at 113.03 117.475 0)
       (effects (font (size 1.27 1.27)) hide)
     )
@@
   (symbol (lib_id "Device:C") (at 69.85 76.835 0) (unit 1)
     (in_bom yes) (on_board yes)
-    (property "Reference" "C46" (id 0) (at 71.12 74.295 0)
+    (property "Reference" "C47" (id 0) (at 71.12 74.295 0)
       (effects (font (size 1.27 1.27)) (justify left))
     )
@@
   (symbol (lib_id "power:GND") (at 75.565 115.57 0) (unit 1)
     (in_bom yes) (on_board yes)
-    (property "Reference" "#PWR038" (id 0) (at 75.565 121.92 0)
+    (property "Reference" "#PWR040" (id 0) (at 75.565 121.92 0)
       (effects (font (size 1.27 1.27)) hide)
     )
@@
   (symbol (lib_id "Device:C") (at 76.2 76.835 0) (unit 1)
     (in_bom yes) (on_board yes)
-    (property "Reference" "C48" (id 0) (at 77.47 74.295 0)
+    (property "Reference" "C49" (id 0) (at 77.47 74.295 0)
       (effects (font (size 1.27 1.27)) (justify left))
     )
@@
   (symbol (lib_id "Device:C_Polarized") (at 124.46 95.885 90) (unit 1)
     (in_bom yes) (on_board yes)
-    (property "Reference" "C51" (id 0) (at 121.92 93.345 0)
-      (effects (font (size 1.27 1.27)) (justify left))
-    )
+    (property "Reference" "C52" (id 0) (at 121.92 93.345 0)
+      (effects (font (size 1.27 1.27)) (justify left))
+    )
