File: Phoenix612.kicad_pcb (KiCad board)
At the start: 2 copper layers, 233.6 x 93.2 mm, 62 parts, among them J1 LO/BFO, J2 BFO/LO, K1 G5V-2, K2 G5V-2, T1 FT50-74 (22:4), T2 FT50-75 (18:7), T3 FT50-75 (7:18), U1 LT1253, U2 QPR_Filter, U3 SA612, U4 SA612, Y1 12 MHz, Y2 12 MHz, Y3 12 MHz, Y4 12 MHz

Commit message: Add AF Stage
Parts:
- added C28: 47u, Capacitor_THT:CP_Radial_D8.0mm_P2.50mm, F.Cu at (225.0, 113.8)
- added C29: 47u, Capacitor_THT:CP_Radial_D8.0mm_P2.50mm, F.Cu at (205.5, 106.2)
- added C30: 47u, Capacitor_THT:CP_Radial_D8.0mm_P2.50mm, F.Cu at (205.2, 124.2)
- added C31: 100u, Capacitor_THT:CP_Radial_D8.0mm_P2.50mm, F.Cu at (199.1, 112.8)
- added C32: 10n, Capacitor_THT:C_Disc_D3.4mm_W2.1mm_P2.50mm, F.Cu at (221.0, 127.3)
- added C33: 1u, Capacitor_THT:C_Disc_D3.4mm_W2.1mm_P2.50mm, F.Cu at (230.6, 147.8)
- added C34: 100n, Capacitor_THT:C_Disc_D3.4mm_W2.1mm_P2.50mm, F.Cu at (236.5, 140.2)
- added C35: 10u, Capacitor_THT:CP_Radial_D8.0mm_P2.50mm, F.Cu at (218.7, 137.0)
- added C36: 1n, Capacitor_THT:C_Disc_D3.4mm_W2.1mm_P2.50mm, F.Cu at (236.5, 143.5)
- added C37: 220u, Capacitor_THT:CP_Radial_D8.0mm_P2.50mm, F.Cu at (236.3, 149.9)
- added C38: 10n, Capacitor_THT:C_Disc_D3.4mm_W2.1mm_P2.50mm, F.Cu at (209.0, 140.7)
- added C39: 100u, Capacitor_THT:CP_Radial_D8.0mm_P2.50mm, F.Cu at (209.4, 150.4)
- added J3: SPK, Connector_PinHeader_2.54mm:PinHeader_1x02_P2.54mm_Vertical, F.Cu at (217.4, 150.1)
- added Q1: 2N3904, Package_TO_SOT_THT:TO-92_Inline, F.Cu at (203.7, 115.4)
- added R14: 100R, Resistor_THT:R_Axial_DIN0207_L6.3mm_D2.5mm_P10.16mm_Horizontal, F.Cu at (229.4, 108.5)
- added R15: 100K, Resistor_THT:R_Axial_DIN0207_L6.3mm_D2.5mm_P10.16mm_Horizontal, F.Cu at (219.7, 112.0)
- added R16: 10K, Resistor_THT:R_Axial_DIN0207_L6.3mm_D2.5mm_P10.16mm_Horizontal, F.Cu at (209.6, 115.6)
- added R17: 1K, Resistor_THT:R_Axial_DIN0207_L6.3mm_D2.5mm_P10.16mm_Horizontal, F.Cu at (217.2, 119.6)
- added R18: 470R, Resistor_THT:R_Axial_DIN0207_L6.3mm_D2.5mm_P10.16mm_Horizontal, F.Cu at (203.7, 119.6)
- added R19: 2.7K, Resistor_THT:R_Axial_DIN0207_L6.3mm_D2.5mm_P10.16mm_Horizontal, F.Cu at (210.8, 124.0)
- added R20: 100R, Resistor_THT:R_Axial_DIN0207_L6.3mm_D2.5mm_P10.16mm_Horizontal, F.Cu at (236.7, 127.0)
- added R21: 10R, Resistor_THT:R_Axial_DIN0207_L6.3mm_D2.5mm_P10.16mm_Horizontal, F.Cu at (222.0, 143.0)
- added RV3: 10K, Potentiometer_THT:Potentiometer_Bourns_3296W_Vertical, F.Cu at (226.3, 124.2)
- added U5: LM386, Package_DIP:DIP-8_W7.62mm_Socket, F.Cu at (225.3, 135.1)
Connections:
- K2 pad 11: unconnected-(K2-Pad11) -> IFAFOUT
- K2 pad 8: unconnected-(K2-Pad8) -> IFPAOUT
Routing:
- net GND: track 378.4 -> 506.5 mm
- net Net-(C38-Pad1): track 0.00 -> 34.9 mm
- net RX12V: track 0.00 -> 21.6 mm
- net Net-(C28-Pad1): track 0.00 -> 17.5 mm
- net Net-(C34-Pad1): track 0.00 -> 16.4 mm
- net Net-(C35-Pad2): track 0.00 -> 14.9 mm
- net Net-(C29-Pad2): track 0.00 -> 14.7 mm
- net Net-(RV3-Pad2): track 0.00 -> 12.7 mm
- net Net-(C33-Pad1): track 0.00 -> 11.3 mm
- net Net-(C31-Pad1): track 0.00 -> 10.1 mm
- net Net-(C30-Pad1): track 0.00 -> 9.84 mm
- net SMeterIN: track 0.00 -> 8.76 mm
- net Net-(C35-Pad1): track 0.00 -> 7.40 mm
- net IFAFOUT: track 0.00 -> 7.26 mm
- net Net-(C30-Pad2): track 0.00 -> 6.73 mm
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Other:
- board size 233.6 x 93.2 mm -> 236.4 x 120.1 mm

Commit message: Continue Migration from D612
Parts:
- added C40: 10u, Capacitor_THT:C_Disc_D3.4mm_W2.1mm_P2.50mm, F.Cu at (230.9, 123.7)
- added C41: 100n, Capacitor_THT:C_Disc_D3.4mm_W2.1mm_P2.50mm, F.Cu at (263.4, 123.0)
- added C42: 1n, Capacitor_THT:C_Disc_D3.4mm_W2.1mm_P2.50mm, F.Cu at (266.7, 123.2)
- added C43: 10u, Capacitor_THT:CP_Radial_D8.0mm_P2.50mm, F.Cu at (257.6, 111.5)
- added C44: 10u, Capacitor_THT:CP_Radial_D8.0mm_P2.50mm, F.Cu at (255.4, 131.8)
- added C45: 10n, Capacitor_THT:C_Disc_D3.4mm_W2.1mm_P2.50mm, F.Cu at (265.4, 147.1)
- added C46: 100n, Capacitor_THT:C_Disc_D3.4mm_W2.1mm_P2.50mm, F.Cu at (55.9, 93.7)
- added C47: 10n, Capacitor_THT:C_Disc_D3.4mm_W2.1mm_P2.50mm, F.Cu at (28.7, 108.7)
- added C48: 1n, Capacitor_THT:C_Disc_D3.4mm_W2.1mm_P2.50mm, F.Cu at (62.0, 93.7)
- added C49: 47u, Capacitor_THT:CP_Radial_D8.0mm_P2.50mm, F.Cu at (47.0, 93.5)
- added C50: 47u, Capacitor_THT:CP_Radial_D8.0mm_P2.50mm, F.Cu at (39.7, 109.0)
- added C51: 47u, Capacitor_THT:CP_Radial_D8.0mm_P2.50mm, F.Cu at (58.3, 109.0)
- added C52: 10n, Capacitor_THT:C_Disc_D3.4mm_W2.1mm_P2.50mm, F.Cu at (76.4, 112.5)
- added C53: 22u, Capacitor_THT:CP_Radial_D8.0mm_P2.50mm, F.Cu at (202.3, 21.1)
- added C54: 22u, Capacitor_THT:CP_Radial_D8.0mm_P2.50mm, F.Cu at (153.3, 21.3)
- added C55: 22u, Capacitor_THT:CP_Radial_D8.0mm_P2.50mm, F.Cu at (219.2, 20.8)
- added C56: 22u, Capacitor_THT:CP_Radial_D8.0mm_P2.50mm, F.Cu at (170.8, 23.1)
- added C57: 0.1u, Capacitor_THT:C_Disc_D3.0mm_W1.6mm_P2.50mm, F.Cu at (214.6, 25.9)
- added C58: 0.1u, Capacitor_THT:C_Disc_D3.0mm_W1.6mm_P2.50mm, F.Cu at (165.1, 29.2)
- added C59: 100n, Capacitor_THT:C_Disc_D3.4mm_W2.1mm_P2.50mm, F.Cu at (98.0, 25.9)
- added C60: 100n, Capacitor_THT:C_Disc_D3.4mm_W2.1mm_P2.50mm, F.Cu at (49.3, 157.0)
- added C61: 100n, Capacitor_THT:C_Disc_D3.4mm_W2.1mm_P2.50mm, F.Cu at (97.5, 147.1)
- added C62: 100n, Capacitor_THT:C_Disc_D3.4mm_W2.1mm_P2.50mm, F.Cu at (107.4, 125.7)
- added D10: 1N914, Diode_THT:D_DO-35_SOD27_P7.62mm_Horizontal, F.Cu at (85.9, 155.2)
- added D11: 1N914, Diode_THT:D_DO-35_SOD27_P7.62mm_Horizontal, F.Cu at (99.6, 125.2)
- added D3: 1N4148, Diode_THT:D_DO-35_SOD27_P7.62mm_Horizontal, F.Cu at (266.2, 138.7)
- added D4: LED, LED_THT:LED_D3.0mm, F.Cu at (182.1, 29.7)
- added D5: LED, LED_THT:LED_D3.0mm, F.Cu at (192.5, 29.7)
- added D6: LED, LED_THT:LED_D3.0mm, F.Cu at (187.5, 29.7)
- added D7: 1N4001, Diode_THT:D_DO-41_SOD81_P10.16mm_Horizontal, F.Cu at (158.5, 16.8)
- added D8: 1N914, Diode_THT:D_DO-35_SOD27_P7.62mm_Horizontal, F.Cu at (95.0, 26.4)
- added D9: 1N914, Diode_THT:D_DO-35_SOD27_P7.62mm_Horizontal, F.Cu at (52.1, 153.7)
- added J10: Rev, Connector_PinHeader_2.54mm:PinHeader_1x02_P2.54mm_Vertical, F.Cu at (106.4, 132.1)
- added J4: Smeter, Connector_PinHeader_2.54mm:PinHeader_1x02_P2.54mm_Vertical, F.Cu at (265.2, 143.3)
- added J5: MICIN, Connector_PinHeader_2.54mm:PinHeader_1x02_P2.54mm_Vertical, F.Cu at (24.4, 111.8)
- added J6: PWR, Connector_PinHeader_2.54mm:PinHeader_1x03_P2.54mm_Vertical, F.Cu at (177.8, 16.8)
- added J7: uC PTT, Connector_PinHeader_2.54mm:PinHeader_1x02_P2.54mm_Vertical, F.Cu at (124.0, 26.7)
- added J8: ANT, Connector_Coaxial:SMA_Amphenol_901-144_Vertical, F.Cu at (36.8, 140.7)
- added J9: Fwd, Connector_PinHeader_2.54mm:PinHeader_1x02_P2.54mm_Vertical, F.Cu at (96.0, 153.2)
- added K3: G5V-2, Relay_THT:Relay_DPDT_Omron_G5V-2, F.Cu at (95.5, 29.7)
- added K4: G5V-2, Relay_THT:Relay_DPDT_Omron_G5V-2, F.Cu at (52.0, 149.3)
- added L3: 20u, Inductor_SMD:L_1206_3216Metric, F.Cu at (33.1, 108.7)
- added Q2: 2N3904, Package_TO_SOT_THT:TO-92_Inline, F.Cu at (50.1, 110.0)
- added Q3: 2N3904, Package_TO_SOT_THT:TO-92_Inline, F.Cu at (109.2, 32.0)
- added R22: 100R, Resistor_THT:R_Axial_DIN0207_L6.3mm_D2.5mm_P10.16mm_Horizontal, F.Cu at (266.2, 110.2)
- added R23: 10R, Resistor_THT:R_Axial_DIN0207_L6.3mm_D2.5mm_P10.16mm_Horizontal, F.Cu at (262.6, 140.2)
- added R24: 100R, Resistor_THT:R_Axial_DIN0207_L6.3mm_D2.5mm_P10.16mm_Horizontal, F.Cu at (34.5, 98.6)
- added R25: 10K, Resistor_THT:R_Axial_DIN0207_L6.3mm_D2.5mm_P10.16mm_Horizontal, F.Cu at (29.2, 94.0)
- added R26: 10K, Resistor_THT:R_Axial_DIN0207_L6.3mm_D2.5mm_P10.16mm_Horizontal, F.Cu at (38.9, 114.6)
- added R27: 220R, Resistor_THT:R_Axial_DIN0207_L6.3mm_D2.5mm_P10.16mm_Horizontal, F.Cu at (47.2, 103.4)
- added R28: 10K, Resistor_THT:R_Axial_DIN0207_L6.3mm_D2.5mm_P10.16mm_Horizontal, F.Cu at (47.5, 98.6)
- added R29: 10R, Resistor_THT:R_Axial_DIN0207_L6.3mm_D2.5mm_P10.16mm_Horizontal, F.Cu at (66.5, 118.6)
- added R30: 200R, Resistor_THT:R_Axial_DIN0207_L6.3mm_D2.5mm_P10.16mm_Horizontal, F.Cu at (182.1, 26.2)
- added R31: 200R, Resistor_THT:R_Axial_DIN0207_L6.3mm_D2.5mm_P10.16mm_Horizontal, F.Cu at (192.3, 26.7)
- added R32: 200R, Resistor_THT:R_Axial_DIN0207_L6.3mm_D2.5mm_P10.16mm_Horizontal, F.Cu at (187.2, 26.7)
- added R33: 100R, Resistor_THT:R_Axial_DIN0207_L6.3mm_D2.5mm_P10.16mm_Horizontal, F.Cu at (99.8, 21.3)
- added R34: 5K, Resistor_THT:R_Axial_DIN0207_L6.3mm_D2.5mm_P10.16mm_Horizontal, F.Cu at (114.3, 30.7)
- added R35: 100R, Resistor_THT:R_Axial_DIN0207_L6.3mm_D2.5mm_P10.16mm_Horizontal, F.Cu at (56.4, 153.4)
- added R36: 51R, Resistor_THT:R_Axial_DIN0207_L6.3mm_D2.5mm_P10.16mm_Horizontal, F.Cu at (81.5, 143.3)
- added R37: 51R, Resistor_THT:R_Axial_DIN0207_L6.3mm_D2.5mm_P10.16mm_Horizontal, F.Cu at (92.2, 138.7)
- added R38: 220R, Resistor_THT:R_Axial_DIN0207_L6.3mm_D2.5mm_P10.16mm_Horizontal, F.Cu at (89.4, 157.2)
- added R39: 220R, Resistor_THT:R_Axial_DIN0207_L6.3mm_D2.5mm_P10.16mm_Horizontal, F.Cu at (99.3, 138.9)
- added RV4: 10K, Potentiometer_THT:Potentiometer_Bourns_3296W_Vertical, F.Cu at (240.5, 123.4)
- added RV5: 10K, Potentiometer_THT:Potentiometer_Bourns_3296W_Vertical, F.Cu at (67.1, 109.5)
- added T4: FT37-43 (1:10), Transformer_THT:Transformer_Toroid_Horizontal_D14.0mm_Amidon-T50, F.Cu at (77.4, 162.2)
- added T5: FT37-43 (1:10), Transformer_THT:Transformer_Toroid_Horizontal_D14.0mm_Amidon-T50, F.Cu at (76.9, 141.1)
- added U6: LM386, Package_DIP:DIP-8_W7.62mm_Socket, F.Cu at (252.7, 118.1)
- added U7: LM7805, Package_TO_SOT_THT:TO-220-3_Vertical, F.Cu at (208.2, 21.5)
- added U8: LM7808, Package_TO_SOT_THT:TO-220-3_Vertical, F.Cu at (159.8, 25.1)
Connections:
- net +5V renamed RX5V
- net +8V renamed 8V
Routing:
- net GND: track 506.5 -> 0.00 mm
- net TX12V: track 115.1 -> 0.00 mm
- net 8V: track 87.3 -> 0.00 mm
- net RX5V: track 41.1 -> 0.00 mm
- net Net-(C38-Pad1): track 34.9 -> 0.00 mm
- net Net-(C23-Pad2): track 22.7 -> 0.00 mm
- net RX12V: track 21.6 -> 0.00 mm
- net IFRFIN: track 19.8 -> 0.00 mm
- net Net-(R8-Pad2): track 19.1 -> 0.00 mm
- net Net-(C2-Pad2): track 17.6 -> 0.00 mm
- net Net-(C28-Pad1): track 17.5 -> 0.00 mm
- net Net-(R5-Pad1): track 17.4 -> 0.00 mm
- net Net-(R5-Pad2): track 17.2 -> 0.00 mm
- net Net-(C34-Pad1): track 16.4 -> 0.00 mm
- net Net-(C27-Pad1): track 15.8 -> 0.00 mm
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Other:
- board size 236.4 x 120.1 mm -> 265.9 x 153.9 mm

Commit message: Update
Parts:
- removed the C54 at (153.3, 21.3)
- removed the C56 at (170.8, 23.1)
- removed the C58 at (165.1, 29.2)
- removed the R1 at (35.1, 77.9)
- added C4: 100n, Capacitor_THT:C_Disc_D3.4mm_W2.1mm_P2.50mm, F.Cu at (25.7, 40.7)
- added C55: 22u, Capacitor_THT:CP_Radial_D8.0mm_P2.50mm, F.Cu at (94.2, 113.3)
- added C57: 22u, Capacitor_THT:CP_Radial_D8.0mm_P2.50mm, F.Cu at (111.4, 113.3)
- added C59: 0.1u, Capacitor_THT:C_Disc_D3.0mm_W1.6mm_P2.50mm, F.Cu at (105.6, 107.2)
- added C64: 10n, Capacitor_THT:C_Disc_D3.4mm_W2.1mm_P2.50mm, F.Cu at (196.8, 81.3)
- added C65: 1u, Capacitor_THT:C_Disc_D3.4mm_W2.1mm_P2.50mm, F.Cu at (114.8, 160.1)
- added C66: 100n, Capacitor_THT:C_Disc_D3.4mm_W2.1mm_P2.50mm, F.Cu at (127.2, 150.4)
- added C67: 100n, Capacitor_THT:C_Disc_D3.4mm_W2.1mm_P2.50mm, F.Cu at (139.7, 141.7)
- added C68: 100n, Capacitor_THT:C_Disc_D3.4mm_W2.1mm_P2.50mm, F.Cu at (118.4, 160.3)
- added C69: 100n, Capacitor_THT:C_Disc_D3.4mm_W2.1mm_P2.50mm, F.Cu at (170.9, 160.4)
- added C70: 1u, Capacitor_THT:C_Disc_D3.4mm_W2.1mm_P2.50mm, F.Cu at (159.8, 147.1)
- added C71: 22u, Capacitor_THT:CP_Radial_D8.0mm_P2.50mm, F.Cu at (153.2, 146.3)
- added C72: 100n, Capacitor_THT:C_Disc_D3.4mm_W2.1mm_P2.50mm, F.Cu at (163.3, 147.1)
- added C73: 100n, Capacitor_THT:C_Disc_D3.4mm_W2.1mm_P2.50mm, F.Cu at (185.4, 108.6)
- added C74: 100n, Capacitor_THT:C_Disc_D3.4mm_W2.1mm_P2.50mm, F.Cu at (187.5, 138.6)
- added C75: 10u, Capacitor_THT:C_Disc_D3.4mm_W2.1mm_P2.50mm, F.Cu at (190.0, 108.6)
- added C76: 100n, Capacitor_THT:C_Disc_D3.4mm_W2.1mm_P2.50mm, F.Cu at (205.2, 127.0)
- added C77: 100n, Capacitor_THT:C_Disc_D3.4mm_W2.1mm_P2.50mm, F.Cu at (216.4, 149.0)
- added C78: 1u, Capacitor_THT:C_Disc_D3.4mm_W2.1mm_P2.50mm, F.Cu at (232.4, 104.5)
- added C79: 100n, Capacitor_THT:C_Disc_D3.4mm_W2.1mm_P2.50mm, F.Cu at (213.4, 139.3)
- added C80: 100n, Capacitor_THT:C_Disc_D3.4mm_W2.1mm_P2.50mm, F.Cu at (210.1, 119.5)
- added C81: .22u, Capacitor_THT:CP_Radial_D8.0mm_P2.50mm, F.Cu at (243.8, 121.4)
- added C82: 100u, Capacitor_THT:CP_Radial_D8.0mm_P2.50mm, F.Cu at (243.8, 108.7)
- added C83: 10u, Capacitor_THT:C_Disc_D3.4mm_W2.1mm_P2.50mm, F.Cu at (213.1, 119.8)
- added C84: 10u, Capacitor_THT:C_Disc_D3.4mm_W2.1mm_P2.50mm, F.Cu at (222.5, 118.0)
- added C85: 100n, Capacitor_THT:C_Disc_D3.4mm_W2.1mm_P2.50mm, F.Cu at (244.1, 127.6)
- added D12: 1N4733A, Diode_THT:D_DO-41_SOD81_P10.16mm_Horizontal, F.Cu at (218.4, 117.7)
- added J1: ANT_IN, Connector_Coaxial:SMA_Amphenol_901-144_Vertical, F.Cu at (37.8, 49.8)
- added J10: ANT_OUT, Connector_Coaxial:SMA_Amphenol_901-144_Vertical, F.Cu at (26.5, 186.3)
- added J12: PA_OUT, Connector_Coaxial:SMA_Amphenol_901-144_Vertical, F.Cu at (94.2, 152.9)
- added J15: Conn_01x01, TestPoint:TestPoint_Pad_2.0x2.0mm, F.Cu at (181.6, 136.7)
- added J16: Conn_01x01, TestPoint:TestPoint_Pad_2.0x2.0mm, F.Cu at (250.4, 136.1)
- added J17: Conn_01x01, TestPoint:TestPoint_Pad_2.0x2.0mm, F.Cu at (250.2, 171.7)
- added J18: Conn_01x01, TestPoint:TestPoint_Pad_2.0x2.0mm, F.Cu at (249.9, 99.3)
- added J19: Conn_01x01, TestPoint:TestPoint_Pad_2.0x2.0mm, F.Cu at (199.1, 99.1)
- added J20: Conn_01x01, TestPoint:TestPoint_Pad_2.0x2.0mm, F.Cu at (214.9, 98.8)
- added J21: Conn_01x01, TestPoint:TestPoint_Pad_2.0x2.0mm, F.Cu at (250.2, 116.6)
- added J22: Conn_01x01, TestPoint:TestPoint_Pad_2.0x2.0mm, F.Cu at (181.4, 171.2)
- added J23: Conn_01x01, TestPoint:TestPoint_Pad_2.0x2.0mm, F.Cu at (181.9, 154.9)
- added J24: Conn_01x01, TestPoint:TestPoint_Pad_2.0x2.0mm, F.Cu at (233.9, 98.8)
- added J25: Conn_01x01, TestPoint:TestPoint_Pad_2.0x2.0mm, F.Cu at (249.7, 155.4)
- added J26: Conn_01x01, TestPoint:TestPoint_Pad_2.0x2.0mm, F.Cu at (214.1, 171.7)
- added J27: Conn_01x01, TestPoint:TestPoint_Pad_2.0x2.0mm, F.Cu at (181.9, 117.1)
- added J28: Conn_01x01, TestPoint:TestPoint_Pad_2.0x2.0mm, F.Cu at (198.1, 171.7)
- added J29: Conn_01x01, TestPoint:TestPoint_Pad_2.0x2.0mm, F.Cu at (233.2, 171.7)
- added J30: Conn_01x01, TestPoint:TestPoint_Pad_2.0x2.0mm, F.Cu at (182.6, 99.1)
- added J31: ANT_OUT, Connector_Coaxial:SMA_Amphenol_901-144_Vertical, F.Cu at (202.4, 160.9)
- added J9: ANT_IN, Connector_Coaxial:SMA_Amphenol_901-144_Vertical, F.Cu at (26.7, 173.9)
- added L4: FT-37-43 (8T), Inductor_THT:L_Toroid_Horizontal_D9.5mm_P15.00mm_Diameter10-5mm_Amidon-T37, F.Cu at (198.1, 109.5)
- added L5: FT-37-43 (8T), Inductor_THT:L_Toroid_Horizontal_D9.5mm_P15.00mm_Diameter10-5mm_Amidon-T37, F.Cu at (233.2, 108.2)
- added Q4: 2N2219, Package_TO_SOT_THT:TO-39-3, F.Cu at (204.0, 140.1)
- added Q5: IRF510, Package_TO_SOT_THT:TO-220-3_Vertical, F.Cu at (246.7, 143.3)
- added R4: 51R, Resistor_THT:R_Axial_DIN0207_L6.3mm_D2.5mm_P10.16mm_Horizontal, F.Cu at (39.1, 40.6)
- added R40: 10K, Resistor_THT:R_Axial_DIN0207_L6.3mm_D2.5mm_P10.16mm_Horizontal, F.Cu at (121.4, 146.3)
- added R41: 10K, Resistor_THT:R_Axial_DIN0207_L6.3mm_D2.5mm_P10.16mm_Horizontal, F.Cu at (121.1, 160.0)
- added R42: 68R, Resistor_THT:R_Axial_DIN0207_L6.3mm_D2.5mm_P10.16mm_Horizontal, F.Cu at (129.5, 145.5)
- added R43: 51R, Resistor_THT:R_Axial_DIN0207_L6.3mm_D2.5mm_P10.16mm_Horizontal, F.Cu at (140.7, 156.5)
- added R44: 680R, Resistor_THT:R_Axial_DIN0207_L6.3mm_D2.5mm_P10.16mm_Horizontal, F.Cu at (143.8, 141.5)
- added R45: 200R, Resistor_THT:R_Axial_DIN0207_L6.3mm_D2.5mm_P10.16mm_Horizontal, F.Cu at (145.8, 163.3)
- added R46: 68R, Resistor_THT:R_Axial_DIN0207_L6.3mm_D2.5mm_P10.16mm_Horizontal, F.Cu at (160.8, 163.4)
- added R47: 680R, Resistor_THT:R_Axial_DIN0207_L6.3mm_D2.5mm_P10.16mm_Horizontal, F.Cu at (158.5, 153.8)
- added R48: 50R, Resistor_THT:R_Axial_DIN0207_L6.3mm_D2.5mm_P10.16mm_Horizontal, F.Cu at (158.5, 150.4)
- added R49: 680R, Resistor_THT:R_Axial_DIN0207_L6.3mm_D2.5mm_P10.16mm_Horizontal, F.Cu at (193.3, 138.3)
- added R50: 1K, Resistor_THT:R_Axial_DIN0207_L6.3mm_D2.5mm_P10.16mm_Horizontal, F.Cu at (189.5, 124.1)
- added R51: 2.2K, Resistor_THT:R_Axial_DIN0207_L6.3mm_D2.5mm_P10.16mm_Horizontal, F.Cu at (199.4, 129.7)
- added R52: 10R, Resistor_THT:R_Axial_DIN0207_L6.3mm_D2.5mm_P10.16mm_Horizontal, F.Cu at (211.3, 145.7)
- added R53: 202R, Resistor_THT:R_Axial_DIN0207_L6.3mm_D2.5mm_P10.16mm_Horizontal, F.Cu at (211.6, 150.2)
- added R54: 51R, Resistor_THT:R_Axial_DIN0207_L6.3mm_D2.5mm_P10.16mm_Horizontal, F.Cu at (219.2, 128.9)
- added R55: 1K, Resistor_THT:R_Axial_DIN0207_L6.3mm_D2.5mm_P10.16mm_Horizontal, F.Cu at (214.1, 106.0)
- added RV6: 10K, Potentiometer_THT:Potentiometer_Bourns_3296W_Vertical, F.Cu at (138.2, 150.4)
- added RV7: 10K, Potentiometer_THT:Potentiometer_Bourns_3296W_Vertical, F.Cu at (166.4, 158.6)
- added RV8: 10K, Potentiometer_THT:Potentiometer_Bourns_3296W_Vertical, F.Cu at (221.8, 122.8)
- added T6: FT50-74 (22:4), Transformer_THT:Transformer_Toroid_Horizontal_D14.0mm_Amidon-T50, F.Cu at (165.4, 114.4)
- added T7: FT3743(10BFT), Transformer_THT:Transformer_Toroid_Horizontal_D10.5mm_Amidon-T37, F.Cu at (227.4, 134.2)
- added U10: LT1253, Package_DIP:DIP-8_W7.62mm, F.Cu at (146.8, 151.4)
- added U11: QPR_Filter, Custom_RF:QRPLabs_Filter_TH, F.Cu at (233.9, 158.2)
- added U9: QPR_Filter, Custom_RF:QRPLabs_Filter_TH, F.Cu at (146.3, 119.3)
- C1: value 100n -> 1u
- U8: value LM7808 -> LM7805
- moved D5 157.0 mm to (44.6, 82.3), turned to 90 degrees
- moved R31 154.5 mm to (48.1, 82.3), turned to -90 degrees
- moved J7 143.1 mm to (44.3, 68.3), turned to 0 degrees
- moved D7 124.0 mm to (51.7, 79.7), turned to 90 degrees
- moved R32 121.0 mm to (84.4, 90.6)
- moved D6 116.2 mm to (88.8, 91.1)
- moved C56 114.3 mm to (107.1, 43.0), turned to -90 degrees
- moved R34 111.3 mm to (26.0, 98.5)
- moved J8 110.7 mm to (39.7, 98.5), turned to 90 degrees
- moved U8 106.2 mm to (100.3, 113.1)
- moved Q3 105.1 mm to (23.9, 93.5), turned to 0 degrees
- moved C58 103.2 mm to (112.3, 38.9), turned to 90 degrees
- moved U7 102.3 mm to (106.4, 32.0), turned to -90 degrees
- moved C54 101.9 mm to (100.6, 26.8), turned to -90 degrees
- moved C46 98.8 mm to (256.1, 48.7), turned to -90 degrees
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- renumbered C9 to C10, C10 to C11, C11 to C12, C12 to C13, C13 to C14, C14 to C15, C15 to C16, C16 to C17, C17 to C18, C18 to C19, C19 to C20, C20 to C21, C21 to C22, C22 to C23, C23 to C24, C24 to C25, C25 to C26, C26 to C27, C27 to C28, C28 to C29, C29 to C30, C30 to C31, C31 to C32, C32 to C33, C33 to C34, C34 to C35, C35 to C36, C36 to C37, C37 to C38, C38 to C39, C39 to C40, C40 to C41, C41 to C42, C42 to C43, C43 to C44, C44 to C45, C45 to C46, C46 to C47, C47 to C48, C48 to C49, C4 to C5, C49 to C50, C50 to C51, C51 to C52, C52 to C53, C53 to C54, C55 to C56, C57 to C58, C5 to C6, C59 to C60, C60 to C61, C61 to C62, C62 to C63, C6 to C7, C7 to C8, C8 to C9, J8 to J11, J9 to J13, J10 to J14, J1 to J2, J2 to J3, J3 to J4, J4 to J5, J5 to J6, J6 to J7, J7 to J8, R2 to R1, R3 to R2, R4 to R3
Connections:
- C2 pad 1: ANT_IN -> Net-(C2-Pad1)
- C54 pad 1: TX12V -> RX12V
- K1 pad 6: unconnected-(K1-Pad6) -> IFRFIN
- K1 pad 9: unconnected-(K1-Pad9) -> IFMICIN
- K2 pad 6: unconnected-(K2-Pad6) -> IFAFOUT
- K2 pad 9: unconnected-(K2-Pad9) -> IFPAOUT
- K3 pad 6: unconnected-(K3-Pad6) -> RX12V
- K3 pad 9: unconnected-(K3-Pad9) -> TX12V
- K4 pad 11: ANT_IN -> Net-(J9-Pad1)
- K4 pad 6: unconnected-(K4-Pad6) -> Net-(J9-Pad1)
- K4 pad 8: ANT_OUT -> Net-(J10-Pad1)
- K4 pad 9: unconnected-(K4-Pad9) -> Net-(J10-Pad1)
- L1 pad 1: 8V -> RX5V
- L2 pad 1: 8V -> RX5V
- R1 pad 2: Net-(C2-Pad2) -> Net-(C1-Pad1)
- R2 pad 1: Net-(C2-Pad2) -> Net-(C1-Pad1)
- U7 pad 1: TX12V -> RX12V
- U8 pad 1: 12V -> TX12V
- U8 pad 3: 8V -> TX5V
Routing:
- net RX12V: track 0.00 -> 347.3 mm
- net TX12V: track 0.00 -> 345.4 mm
- net RX5V: track 0.00 -> 141.4 mm
- net TX5V: track 0.00 -> 118.6 mm
- net Net-(RV3-Pad2): track 0.00 -> 68.5 mm
- net Net-(C64-Pad2): track 0.00 -> 54.8 mm
- net Net-(D11-Pad2): track 0.00 -> 39.4 mm
- net Net-(C47-Pad1): track 0.00 -> 33.9 mm
- net Net-(C41-Pad2): track 0.00 -> 33.3 mm
- net Net-(C66-Pad1): track 0.00 -> 29.9 mm
- net Net-(C39-Pad1): track 0.00 -> 26.7 mm
- net IFRFIN: track 0.00 -> 26.4 mm
- net Net-(T1-Pad4): track 0.00 -> 26.2 mm
- net Net-(C81-Pad1): track 0.00 -> 25.4 mm
- net Net-(C30-Pad2): track 0.00 -> 24.8 mm
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Other:
- board size 265.9 x 153.9 mm -> 246.9 x 181.9 mm
