File: Smeter.kicad_sch (KiCad schematic)
At the start: 12 parts, among them J4 Smeter, U6 LM386

Commit message: Update
Parts:
- renumbered C40 to C41, C41 to C42, C42 to C43, C43 to C44, C44 to C45, C45 to C46, J4 to J5
Changed lines of the file:
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@@
   (symbol (lib_id "power:GND") (at 154.94 92.075 0) (unit 1)
     (in_bom yes) (on_board yes)
-    (property "Reference" "#PWR031" (id 0) (at 154.94 98.425 0)
+    (property "Reference" "#PWR033" (id 0) (at 154.94 98.425 0)
       (effects (font (size 1.27 1.27)) hide)
     )
@@
   (symbol (lib_id "power:GND") (at 146.685 74.93 0) (unit 1)
     (in_bom yes) (on_board yes)
-    (property "Reference" "#PWR029" (id 0) (at 146.685 81.28 0)
+    (property "Reference" "#PWR031" (id 0) (at 146.685 81.28 0)
       (effects (font (size 1.27 1.27)) hide)
     )
@@
   (symbol (lib_id "Device:C") (at 201.295 97.155 0) (unit 1)
     (in_bom yes) (on_board yes) (fields_autoplaced)
-    (property "Reference" "C45" (id 0) (at 204.47 95.8849 0)
+    (property "Reference" "C46" (id 0) (at 204.47 95.8849 0)
       (effects (font (size 1.27 1.27)) (justify left))
     )
@@
   (symbol (lib_id "power:GND") (at 155.575 74.93 0) (unit 1)
     (in_bom yes) (on_board yes)
-    (property "Reference" "#PWR032" (id 0) (at 155.575 81.28 0)
+    (property "Reference" "#PWR034" (id 0) (at 155.575 81.28 0)
       (effects (font (size 1.27 1.27)) hide)
     )
@@
   (symbol (lib_id "Device:C_Polarized") (at 168.91 104.14 90) (unit 1)
     (in_bom yes) (on_board yes)
-    (property "Reference" "C43" (id 0) (at 166.37 101.6 0)
+    (property "Reference" "C44" (id 0) (at 166.37 101.6 0)
       (effects (font (size 1.27 1.27)) (justify left))
     )
@@
   (symbol (lib_id "power:GND") (at 162.56 103.505 0) (unit 1)
     (in_bom yes) (on_board yes)
-    (property "Reference" "#PWR033" (id 0) (at 162.56 109.855 0)
+    (property "Reference" "#PWR035" (id 0) (at 162.56 109.855 0)
       (effects (font (size 1.27 1.27)) hide)
     )
@@
   (symbol (lib_id "power:GND") (at 148.59 113.665 0) (unit 1)
     (in_bom yes) (on_board yes)
-    (property "Reference" "#PWR030" (id 0) (at 148.59 120.015 0)
+    (property "Reference" "#PWR032" (id 0) (at 148.59 120.015 0)
       (effects (font (size 1.27 1.27)) hide)
     )
@@
   (symbol (lib_id "power:GND") (at 184.15 104.775 0) (unit 1)
     (in_bom yes) (on_board yes) (fields_autoplaced)
-    (property "Reference" "#PWR034" (id 0) (at 184.15 111.125 0)
+    (property "Reference" "#PWR036" (id 0) (at 184.15 111.125 0)
       (effects (font (size 1.27 1.27)) hide)
     )
@@
   (symbol (lib_id "Device:C") (at 135.89 94.615 90) (unit 1)
     (in_bom yes) (on_board yes) (fields_autoplaced)
-    (property "Reference" "C40" (id 0) (at 135.89 87.63 90))
+    (property "Reference" "C41" (id 0) (at 135.89 87.63 90))
     (property "Value" "10u" (id 1) (at 135.89 90.17 90))
     (property "Footprint" "Capacitor_THT:C_Disc_D3.4mm_W2.1mm_P2.50mm" (id 2) (at 139.7 93.6498 0)
@@
   (symbol (lib_id "Connector_Generic:Conn_01x02") (at 215.265 92.075 0) (unit 1)
     (in_bom yes) (on_board yes) (fields_autoplaced)
-    (property "Reference" "J4" (id 0) (at 218.44 92.0749 0)
+    (property "Reference" "J5" (id 0) (at 218.44 92.0749 0)
       (effects (font (size 1.27 1.27)) (justify left))
     )
@@
   (symbol (lib_id "power:GND") (at 210.185 98.425 0) (unit 1)
     (in_bom yes) (on_board yes)
-    (property "Reference" "#PWR036" (id 0) (at 210.185 104.775 0)
+    (property "Reference" "#PWR038" (id 0) (at 210.185 104.775 0)
       (effects (font (size 1.27 1.27)) hide)
     )
@@
   (symbol (lib_id "Device:C") (at 155.575 71.12 0) (unit 1)
     (in_bom yes) (on_board yes)
-    (property "Reference" "C42" (id 0) (at 156.845 68.58 0)
+    (property "Reference" "C43" (id 0) (at 156.845 68.58 0)
       (effects (font (size 1.27 1.27)) (justify left))
     )
@@
   (symbol (lib_id "power:GND") (at 201.295 104.14 0) (unit 1)
     (in_bom yes) (on_board yes) (fields_autoplaced)
-    (property "Reference" "#PWR035" (id 0) (at 201.295 110.49 0)
+    (property "Reference" "#PWR037" (id 0) (at 201.295 110.49 0)
       (effects (font (size 1.27 1.27)) hide)
     )
@@
   (symbol (lib_id "Device:C_Polarized") (at 179.705 92.075 90) (unit 1)
     (in_bom yes) (on_board yes)
-    (property "Reference" "C44" (id 0) (at 177.165 89.535 0)
+    (property "Reference" "C45" (id 0) (at 177.165 89.535 0)
       (effects (font (size 1.27 1.27)) (justify left))
     )
@@
   (symbol (lib_id "Device:C") (at 146.685 71.12 0) (unit 1)
     (in_bom yes) (on_board yes)
-    (property "Reference" "C41" (id 0) (at 147.955 68.58 0)
-      (effects (font (size 1.27 1.27)) (justify left))
-    )
+    (property "Reference" "C42" (id 0) (at 147.955 68.58 0)
+      (effects (font (size 1.27 1.27)) (justify left))
+    )
