File: Phoenix612 Complete/Version 1/AF_amp.kicad_sch (KiCad schematic)
At the start: 29 parts, among them J10 SPK, J9 TP, U5 NE5532, U7 LM380N

Commit message: Upload 21Mar23
Parts:
- added L4: 20u, Inductor_SMD:L_1206_3216Metric, symbol Device:L
- C37: renamed from C34; value 68nf -> 68n
- renumbered C31 to C34, C32 to C35, C33 to C36, C35 to C38, C36 to C39, C37 to C40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
Connections:
- net RX12V: now also L4.1; no longer R25.1
- new net: L4.2, R25.1
