File: Phoenix612 Complete/Version 1/AntSwitch.kicad_sch (KiCad schematic)
At the start: 21 parts, among them J15 ANT_IN, J16 ANT, J17 ANT_OUT, J18 Fwd, J19 Rev, J44 PA_OUT, J45 ANT_OUT, K4 G5V-2, T3 FT37-43 (1:10), T4 FT37-43 (1:10)

Commit message: Upload 21Mar23
Parts:
- removed J15: ANT_IN, Connector_Coaxial:SMA_Amphenol_901-144_Vertical, symbol Connector:Conn_Coaxial
- removed J17, J45: ANT_OUT, Connector_Coaxial:SMA_Amphenol_901-144_Vertical, symbol Connector:Conn_Coaxial
- removed J44: PA_OUT, Connector_Coaxial:SMA_Amphenol_901-144_Vertical, symbol Connector:Conn_Coaxial
- added J35, J36, J37, J38, J39, J40, J41, J42, J43, J44, J45, J46: SHD, TestPoint:TestPoint_Pad_2.0x2.0mm, symbol Connector_Generic:Conn_01x01
- renumbered C70 to C84, C71 to C85, C72 to C86, J16 to J32, J18 to J33, J19 to J34, R50 to R59, R51 to R60, R52 to R61, R53 to R62, R54 to R63, T3 to T5, T4 to T6
Connections:
- net ANT_OUT: now also K4.8, K4.9
- net GND: now also J35.1 (Pin_1), J36.1 (Pin_1), J37.1 (Pin_1), J38.1 (Pin_1), J39.1 (Pin_1), J40.1 (Pin_1), J41.1 (Pin_1), J42.1 (Pin_1), J43.1 (Pin_1), J44.1 (Pin_1), J45.1 (Pin_1), J46.1 (Pin_1)
- net ANT_IN: now reaches K4.11, K4.6
