File: Phoenix612 Complete/Version 1/IF_Stage.kicad_sch (KiCad schematic)
At the start: 52 parts, among them J3 TP, J4 VFO, J5 TP, J6 TP, J7 BFO, J8 TP, K1 G5V-2, K2 G5V-2, T1 FT50-75 (18:7), T2 FT50-75 (7:18), U3 SA612, U4 SA612, Y1 12 MHz, Y2 12 MHz, Y3 12 MHz, Y4 12 MHz

Commit message: Upload 21Mar23
Parts:
- removed C29: 47u, Capacitor_THT:CP_Radial_D8.0mm_P2.50mm, symbol Device:C_Polarized
- removed C30: 100n, Capacitor_SMD:C_1206_3216Metric, symbol Device:C
- added J7: TP, Connector_PinHeader_1.00mm:PinHeader_1x01_P1.00mm_Vertical, symbol Connector_Generic:Conn_01x01
- C25: renamed from C20; footprint Capacitor_SMD:C_1206_3216Metric -> Capacitor_THT:C_Disc_D4.7mm_W2.5mm_P5.00mm
- C26: renamed from C21; footprint Capacitor_SMD:C_1206_3216Metric -> Capacitor_THT:C_Disc_D4.7mm_W2.5mm_P5.00mm
- C27: renamed from C22; footprint Capacitor_SMD:C_1206_3216Metric -> Capacitor_THT:C_Disc_D4.7mm_W2.5mm_P5.00mm
- renumbered C9 to C14, C10 to C15, C11 to C16, C12 to C17, c13 to C18, C14 to C19, C15 to C20, C16 to C21, C17 to C22, C18 to C23, C19 to C24, C23 to C28, C24 to C29, C25 to C30, C26 to C31, C27 to C32, C28 to C33, D1 to D6, D2 to D7, J8 to J10, J3 to J4, J4 to J5, J5 to J6, J6 to J8, J7 to J9, K1 to K2, K2 to K3, R10 to R15, R11 to R16, R12 to R17, R13 to R18, R14 to R19, R15 to R20, R16 to R21, R17 to R22, R18 to R23, R19 to R24, U3 to U4, U4 to U5
Connections:
- net IFAFOUT: now also K3.11, K3.6
- net IFPAOUT: now also K3.8, K3.9
- net at C31.2, U5.6 (OSC_B): now also J7.1 (Pin_1)
- net RX5V renamed 5V
Other:
- note removed: "Can also be 5V for Less gain"
