File: Phoenix612 Complete/Version 1/MicPreamp.kicad_sch (KiCad schematic)
At the start: 18 parts, among them J12 MICIN, Q1 2N3904

Commit message: Upload 21Mar23
Parts:
- renumbered C56 to C47, C57 to C48, C58 to C49, C59 to C50, C60 to C51, C61 to C52, C62 to C53, J12 to J13, L8 to L7, L9 to L8, Q1 to Q2, R39 to R34, R40 to R35, R41 to R36, R42 to R37, R43 to R38, R44 to R39, RV5 to RV4
Changed lines of the file:
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@@
   (symbol (lib_id "Connector_Generic:Conn_01x02") (at 62.23 104.775 180) (unit 1)
     (in_bom yes) (on_board yes) (fields_autoplaced)
-    (property "Reference" "J12" (id 0) (at 62.23 95.25 0))
+    (property "Reference" "J13" (id 0) (at 62.23 95.25 0))
     (property "Value" "MICIN" (id 1) (at 62.23 97.79 0))
     (property "Footprint" "Connector_PinHeader_2.54mm:PinHeader_1x02_P2.54mm_Vertical" (id 2) (at 62.23 104.775 0)
@@
   (symbol (lib_id "power:GND") (at 67.31 107.315 0) (unit 1)
     (in_bom yes) (on_board yes)
-    (property "Reference" "#PWR051" (id 0) (at 67.31 113.665 0)
+    (property "Reference" "#PWR046" (id 0) (at 67.31 113.665 0)
       (effects (font (size 1.27 1.27)) hide)
     )
@@
   (symbol (lib_id "Device:C") (at 75.565 108.585 0) (unit 1)
     (in_bom yes) (on_board yes)
-    (property "Reference" "C62" (id 0) (at 76.835 111.125 90))
+    (property "Reference" "C53" (id 0) (at 76.835 111.125 90))
     (property "Value" "10n" (id 1) (at 73.66 111.76 90))
     (property "Footprint" "Capacitor_SMD:C_1206_3216Metric" (id 2) (at 76.5302 112.395 0)
@@
   (symbol (lib_id "Device:R_US") (at 90.17 108.585 0) (unit 1)
     (in_bom yes) (on_board yes) (fields_autoplaced)
-    (property "Reference" "R44" (id 0) (at 92.71 107.3149 0)
+    (property "Reference" "R39" (id 0) (at 92.71 107.3149 0)
       (effects (font (size 1.27 1.27)) (justify left))
     )
@@
   (symbol (lib_id "power:GND") (at 76.2 83.185 0) (unit 1)
     (in_bom yes) (on_board yes)
-    (property "Reference" "#PWR049" (id 0) (at 76.2 89.535 0)
+    (property "Reference" "#PWR044" (id 0) (at 76.2 89.535 0)
       (effects (font (size 1.27 1.27)) hide)
     )
@@
   (symbol (lib_id "Device:C") (at 150.495 97.155 0) (unit 1)
     (in_bom yes) (on_board yes) (fields_autoplaced)
-    (property "Reference" "C60" (id 0) (at 153.67 95.8849 0)
+    (property "Reference" "C51" (id 0) (at 153.67 95.8849 0)
       (effects (font (size 1.27 1.27)) (justify left))
     )
@@
   (symbol (lib_id "Device:R_US") (at 109.22 95.885 90) (unit 1)
     (in_bom yes) (on_board yes) (fields_autoplaced)
-    (property "Reference" "R42" (id 0) (at 109.22 90.17 90))
+    (property "Reference" "R37" (id 0) (at 109.22 90.17 90))
     (property "Value" "220" (id 1) (at 109.22 92.71 90))
     (property "Footprint" "Resistor_SMD:R_1206_3216Metric" (id 2) (at 109.474 94.869 90)
@@
   (symbol (lib_id "power:GND") (at 90.17 114.935 0) (unit 1)
     (in_bom yes) (on_board yes)
-    (property "Reference" "#PWR054" (id 0) (at 90.17 121.285 0)
+    (property "Reference" "#PWR049" (id 0) (at 90.17 121.285 0)
       (effects (font (size 1.27 1.27)) hide)
     )
@@
   (symbol (lib_id "Device:R_US") (at 90.17 66.04 0) (unit 1)
     (in_bom yes) (on_board yes) (fields_autoplaced)
-    (property "Reference" "R39" (id 0) (at 92.71 64.7699 0)
+    (property "Reference" "R34" (id 0) (at 92.71 64.7699 0)
       (effects (font (size 1.27 1.27)) (justify left))
     )
@@
   (symbol (lib_id "Device:C_Polarized") (at 96.52 102.235 90) (unit 1)
     (in_bom yes) (on_board yes)
-    (property "Reference" "C61" (id 0) (at 93.98 99.695 0)
+    (property "Reference" "C52" (id 0) (at 93.98 99.695 0)
       (effects (font (size 1.27 1.27)) (justify left))
     )
@@
   (symbol (lib_id "Device:L") (at 90.17 54.61 0) (unit 1)
     (in_bom yes) (on_board yes) (fields_autoplaced)
-    (property "Reference" "L8" (id 0) (at 91.44 53.3399 0)
+    (property "Reference" "L7" (id 0) (at 91.44 53.3399 0)
       (effects (font (size 1.27 1.27)) (justify left))
     )
@@
   (symbol (lib_id "Device:R_US") (at 150.495 106.68 180) (unit 1)
     (in_bom yes) (on_board yes) (fields_autoplaced)
-    (property "Reference" "R43" (id 0) (at 152.4 105.4099 0)
+    (property "Reference" "R38" (id 0) (at 152.4 105.4099 0)
       (effects (font (size 1.27 1.27)) (justify right))
     )
@@
   (symbol (lib_id "Device:R_US") (at 113.03 81.28 0) (unit 1)
     (in_bom yes) (on_board yes) (fields_autoplaced)
-    (property "Reference" "R41" (id 0) (at 114.935 80.0099 0)
+    (property "Reference" "R36" (id 0) (at 114.935 80.0099 0)
       (effects (font (size 1.27 1.27)) (justify left))
     )
@@
   (symbol (lib_id "power:GND") (at 142.24 99.06 0) (unit 1)
     (in_bom yes) (on_board yes)
-    (property "Reference" "#PWR050" (id 0) (at 142.24 105.41 0)
+    (property "Reference" "#PWR045" (id 0) (at 142.24 105.41 0)
       (effects (font (size 1.27 1.27)) hide)
     )
@@
   (symbol (lib_id "power:PWR_FLAG") (at 76.2 69.215 0) (unit 1)
     (in_bom yes) (on_board yes)
-    (property "Reference" "#FLG05" (id 0) (at 76.2 67.31 0)
+    (property "Reference" "#FLG010" (id 0) (at 76.2 67.31 0)
       (effects (font (size 1.27 1.27)) hide)
     )
@@
   (symbol (lib_id "Device:C_Polarized") (at 82.55 76.835 0) (unit 1)
     (in_bom yes) (on_board yes)
-    (property "Reference" "C58" (id 0) (at 85.09 74.295 0)
+    (property "Reference" "C49" (id 0) (at 85.09 74.295 0)
       (effects (font (size 1.27 1.27)) (justify left))
     )
@@
   (symbol (lib_id "Transistor_BJT:2N3904") (at 110.49 102.235 0) (unit 1)
     (in_bom yes) (on_board yes) (fields_autoplaced)
-    (property "Reference" "Q1" (id 0) (at 115.57 100.9649 0)
+    (property "Reference" "Q2" (id 0) (at 115.57 100.9649 0)
       (effects (font (size 1.27 1.27)) (justify left))
     )
@@
   (symbol (lib_id "power:GND") (at 150.495 112.395 0) (unit 1)
     (in_bom yes) (on_board yes) (fields_autoplaced)
-    (property "Reference" "#PWR053" (id 0) (at 150.495 118.745 0)
+    (property "Reference" "#PWR048" (id 0) (at 150.495 118.745 0)
       (effects (font (size 1.27 1.27)) hide)
     )
@@
   (symbol (lib_id "power:GND") (at 113.03 111.125 0) (unit 1)
     (in_bom yes) (on_board yes)
-    (property "Reference" "#PWR052" (id 0) (at 113.03 117.475 0)
+    (property "Reference" "#PWR047" (id 0) (at 113.03 117.475 0)
       (effects (font (size 1.27 1.27)) hide)
     )
@@
   (symbol (lib_id "Device:R_US") (at 90.17 80.645 0) (unit 1)
     (in_bom yes) (on_board yes) (fields_autoplaced)
-    (property "Reference" "R40" (id 0) (at 92.075 79.3749 0)
+    (property "Reference" "R35" (id 0) (at 92.075 79.3749 0)
       (effects (font (size 1.27 1.27)) (justify left))
     )
@@
   (symbol (lib_id "Device:C") (at 69.85 76.835 0) (unit 1)
     (in_bom yes) (on_board yes)
-    (property "Reference" "C56" (id 0) (at 71.12 74.295 0)
+    (property "Reference" "C47" (id 0) (at 71.12 74.295 0)
       (effects (font (size 1.27 1.27)) (justify left))
     )
@@
   (symbol (lib_id "power:GND") (at 75.565 115.57 0) (unit 1)
     (in_bom yes) (on_board yes)
-    (property "Reference" "#PWR055" (id 0) (at 75.565 121.92 0)
+    (property "Reference" "#PWR050" (id 0) (at 75.565 121.92 0)
       (effects (font (size 1.27 1.27)) hide)
     )
@@
   (symbol (lib_id "Device:C") (at 76.2 76.835 0) (unit 1)
     (in_bom yes) (on_board yes)
-    (property "Reference" "C57" (id 0) (at 77.47 74.295 0)
+    (property "Reference" "C48" (id 0) (at 77.47 74.295 0)
       (effects (font (size 1.27 1.27)) (justify left))
     )
@@
   (symbol (lib_id "Device:R_Potentiometer_Trim") (at 134.62 95.885 90) (unit 1)
     (in_bom yes) (on_board yes) (fields_autoplaced)
-    (property "Reference" "RV5" (id 0) (at 134.62 99.06 90))
+    (property "Reference" "RV4" (id 0) (at 134.62 99.06 90))
     (property "Value" "10K" (id 1) (at 134.62 101.6 90))
     (property "Footprint" "Potentiometer_THT:Potentiometer_Bourns_3296W_Vertical" (id 2) (at 134.62 95.885 0)
@@
   (symbol (lib_id "Device:L") (at 83.185 102.235 90) (unit 1)
     (in_bom yes) (on_board yes)
-    (property "Reference" "L9" (id 0) (at 83.185 99.695 90))
+    (property "Reference" "L8" (id 0) (at 83.185 99.695 90))
     (property "Value" "20u" (id 1) (at 83.185 104.14 90))
     (property "Footprint" "Inductor_SMD:L_1206_3216Metric" (id 2) (at 83.185 102.235 0)
@@
   (symbol (lib_id "Device:C_Polarized") (at 124.46 95.885 90) (unit 1)
     (in_bom yes) (on_board yes)
-    (property "Reference" "C59" (id 0) (at 121.92 93.345 0)
-      (effects (font (size 1.27 1.27)) (justify left))
-    )
+    (property "Reference" "C50" (id 0) (at 121.92 93.345 0)
+      (effects (font (size 1.27 1.27)) (justify left))
+    )
