File: Phoenix612 Complete/Version 1/PA_Driver.kicad_sch (KiCad schematic)
At the start: 24 parts, among them J41 TP, J42 TP, J43 RF_IN, U14 OPA2674I-14

Commit message: Upload 21Mar23
Parts:
- removed J43: RF_IN, Connector_Coaxial:SMA_Amphenol_901-144_Vertical, symbol Connector:Conn_Coaxial
- U10: renamed from U14; value OPA2674I-14 -> OPA2674
- renumbered C94 to C62, C95 to C63, C96 to C64, C97 to C65, C98 to C66, C99 to C67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
Connections:
- net PA_DRIVER_IN: now reaches C63.1
