File: Phoenix612 Complete/Version 1/PA_Preamp.kicad_sch (KiCad schematic)
At the start: 21 parts, among them J20 TP, J21 TP, T5 FT50-74 (22:4), U11 LT1253, U12 QPR_Filter

Commit message: Upload 21Mar23
Parts:
- removed T5: FT50-74 (22:4), Transformer_THT:Transformer_Toroid_Horizontal_D14.0mm_Amidon-T50, symbol Device:Transformer_1P_1S
- removed U11: LT1253, Package_DIP:DIP-8_W7.62mm, symbol Custom_RF:LT1253
- added TR2: T50-22:4, Custom_RF:T50-1Tap-Close, symbol Custom_RF:T50
- added U8: LT1253, Package_DIP:DIP-8_W7.62mm, symbol Custom_RF:LT1253
- C58: renamed from C77; value 1u -> 10n; footprint Capacitor_THT:C_Disc_D3.4mm_W2.1mm_P2.50mm -> Capacitor_SMD:C_1206_3216Metric
- renumbered C73 to C54, C74 to C55, C75 to C56, C76 to C57, C78 to C59, C79 to C60, C80 to C61, J20 to J14, J21 to J15, L10 to L9, R55 to R40, R56 to R41, R57 to R42, R58 to R43, R59 to R44, R60 to R45, RV6 to RV5, U12 to U9
Connections:
- net GND: now also TR2.3, U8.4 (V-)
- net at R44.1, RV5.1: now also U8.2 (InA-)
- net at R43.1, R44.2: now also U8.1 (OutA)
- net at U9.1 (IN), U9.2 (IN): now also TR2.2
- net at C54.1, C55.1, C56.1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: now also U8.8 (V+)
- net at C60.2, R42.1: now also U8.3 (InA+)
- net at C59.2: now also TR2.1
- net PA_IN renamed PA_DRIVER_IN
- no-connect marks 0 -> 3
Other:
- moved on the sheet: C59
