File: Phoenix612 Complete/Version 1/Phoenix612 Complete v1.kicad_sch (KiCad schematic)
At the start: 0 parts

Commit message: Upload 21Mar23
Other:
- removed sheet AF Amp
- removed sheet Ant Switch Sheet
- removed sheet IF Mixer and Filter
- removed sheet MicPreamp Sheet
- removed sheet PA Preamp
- removed sheet Power Amp
- removed sheet Power Supply Sheet
- removed sheet Smeter Sheet
- added sheet AF_Amp (AF_Amp.kicad_sch)
- added sheet AntSwitch (AntSwitch.kicad_sch)
- added sheet IF_Stage (IF_Stage.kicad_sch)
- added sheet MicPreamp (MicPreamp.kicad_sch)
- added sheet PA_Preamp (PA_Preamp.kicad_sch)
- added sheet Power Supply (PowerSupply.kicad_sch)
- added sheet PowerAmp (PowerAmp.kicad_sch)
