File: Phoenix612 Complete/Version 1/PowerAmp.kicad_sch (KiCad schematic)
At the start: 44 parts, among them J22 TP, J23 TP, J24 JMP, J25 SHD, J26 SHD, J27 SHD, J28 SHD, J29 SHD, J30 SHD, J31 SHD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

Commit message: Upload 21Mar23
Parts:
- removed J28, J31, J34, J36, J39: SHD, TestPoint:TestPoint_Pad_2.0x2.0mm, symbol Connector_Generic:Conn_01x01
- removed J46: PA_OUT, Connector_Coaxial:SMA_Amphenol_901-144_Vertical, symbol Connector:Conn_Coaxial
- R55: renamed from R61; value 220 -> 680
- renumbered C81 to C71, C82 to C72, C83 to C73, C84 to C74, C85 to C75, C86 to C76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
