File: Phoenix612 Complete/Version 1/PowerSupply.kicad_sch (KiCad schematic)
At the start: 23 parts, among them J13 PWR, J14 uC PTT, K3 G5V-2, Q2 2N3904, U10 LM7805, U9 LM7805

Commit message: Upload 21Mar23
Parts:
- removed C67, C68: 22u, Capacitor_THT:CP_Radial_D8.0mm_P2.50mm, symbol Device:C_Polarized
- removed C69: 0.1u, Capacitor_SMD:C_1206_3216Metric, symbol Device:C
- removed U10: LM7805, Package_TO_SOT_THT:TO-220-3_Vertical, symbol Regulator_Linear:LM7805_TO220
- added C13: 10n, Capacitor_SMD:C_1206_3216Metric, symbol Device:C
- C11: renamed from C65; value 0.1u -> 100n
- D2: renamed from D5; value LED -> RX
- D3: renamed from D6; value LED -> PWR
- D4: renamed from D7; value LED -> TX
- renumbered C64 to C10, C66 to C12, C63 to C9, D4 to D1, D8 to D5, J13 to J2, J14 to J3, K3 to K1, Q2 to Q1, R45 to R10, R46 to R11, R47 to R12, R48 to R13, R49 to R14, U9 to U3
Connections:
- net GND: now also C13.1
- net at J3.1 (Pin_1), R14.2: now also C13.2
