File: Phoenix612 Complete/Version 1/RF_amp.kicad_sch (KiCad schematic)
At the start: 24 parts, among them J1 TP, J2 ANT_IN, U1 LT1253, U2 QPR_Filter

Commit message: Upload 21Mar23
Parts:
- removed J2: ANT_IN, Connector_Coaxial:SMA_Amphenol_901-144_Vertical, symbol Connector:Conn_Coaxial
- added C87: 100n, Capacitor_SMD:C_1206_3216Metric, symbol Device:C
- added L14: 20u, Inductor_SMD:L_1206_3216Metric, symbol Device:L
- added R64: 200R, Resistor_SMD:R_1206_3216Metric, symbol Device:R_US
- added TR1: T50-22:4, Custom_RF:T50-1Tap-Close, symbol Custom_RF:T50
Connections:
- net GND: now also TR1.1
- net IFRFIN: now also TR1.3; no longer U2.7 (OUT), U2.8 (OUT)
- net RX12V: now also L14.1; no longer R1.1
- net at C6.2, R3.1: now also R64.1; no longer U1.3 (InA+)
- net ANT_IN: now reaches C6.1
- net at U2.1 (IN), U2.2 (IN): now also C87.2; no longer R5.2
- new net: C87.1, R5.2
- new net: R64.2, U1.3 (InA+)
- new net: TR1.2, U2.7 (OUT), U2.8 (OUT)
- new net: L14.2, R1.1
Other:
- moved on the sheet: C6, R5
