File: Phoenix612 Complete/Version 1.1/AntSwitch.kicad_sch (KiCad schematic)
At the start: 29 parts, among them J32 ANT, J33 Fwd, J34 Rev, J35 SHD, J36 SHD, J37 SHD, J38 SHD, J39 SHD, J40 SHD, J41 SHD, J42 SHD, J43 SHD, J44 SHD, J45 SHD, J46 SHD, K4 G5V-2, T4 FT37-43 (1:10), T5 FT37-43 (1:10)

Commit message: Update 9Mar23
Connections:
- net ANT_OUT: now also T5.2 (AB); no longer T4.4 (SB), T5.1 (AA)
- net PA_OUT: now also T4.4 (SB), T5.1 (AA); no longer T5.2 (AB)
Changed lines of the file:
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@@
     (effects (font (size 1.27 1.27)) (justify left bottom))
   )
-  (global_label "PA_OUT" (shape output) (at 181.61 54.61 180) (fields_autoplaced)
+  (global_label "ANT_OUT" (shape output) (at 181.61 54.61 180) (fields_autoplaced)
     (effects (font (size 1.27 1.27)) (justify right))
-    (property "Intersheet References" "${INTERSHEET_REFS}" (id 0) (at 172.2421 54.5306 0)
+    (property "Intersheet References" "${INTERSHEET_REFS}" (id 0) (at 171.214 54.6894 0)
       (effects (font (size 1.27 1.27)) (justify right) hide)
     )
@@
     )
   )
-  (global_label "ANT_OUT" (shape output) (at 207.01 55.88 90) (fields_autoplaced)
-    (effects (font (size 1.27 1.27)) (justify left))
-    (property "Intersheet References" "${INTERSHEET_REFS}" (id 0) (at 206.9306 45.484 90)
-      (effects (font (size 1.27 1.27)) (justify left) hide)
-    )
-  )
   (global_label "ANT_OUT" (shape output) (at 92.075 66.675 270) (fields_autoplaced)
     (effects (font (size 1.27 1.27)) (justify right))
@@
     )
   )
+  (global_label "PA_OUT" (shape output) (at 207.01 55.88 90) (fields_autoplaced)
+    (effects (font (size 1.27 1.27)) (justify left))
+    (property "Intersheet References" "${INTERSHEET_REFS}" (id 0) (at 207.0894 46.5121 90)
+      (effects (font (size 1.27 1.27)) (justify left) hide)
+    )
+  )

Commit message: Update 17Mar23
Parts:
- removed J35, J40: SHD, TestPoint:TestPoint_Pad_2.0x2.0mm, symbol Connector_Generic:Conn_01x01
- renumbered C85 to C86, C86 to C87, C87 to C88, J32 to J43, J33 to J44, J34 to J45, J38 to J46, J36 to J47, J37 to J48, J39 to J49, J41 to J50, J42 to J51, J43 to J52, J44 to J53, J45 to J54, J46 to J55, R60 to R59, R61 to R60, R62 to R61, R63 to R62, R64 to R63
Other:
- moved on the sheet: J46
