File: Phoenix612 Complete/Version 1.1/AF_amp.kicad_sch (KiCad schematic)
At the start: 30 parts, among them J11 TP, J12 SPK, U6 NE5532, U7 LM380N

Commit message: Update 9Mar23
Parts:
- removed J11: TP, Connector_PinHeader_1.00mm:PinHeader_1x01_P1.00mm_Vertical, symbol Connector_Generic:Conn_01x01
- added J11: TP9, Connector_PinSocket_2.54mm:PinSocket_1x02_P2.54mm_Vertical, symbol Connector_Generic:Conn_01x02
- C37: value 47uf -> 47u
Connections:
- net GND: now also J11.2 (Pin_2)
- net at C39.2, RV3.1: now also J11.1 (Pin_1)
Changed lines of the file:
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@@
   (junction (at 106.68 111.125) (diameter 0) (color 0 0 0 0)
   )
-  (junction (at 123.19 94.615) (diameter 0) (color 0 0 0 0)
+  (junction (at 122.555 94.615) (diameter 0) (color 0 0 0 0)
   )
   (junction (at 148.59 71.12) (diameter 0) (color 0 0 0 0)
@@
     (stroke (width 0) (type default) (color 0 0 0 0))
   )
+  (wire (pts (xy 122.555 94.615) (xy 125.73 94.615))
+    (stroke (width 0) (type default) (color 0 0 0 0))
+  )
   (wire (pts (xy 151.13 88.265) (xy 151.13 89.535))
     (stroke (width 0) (type default) (color 0 0 0 0))
@@
     (stroke (width 0) (type default) (color 0 0 0 0))
   )
-  (wire (pts (xy 118.11 94.615) (xy 123.19 94.615))
-    (stroke (width 0) (type default) (color 0 0 0 0))
-  )
   (wire (pts (xy 125.73 103.505) (xy 125.73 105.41))
     (stroke (width 0) (type default) (color 0 0 0 0))
@@
     (stroke (width 0) (type default) (color 0 0 0 0))
   )
+  (wire (pts (xy 122.555 87.63) (xy 122.555 94.615))
+    (stroke (width 0) (type default) (color 0 0 0 0))
+  )
   (wire (pts (xy 73.66 92.075) (xy 80.01 92.075))
     (stroke (width 0) (type default) (color 0 0 0 0))
@@
     (stroke (width 0) (type default) (color 0 0 0 0))
   )
-  (wire (pts (xy 123.19 94.615) (xy 125.73 94.615))
+  (wire (pts (xy 118.11 94.615) (xy 122.555 94.615))
     (stroke (width 0) (type default) (color 0 0 0 0))
   )
@@
     (pin "8")
   )
-  (symbol (lib_id "Connector_Generic:Conn_01x01") (at 123.19 89.535 90) (unit 1)
-    (in_bom yes) (on_board yes) (fields_autoplaced)
-    (property "Reference" "J11" (id 0) (at 125.73 88.2649 90)
-      (effects (font (size 1.27 1.27)) (justify right))
-    )
-    (property "Value" "TP" (id 1) (at 125.73 90.8049 90)
-      (effects (font (size 1.27 1.27)) (justify right))
-    )
-    (property "Footprint" "Connector_PinHeader_1.00mm:PinHeader_1x01_P1.00mm_Vertical" (id 2) (at 123.19 89.535 0)
-      (effects (font (size 1.27 1.27)) hide)
-    )
-    (property "Datasheet" "~" (id 3) (at 123.19 89.535 0)
+  (symbol (lib_id "power:GND") (at 125.095 87.63 0) (unit 1)
+    (in_bom yes) (on_board yes)
+    (property "Reference" "#PWR0103" (id 0) (at 125.095 93.98 0)
+      (effects (font (size 1.27 1.27)) hide)
+    )
+    (property "Value" "GND" (id 1) (at 125.095 91.44 0))
+    (property "Footprint" "" (id 2) (at 125.095 87.63 0)
+      (effects (font (size 1.27 1.27)) hide)
+    )
+    (property "Datasheet" "" (id 3) (at 125.095 87.63 0)
       (effects (font (size 1.27 1.27)) hide)
     )
@@
     )
     (property "Datasheet" "~" (id 3) (at 153.67 74.93 0)
+      (effects (font (size 1.27 1.27)) hide)
+    )
+    (pin "1")
+    (pin "2")
+  )
+  (symbol (lib_id "Connector_Generic:Conn_01x02") (at 122.555 82.55 90) (unit 1)
+    (in_bom yes) (on_board yes) (fields_autoplaced)
+    (property "Reference" "J11" (id 0) (at 128.27 81.2799 90)
+      (effects (font (size 1.27 1.27)) (justify right))
+    )
+    (property "Value" "TP9" (id 1) (at 128.27 83.8199 90)
+      (effects (font (size 1.27 1.27)) (justify right))
+    )
+    (property "Footprint" "Connector_PinSocket_2.54mm:PinSocket_1x02_P2.54mm_Vertical" (id 2) (at 122.555 82.55 0)
+      (effects (font (size 1.27 1.27)) hide)
+    )
+    (property "Datasheet" "~" (id 3) (at 122.555 82.55 0)
       (effects (font (size 1.27 1.27)) hide)
     )
@@
       (effects (font (size 1.27 1.27)) (justify left))
     )
-    (property "Value" "47uf" (id 1) (at 156.21 86.995 0)
-      (effects (font (size 1.27 1.27)) (justify left))
-    )
+    (property "Value" "47u" (id 1) (at 156.21 86.995 0)
+      (effects (font (size 1.27 1.27)) (justify left))
+    )

Commit message: Update 17Mar23
Parts:
- renumbered C35 to C36, C36 to C37, C37 to C38, C38 to C39, C39 to C40, C40 to C41, C41 to C42, C42 to C43, C43 to C44, C44 to C45, C45 to C46, C46 to C47, C47 to C48, J11 to J14, J12 to J15
Changed lines of the file:
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@@
   (symbol (lib_id "Device:C_Small") (at 89.535 169.545 0) (unit 1)
     (in_bom yes) (on_board yes) (fields_autoplaced)
-    (property "Reference" "C47" (id 0) (at 92.075 168.2812 0)
+    (property "Reference" "C48" (id 0) (at 92.075 168.2812 0)
       (effects (font (size 1.27 1.27)) (justify left))
     )
@@
   (symbol (lib_id "power:GND") (at 125.095 87.63 0) (unit 1)
     (in_bom yes) (on_board yes)
-    (property "Reference" "#PWR0103" (id 0) (at 125.095 93.98 0)
+    (property "Reference" "#PWR050" (id 0) (at 125.095 93.98 0)
       (effects (font (size 1.27 1.27)) hide)
     )
@@
   (symbol (lib_id "power:GND") (at 167.64 112.395 0) (unit 1)
     (in_bom yes) (on_board yes)
-    (property "Reference" "#PWR037" (id 0) (at 167.64 118.745 0)
+    (property "Reference" "#PWR055" (id 0) (at 167.64 118.745 0)
       (effects (font (size 1.27 1.27)) hide)
     )
@@
   (symbol (lib_id "Device:C_Polarized_Small_US") (at 78.105 169.545 0) (unit 1)
     (in_bom yes) (on_board yes) (fields_autoplaced)
-    (property "Reference" "C46" (id 0) (at 81.28 167.8431 0)
+    (property "Reference" "C47" (id 0) (at 81.28 167.8431 0)
       (effects (font (size 1.27 1.27)) (justify left))
     )
@@
   (symbol (lib_id "Device:C_Small") (at 101.6 116.205 90) (unit 1)
     (in_bom yes) (on_board yes)
-    (property "Reference" "C42" (id 0) (at 101.6 113.665 90))
+    (property "Reference" "C43" (id 0) (at 101.6 113.665 90))
     (property "Value" "470p" (id 1) (at 102.87 120.015 90))
     (property "Footprint" "Capacitor_SMD:C_1206_3216Metric" (id 2) (at 101.6 116.205 0)
@@
   (symbol (lib_id "power:GND") (at 144.78 108.585 0) (unit 1)
     (in_bom yes) (on_board yes)
-    (property "Reference" "#PWR036" (id 0) (at 144.78 114.935 0)
+    (property "Reference" "#PWR054" (id 0) (at 144.78 114.935 0)
       (effects (font (size 1.27 1.27)) hide)
     )
@@
   (symbol (lib_id "power:PWR_FLAG") (at 89.535 163.195 0) (unit 1)
     (in_bom yes) (on_board yes) (fields_autoplaced)
-    (property "Reference" "#FLG09" (id 0) (at 89.535 161.29 0)
+    (property "Reference" "#FLG010" (id 0) (at 89.535 161.29 0)
       (effects (font (size 1.27 1.27)) hide)
     )
@@
   (symbol (lib_id "power:GND") (at 110.49 173.355 0) (unit 1)
     (in_bom yes) (on_board yes)
-    (property "Reference" "#PWR042" (id 0) (at 110.49 179.705 0)
+    (property "Reference" "#PWR060" (id 0) (at 110.49 179.705 0)
       (effects (font (size 1.27 1.27)) hide)
     )
@@
   (symbol (lib_id "Device:C_Small") (at 71.12 92.075 90) (unit 1)
     (in_bom yes) (on_board yes)
-    (property "Reference" "C38" (id 0) (at 71.12 88.265 90))
+    (property "Reference" "C39" (id 0) (at 71.12 88.265 90))
     (property "Value" "68n" (id 1) (at 71.12 95.885 90))
     (property "Footprint" "Capacitor_SMD:C_1206_3216Metric" (id 2) (at 71.12 92.075 0)
@@
   (symbol (lib_id "Device:C_Small") (at 129.54 168.91 0) (unit 1)
     (in_bom yes) (on_board yes)
-    (property "Reference" "C45" (id 0) (at 131.445 167.005 0)
+    (property "Reference" "C46" (id 0) (at 131.445 167.005 0)
       (effects (font (size 1.27 1.27)) (justify left))
     )
@@
   (symbol (lib_id "power:GND") (at 153.67 77.47 0) (unit 1)
     (in_bom yes) (on_board yes)
-    (property "Reference" "#PWR032" (id 0) (at 153.67 83.82 0)
+    (property "Reference" "#PWR049" (id 0) (at 153.67 83.82 0)
       (effects (font (size 1.27 1.27)) hide)
     )
@@
   (symbol (lib_id "power:GND") (at 158.75 88.9 0) (unit 1)
     (in_bom yes) (on_board yes)
-    (property "Reference" "#PWR033" (id 0) (at 158.75 95.25 0)
+    (property "Reference" "#PWR051" (id 0) (at 158.75 95.25 0)
       (effects (font (size 1.27 1.27)) hide)
     )
@@
   (symbol (lib_id "Device:C_Small") (at 167.64 109.855 0) (unit 1)
     (in_bom yes) (on_board yes) (fields_autoplaced)
-    (property "Reference" "C41" (id 0) (at 170.18 108.5912 0)
+    (property "Reference" "C42" (id 0) (at 170.18 108.5912 0)
       (effects (font (size 1.27 1.27)) (justify left))
     )
@@
   (symbol (lib_id "Device:C_Polarized_Small_US") (at 88.9 123.825 0) (unit 1)
     (in_bom yes) (on_board yes) (fields_autoplaced)
-    (property "Reference" "C43" (id 0) (at 91.44 122.1231 0)
+    (property "Reference" "C44" (id 0) (at 91.44 122.1231 0)
       (effects (font (size 1.27 1.27)) (justify left))
     )
@@
   (symbol (lib_id "Device:C_Small") (at 115.57 94.615 90) (unit 1)
     (in_bom yes) (on_board yes)
-    (property "Reference" "C39" (id 0) (at 115.57 90.17 90))
+    (property "Reference" "C40" (id 0) (at 115.57 90.17 90))
     (property "Value" ".22u" (id 1) (at 115.57 98.425 90))
     (property "Footprint" "Capacitor_SMD:C_1206_3216Metric_Pad1.33x1.80mm_HandSolder" (id 2) (at 115.57 94.615 0)
@@
   (symbol (lib_id "power:GND") (at 58.42 166.37 0) (unit 1)
     (in_bom yes) (on_board yes)
-    (property "Reference" "#PWR039" (id 0) (at 58.42 172.72 0)
+    (property "Reference" "#PWR057" (id 0) (at 58.42 172.72 0)
       (effects (font (size 1.27 1.27)) hide)
     )
@@
   (symbol (lib_id "Device:C_Polarized_Small_US") (at 139.7 168.275 0) (unit 1)
     (in_bom yes) (on_board yes)
-    (property "Reference" "C44" (id 0) (at 142.24 167.005 0)
+    (property "Reference" "C45" (id 0) (at 142.24 167.005 0)
       (effects (font (size 1.27 1.27)) (justify left))
     )
@@
   (symbol (lib_id "Device:C_Polarized_Small_US") (at 143.51 74.295 0) (unit 1)
     (in_bom yes) (on_board yes)
-    (property "Reference" "C35" (id 0) (at 138.43 73.025 0)
+    (property "Reference" "C36" (id 0) (at 138.43 73.025 0)
       (effects (font (size 1.27 1.27)) (justify left))
     )
@@
   (symbol (lib_id "Device:C_Small") (at 153.67 74.93 0) (unit 1)
     (in_bom yes) (on_board yes) (fields_autoplaced)
-    (property "Reference" "C36" (id 0) (at 156.21 73.6662 0)
+    (property "Reference" "C37" (id 0) (at 156.21 73.6662 0)
       (effects (font (size 1.27 1.27)) (justify left))
     )
@@
   (symbol (lib_id "Connector_Generic:Conn_01x02") (at 122.555 82.55 90) (unit 1)
     (in_bom yes) (on_board yes) (fields_autoplaced)
-    (property "Reference" "J11" (id 0) (at 128.27 81.2799 90)
+    (property "Reference" "J14" (id 0) (at 128.27 81.2799 90)
       (effects (font (size 1.27 1.27)) (justify right))
     )
@@
   (symbol (lib_id "Connector_Generic:Conn_01x02") (at 186.69 97.155 0) (unit 1)
     (in_bom yes) (on_board yes) (fields_autoplaced)
-    (property "Reference" "J12" (id 0) (at 189.23 97.1549 0)
+    (property "Reference" "J15" (id 0) (at 189.23 97.1549 0)
       (effects (font (size 1.27 1.27)) (justify left))
     )
@@
   (symbol (lib_id "power:GND") (at 78.105 172.085 0) (unit 1)
     (in_bom yes) (on_board yes)
-    (property "Reference" "#PWR040" (id 0) (at 78.105 178.435 0)
+    (property "Reference" "#PWR058" (id 0) (at 78.105 178.435 0)
       (effects (font (size 1.27 1.27)) hide)
     )
@@
   (symbol (lib_id "power:GND") (at 139.7 173.355 0) (unit 1)
     (in_bom yes) (on_board yes)
-    (property "Reference" "#PWR044" (id 0) (at 139.7 179.705 0)
+    (property "Reference" "#PWR062" (id 0) (at 139.7 179.705 0)
       (effects (font (size 1.27 1.27)) hide)
     )
@@
   (symbol (lib_id "power:PWR_FLAG") (at 153.67 71.12 0) (unit 1)
     (in_bom yes) (on_board yes) (fields_autoplaced)
-    (property "Reference" "#FLG08" (id 0) (at 153.67 69.215 0)
+    (property "Reference" "#FLG09" (id 0) (at 153.67 69.215 0)
       (effects (font (size 1.27 1.27)) hide)
     )
@@
   (symbol (lib_id "power:GND") (at 129.54 173.355 0) (unit 1)
     (in_bom yes) (on_board yes)
-    (property "Reference" "#PWR043" (id 0) (at 129.54 179.705 0)
+    (property "Reference" "#PWR061" (id 0) (at 129.54 179.705 0)
       (effects (font (size 1.27 1.27)) hide)
     )
@@
   (symbol (lib_id "power:GND") (at 89.535 172.085 0) (unit 1)
     (in_bom yes) (on_board yes)
-    (property "Reference" "#PWR041" (id 0) (at 89.535 178.435 0)
+    (property "Reference" "#PWR059" (id 0) (at 89.535 178.435 0)
       (effects (font (size 1.27 1.27)) hide)
     )
@@
   (symbol (lib_id "Device:C_Polarized_Small_US") (at 153.67 88.265 90) (unit 1)
     (in_bom yes) (on_board yes)
-    (property "Reference" "C37" (id 0) (at 151.13 86.995 0)
+    (property "Reference" "C38" (id 0) (at 151.13 86.995 0)
       (effects (font (size 1.27 1.27)) (justify left))
     )
@@
   (symbol (lib_id "power:GND") (at 143.51 76.835 0) (unit 1)
     (in_bom yes) (on_board yes)
-    (property "Reference" "#PWR031" (id 0) (at 143.51 83.185 0)
+    (property "Reference" "#PWR048" (id 0) (at 143.51 83.185 0)
       (effects (font (size 1.27 1.27)) hide)
     )
@@
   (symbol (lib_id "power:GND") (at 125.73 105.41 0) (unit 1)
     (in_bom yes) (on_board yes)
-    (property "Reference" "#PWR035" (id 0) (at 125.73 111.76 0)
+    (property "Reference" "#PWR053" (id 0) (at 125.73 111.76 0)
       (effects (font (size 1.27 1.27)) hide)
     )
@@
   (symbol (lib_id "power:GND") (at 179.705 101.6 0) (unit 1)
     (in_bom yes) (on_board yes)
-    (property "Reference" "#PWR034" (id 0) (at 179.705 107.95 0)
+    (property "Reference" "#PWR052" (id 0) (at 179.705 107.95 0)
       (effects (font (size 1.27 1.27)) hide)
     )
@@
   (symbol (lib_id "Device:C_Polarized_Small_US") (at 175.26 97.155 90) (unit 1)
     (in_bom yes) (on_board yes)
-    (property "Reference" "C40" (id 0) (at 175.26 91.44 90))
+    (property "Reference" "C41" (id 0) (at 175.26 91.44 90))
     (property "Value" "470u" (id 1) (at 175.895 93.98 90))
     (property "Footprint" "Capacitor_THT:CP_Radial_D8.0mm_P3.50mm" (id 2) (at 175.26 97.155 0)
@@
   (symbol (lib_id "power:GND") (at 88.9 126.365 0) (unit 1)
     (in_bom yes) (on_board yes)
-    (property "Reference" "#PWR038" (id 0) (at 88.9 132.715 0)
-      (effects (font (size 1.27 1.27)) hide)
-    )
+    (property "Reference" "#PWR056" (id 0) (at 88.9 132.715 0)
+      (effects (font (size 1.27 1.27)) hide)
+    )

Commit message: Update 24Mar23
Parts:
- AFG1: renamed from RV3; value 10k -> 10K
Connections:
- net GND: now also AFG1.1; no longer AFG1.3
- net at C40.2, J14.1 (Pin_1): now also AFG1.3; no longer AFG1.1
Other:
- moved on the sheet: AFG1
Changed lines of the file:
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@@
-    (stroke (width 0) (type default) (color 0 0 0 0))
-  )
-  (wire (pts (xy 133.35 99.695) (xy 129.54 99.695))
     (stroke (width 0) (type default) (color 0 0 0 0))
   )
@@
     (stroke (width 0) (type default) (color 0 0 0 0))
   )
-  (wire (pts (xy 133.35 94.615) (xy 133.35 99.695))
+  (wire (pts (xy 133.35 94.615) (xy 133.35 100.965))
     (stroke (width 0) (type default) (color 0 0 0 0))
   )
@@
     (stroke (width 0) (type default) (color 0 0 0 0))
   )
+  (wire (pts (xy 148.59 107.315) (xy 144.78 107.315))
+    (stroke (width 0) (type default) (color 0 0 0 0))
+  )
+  (wire (pts (xy 80.01 92.075) (xy 91.44 92.075))
+    (stroke (width 0) (type default) (color 0 0 0 0))
+  )
+  (wire (pts (xy 140.97 99.695) (xy 143.51 99.695))
+    (stroke (width 0) (type default) (color 0 0 0 0))
+  )
+  (wire (pts (xy 144.78 107.315) (xy 144.78 108.585))
+    (stroke (width 0) (type default) (color 0 0 0 0))
+  )
+  (wire (pts (xy 124.46 164.465) (xy 129.54 164.465))
+    (stroke (width 0) (type default) (color 0 0 0 0))
+  )
+  (wire (pts (xy 143.51 71.12) (xy 148.59 71.12))
+    (stroke (width 0) (type default) (color 0 0 0 0))
+  )
+  (wire (pts (xy 110.49 94.615) (xy 113.03 94.615))
+    (stroke (width 0) (type default) (color 0 0 0 0))
+  )
+  (wire (pts (xy 106.68 94.615) (xy 110.49 94.615))
+    (stroke (width 0) (type default) (color 0 0 0 0))
+  )
+  (wire (pts (xy 148.59 107.315) (xy 151.13 107.315))
+    (stroke (width 0) (type default) (color 0 0 0 0))
+  )
+  (wire (pts (xy 78.105 165.735) (xy 89.535 165.735))
+    (stroke (width 0) (type default) (color 0 0 0 0))
+  )
+  (wire (pts (xy 125.73 103.505) (xy 125.73 105.41))
+    (stroke (width 0) (type default) (color 0 0 0 0))
+  )
+  (wire (pts (xy 70.485 165.735) (xy 70.485 164.465))
+    (stroke (width 0) (type default) (color 0 0 0 0))
+  )
+  (wire (pts (xy 151.13 104.775) (xy 151.13 107.315))
+    (stroke (width 0) (type default) (color 0 0 0 0))
+  )
+  (wire (pts (xy 124.46 148.59) (xy 124.46 149.225))
+    (stroke (width 0) (type default) (color 0 0 0 0))
+  )
+  (wire (pts (xy 148.59 71.12) (xy 153.67 71.12))
+    (stroke (width 0) (type default) (color 0 0 0 0))
+  )
+  (wire (pts (xy 91.44 97.155) (xy 88.9 97.155))
+    (stroke (width 0) (type default) (color 0 0 0 0))
+  )
+  (wire (pts (xy 142.24 94.615) (xy 143.51 94.615))
+    (stroke (width 0) (type default) (color 0 0 0 0))
+  )
+  (wire (pts (xy 104.14 116.205) (xy 106.68 116.205))
+    (stroke (width 0) (type default) (color 0 0 0 0))
+  )
+  (wire (pts (xy 134.62 94.615) (xy 133.35 94.615))
+    (stroke (width 0) (type default) (color 0 0 0 0))
+  )
+  (wire (pts (xy 121.92 100.965) (xy 133.35 100.965))
+    (stroke (width 0) (type default) (color 0 0 0 0))
+  )
+  (wire (pts (xy 129.54 173.355) (xy 129.54 171.45))
+    (stroke (width 0) (type default) (color 0 0 0 0))
+  )
+  (wire (pts (xy 158.75 88.265) (xy 158.75 88.9))
+    (stroke (width 0) (type default) (color 0 0 0 0))
+  )
+  (wire (pts (xy 156.21 88.265) (xy 158.75 88.265))
+    (stroke (width 0) (type default) (color 0 0 0 0))
+  )
+  (wire (pts (xy 148.59 48.26) (xy 148.59 51.435))
+    (stroke (width 0) (type default) (color 0 0 0 0))
+  )
+  (wire (pts (xy 110.49 94.615) (xy 110.49 111.125))
+    (stroke (width 0) (type default) (color 0 0 0 0))
+  )
+  (wire (pts (xy 167.64 99.695) (xy 167.64 97.155))
+    (stroke (width 0) (type default) (color 0 0 0 0))
+  )
   (wire (pts (xy 125.73 94.615) (xy 125.73 95.885))
     (stroke (width 0) (type default) (color 0 0 0 0))
   )
-  (wire (pts (xy 148.59 107.315) (xy 144.78 107.315))
-    (stroke (width 0) (type default) (color 0 0 0 0))
-  )
-  (wire (pts (xy 80.01 92.075) (xy 91.44 92.075))
-    (stroke (width 0) (type default) (color 0 0 0 0))
-  )
-  (wire (pts (xy 140.97 99.695) (xy 143.51 99.695))
-    (stroke (width 0) (type default) (color 0 0 0 0))
-  )
-  (wire (pts (xy 144.78 107.315) (xy 144.78 108.585))
-    (stroke (width 0) (type default) (color 0 0 0 0))
-  )
-  (wire (pts (xy 124.46 164.465) (xy 129.54 164.465))
-    (stroke (width 0) (type default) (color 0 0 0 0))
-  )
-  (wire (pts (xy 143.51 71.12) (xy 148.59 71.12))
-    (stroke (width 0) (type default) (color 0 0 0 0))
-  )
-  (wire (pts (xy 110.49 94.615) (xy 113.03 94.615))
-    (stroke (width 0) (type default) (color 0 0 0 0))
-  )
-  (wire (pts (xy 106.68 94.615) (xy 110.49 94.615))
-    (stroke (width 0) (type default) (color 0 0 0 0))
-  )
-  (wire (pts (xy 148.59 107.315) (xy 151.13 107.315))
-    (stroke (width 0) (type default) (color 0 0 0 0))
-  )
-  (wire (pts (xy 78.105 165.735) (xy 89.535 165.735))
-    (stroke (width 0) (type default) (color 0 0 0 0))
-  )
-  (wire (pts (xy 70.485 165.735) (xy 70.485 164.465))
-    (stroke (width 0) (type default) (color 0 0 0 0))
-  )
-  (wire (pts (xy 151.13 104.775) (xy 151.13 107.315))
-    (stroke (width 0) (type default) (color 0 0 0 0))
-  )
-  (wire (pts (xy 124.46 148.59) (xy 124.46 149.225))
-    (stroke (width 0) (type default) (color 0 0 0 0))
-  )
-  (wire (pts (xy 148.59 71.12) (xy 153.67 71.12))
-    (stroke (width 0) (type default) (color 0 0 0 0))
-  )
-  (wire (pts (xy 91.44 97.155) (xy 88.9 97.155))
-    (stroke (width 0) (type default) (color 0 0 0 0))
-  )
-  (wire (pts (xy 142.24 94.615) (xy 143.51 94.615))
-    (stroke (width 0) (type default) (color 0 0 0 0))
-  )
-  (wire (pts (xy 125.73 103.505) (xy 125.73 105.41))
-    (stroke (width 0) (type default) (color 0 0 0 0))
-  )
-  (wire (pts (xy 104.14 116.205) (xy 106.68 116.205))
-    (stroke (width 0) (type default) (color 0 0 0 0))
-  )
-  (wire (pts (xy 134.62 94.615) (xy 133.35 94.615))
-    (stroke (width 0) (type default) (color 0 0 0 0))
-  )
-  (wire (pts (xy 129.54 173.355) (xy 129.54 171.45))
-    (stroke (width 0) (type default) (color 0 0 0 0))
-  )
-  (wire (pts (xy 158.75 88.265) (xy 158.75 88.9))
-    (stroke (width 0) (type default) (color 0 0 0 0))
-  )
-  (wire (pts (xy 156.21 88.265) (xy 158.75 88.265))
-    (stroke (width 0) (type default) (color 0 0 0 0))
-  )
-  (wire (pts (xy 148.59 48.26) (xy 148.59 51.435))
-    (stroke (width 0) (type default) (color 0 0 0 0))
-  )
-  (wire (pts (xy 110.49 94.615) (xy 110.49 111.125))
-    (stroke (width 0) (type default) (color 0 0 0 0))
-  )
-  (wire (pts (xy 167.64 99.695) (xy 167.64 97.155))
-    (stroke (width 0) (type default) (color 0 0 0 0))
-  )
   (wire (pts (xy 106.68 116.205) (xy 106.68 111.125))
     (stroke (width 0) (type default) (color 0 0 0 0))
@@
   )
   (wire (pts (xy 148.59 71.12) (xy 148.59 89.535))
+    (stroke (width 0) (type default) (color 0 0 0 0))
+  )
+  (wire (pts (xy 121.92 99.695) (xy 121.92 100.965))
     (stroke (width 0) (type default) (color 0 0 0 0))
   )
@@
     (pin "1")
   )
-  (symbol (lib_id "Device:R_Potentiometer") (at 125.73 99.695 0) (unit 1)
-    (in_bom yes) (on_board yes)
-    (property "Reference" "RV3" (id 0) (at 123.825 101.6 0)
+  (symbol (lib_id "Device:R_Potentiometer") (at 125.73 99.695 180) (unit 1)
+    (in_bom yes) (on_board yes)
+    (property "Reference" "AFG1" (id 0) (at 127.635 97.79 0)
       (effects (font (size 1.27 1.27)) (justify right))
     )
-    (property "Value" "10k" (id 1) (at 130.81 101.6 0)
+    (property "Value" "10K" (id 1) (at 120.65 97.79 0)
       (effects (font (size 1.27 1.27)) (justify right))
     )
