File: Phoenix612 Complete/Version 1.1/PowerAmp.kicad_sch (KiCad schematic)
At the start: 38 parts, among them J18 TP, J19 TP, J20 JMP, J21 SHD, J22 SHD, J23 SHD, J24 SHD, J25 SHD, J26 SHD, J27 SHD, J28 SHD, J29 SHD, J30 SHD, J31 SHD, Q3 RD16HHF1, T3 FT37-43 1:4, U11 QPR_Filter

Commit message: Update 9Mar23
Parts:
- removed J18, J19: TP, Connector_PinHeader_1.00mm:PinHeader_1x01_P1.00mm_Vertical, symbol Connector_Generic:Conn_01x01
- added J18: TP16, Connector_PinSocket_2.54mm:PinSocket_1x02_P2.54mm_Vertical, symbol Connector_Generic:Conn_01x02
- added J19: TP15, Connector_PinSocket_2.54mm:PinSocket_1x02_P2.54mm_Vertical, symbol Connector_Generic:Conn_01x02
Connections:
- net GND: now also J18.2 (Pin_2), J19.2 (Pin_2)
- net PA_OUT: now also J18.1 (Pin_1)
- net at C78.2, C79.1, C80.1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: now also J19.1 (Pin_1)
Changed lines of the file:
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@@
   (junction (at 101.6 137.795) (diameter 0) (color 0 0 0 0)
   )
+  (junction (at 151.13 62.865) (diameter 0) (color 0 0 0 0)
+  )
   (junction (at 73.66 80.01) (diameter 0) (color 0 0 0 0)
   )
@@
   (junction (at 86.36 99.695) (diameter 0) (color 0 0 0 0)
   )
-  (junction (at 150.495 62.865) (diameter 0) (color 0 0 0 0)
-  )
   (junction (at 77.47 136.525) (diameter 0) (color 0 0 0 0)
   )
@@
     (stroke (width 0) (type default) (color 0 0 0 0))
   )
+  (wire (pts (xy 151.13 46.99) (xy 151.13 62.865))
+    (stroke (width 0) (type default) (color 0 0 0 0))
+  )
   (wire (pts (xy 36.195 74.295) (xy 40.005 74.295))
     (stroke (width 0) (type default) (color 0 0 0 0))
@@
     (stroke (width 0) (type default) (color 0 0 0 0))
   )
+  (wire (pts (xy 151.13 62.865) (xy 160.655 62.865))
+    (stroke (width 0) (type default) (color 0 0 0 0))
+  )
   (wire (pts (xy 242.57 25.4) (xy 242.57 31.115))
     (stroke (width 0) (type default) (color 0 0 0 0))
   )
-  (wire (pts (xy 150.495 62.865) (xy 144.78 62.865))
-    (stroke (width 0) (type default) (color 0 0 0 0))
-  )
   (wire (pts (xy 86.36 99.695) (xy 93.345 99.695))
     (stroke (width 0) (type default) (color 0 0 0 0))
@@
     (stroke (width 0) (type default) (color 0 0 0 0))
   )
-  (wire (pts (xy 50.165 73.66) (xy 50.165 68.58))
+  (wire (pts (xy 50.165 53.34) (xy 50.165 73.66))
     (stroke (width 0) (type default) (color 0 0 0 0))
   )
@@
     (stroke (width 0) (type default) (color 0 0 0 0))
   )
-  (wire (pts (xy 150.495 62.865) (xy 160.655 62.865))
+  (wire (pts (xy 144.78 62.865) (xy 151.13 62.865))
     (stroke (width 0) (type default) (color 0 0 0 0))
   )
@@
     (pin "1")
   )
+  (symbol (lib_id "Connector_Generic:Conn_01x02") (at 151.13 41.91 90) (unit 1)
+    (in_bom yes) (on_board yes) (fields_autoplaced)
+    (property "Reference" "J18" (id 0) (at 156.21 40.6399 90)
+      (effects (font (size 1.27 1.27)) (justify right))
+    )
+    (property "Value" "TP16" (id 1) (at 156.21 43.1799 90)
+      (effects (font (size 1.27 1.27)) (justify right))
+    )
+    (property "Footprint" "Connector_PinSocket_2.54mm:PinSocket_1x02_P2.54mm_Vertical" (id 2) (at 151.13 41.91 0)
+      (effects (font (size 1.27 1.27)) hide)
+    )
+    (property "Datasheet" "~" (id 3) (at 151.13 41.91 0)
+      (effects (font (size 1.27 1.27)) hide)
+    )
+    (pin "1")
+    (pin "2")
+  )
   (symbol (lib_id "Device:C") (at 218.44 53.975 0) (unit 1)
     (in_bom yes) (on_board yes) (fields_autoplaced)
@@
     (pin "2")
   )
-  (symbol (lib_id "Connector_Generic:Conn_01x01") (at 150.495 57.785 90) (unit 1)
-    (in_bom yes) (on_board yes) (fields_autoplaced)
-    (property "Reference" "J18" (id 0) (at 153.035 56.5149 90)
+  (symbol (lib_id "Connector_Generic:Conn_01x02") (at 50.165 48.26 90) (unit 1)
+    (in_bom yes) (on_board yes) (fields_autoplaced)
+    (property "Reference" "J19" (id 0) (at 55.88 46.9899 90)
       (effects (font (size 1.27 1.27)) (justify right))
     )
-    (property "Value" "TP" (id 1) (at 153.035 59.0549 90)
+    (property "Value" "TP15" (id 1) (at 55.88 49.5299 90)
       (effects (font (size 1.27 1.27)) (justify right))
     )
-    (property "Footprint" "Connector_PinHeader_1.00mm:PinHeader_1x01_P1.00mm_Vertical" (id 2) (at 150.495 57.785 0)
-      (effects (font (size 1.27 1.27)) hide)
-    )
-    (property "Datasheet" "~" (id 3) (at 150.495 57.785 0)
-      (effects (font (size 1.27 1.27)) hide)
-    )
-    (pin "1")
+    (property "Footprint" "Connector_PinSocket_2.54mm:PinSocket_1x02_P2.54mm_Vertical" (id 2) (at 50.165 48.26 0)
+      (effects (font (size 1.27 1.27)) hide)
+    )
+    (property "Datasheet" "~" (id 3) (at 50.165 48.26 0)
+      (effects (font (size 1.27 1.27)) hide)
+    )
+    (pin "1")
+    (pin "2")
   )
   (symbol (lib_id "Device:L_Ferrite") (at 242.57 34.925 0) (unit 1)
@@
     (pin "1")
     (pin "2")
+  )
+  (symbol (lib_id "power:GND") (at 153.67 46.99 0) (unit 1)
+    (in_bom yes) (on_board yes)
+    (property "Reference" "#PWR0111" (id 0) (at 153.67 53.34 0)
+      (effects (font (size 1.27 1.27)) hide)
+    )
+    (property "Value" "GND" (id 1) (at 153.67 50.8 0))
+    (property "Footprint" "" (id 2) (at 153.67 46.99 0)
+      (effects (font (size 1.27 1.27)) hide)
+    )
+    (property "Datasheet" "" (id 3) (at 153.67 46.99 0)
+      (effects (font (size 1.27 1.27)) hide)
+    )
+    (pin "1")
   )
   (symbol (lib_id "Device:R_US") (at 67.31 73.66 270) (unit 1)
@@
     (pin "2")
   )
-  (symbol (lib_id "Connector_Generic:Conn_01x01") (at 50.165 63.5 90) (unit 1)
-    (in_bom yes) (on_board yes) (fields_autoplaced)
-    (property "Reference" "J19" (id 0) (at 53.34 62.2299 90)
-      (effects (font (size 1.27 1.27)) (justify right))
-    )
-    (property "Value" "TP" (id 1) (at 53.34 64.7699 90)
-      (effects (font (size 1.27 1.27)) (justify right))
-    )
-    (property "Footprint" "Connector_PinHeader_1.00mm:PinHeader_1x01_P1.00mm_Vertical" (id 2) (at 50.165 63.5 0)
-      (effects (font (size 1.27 1.27)) hide)
-    )
-    (property "Datasheet" "~" (id 3) (at 50.165 63.5 0)
-      (effects (font (size 1.27 1.27)) hide)
-    )
-    (pin "1")
-  )
   (symbol (lib_id "Device:C") (at 53.975 104.775 0) (unit 1)
     (in_bom yes) (on_board yes)
@@
     (pin "2")
   )
+  (symbol (lib_id "power:GND") (at 52.705 53.34 0) (unit 1)
+    (in_bom yes) (on_board yes)
+    (property "Reference" "#PWR0110" (id 0) (at 52.705 59.69 0)
+      (effects (font (size 1.27 1.27)) hide)
+    )
+    (property "Value" "GND" (id 1) (at 52.705 57.15 0))
+    (property "Footprint" "" (id 2) (at 52.705 53.34 0)
+      (effects (font (size 1.27 1.27)) hide)
+    )
+    (property "Datasheet" "" (id 3) (at 52.705 53.34 0)
+      (effects (font (size 1.27 1.27)) hide)
+    )
+    (pin "1")
+  )
   (symbol (lib_id "Connector_Generic:Conn_01x01") (at 82.55 167.64 0) (unit 1)

Commit message: Update 17Mar23
Parts:
- added J27, J29, J32, J33, J35, J38, J39, J57: SHD, Connector_PinHeader_2.54mm:PinHeader_1x01_P2.54mm_Vertical, symbol Connector_Generic:Conn_01x01
- added Q4: IRF510, TO220, symbol Custom_RF:IRF510
- renumbered C72 to C73, C73 to C74, C74 to C75, C75 to C76, C76 to C77, C77 to C78, C78 to C79, C79 to C80, C80 to C81, C81 to C82, C82 to C83, C83 to C84, C84 to C85, J18 to J22, J19 to J23, J20 to J24, J21 to J25, J22 to J26, J23 to J28, J24 to J30, J25 to J31, J26 to J34, J27 to J36, J28 to J37, J29 to J40, J30 to J41, J31 to J42, R56 to R55, R57 to R56, R58 to R57, R59 to R58
Connections:
- net GND: now also J27.1 (Pin_1), J29.1 (Pin_1), J32.1 (Pin_1), J33.1 (Pin_1), J35.1 (Pin_1), J38.1 (Pin_1), J39.1 (Pin_1), J57.1 (Pin_1), Q4.1
- net at Q3.1, R56.1: now also Q4.3
- net at J24.2 (Pin_2), Q3.3, R55.1: now also Q4.2
Other:
- moved on the sheet: C82, C83, C84, C85, D8, L14, R58, RV6

Commit message: Update LT1253 Tx
Parts:
- Q4: footprint TO220 -> Custom_RF:TO-220-3_REV
Changed lines of the file:
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@@
       (effects (font (size 1.27 1.27)) (justify left))
     )
-    (property "Footprint" "TO220" (id 2) (at 90.17 91.44 0)
+    (property "Footprint" "Custom_RF:TO-220-3_REV" (id 2) (at 93.98 88.9 0)
       (effects (font (size 1.27 1.27)) (justify left bottom) hide)
     )

Commit message: Update 24Mar23
Parts:
- renumbered RV6 to BS1
Changed lines of the file:
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@@
   (symbol (lib_id "Device:R_Potentiometer_Trim") (at 76.835 113.03 180) (unit 1)
     (in_bom yes) (on_board yes)
-    (property "Reference" "RV6" (id 0) (at 78.74 115.57 0)
+    (property "Reference" "BS1" (id 0) (at 78.74 116.84 0)
       (effects (font (size 1.27 1.27)) (justify right))
     )
