File: Phoenix612 Complete/Version 1.1/IF_Stage.kicad_sch (KiCad schematic)
At the start: 51 parts, among them J10 TP, J4 TP, J5 VFO, J6 TP, J7 TP, J8 TP, J9 BFO, K2 G5V-2, K3 G5V-2, T1 FT50-75 (18:7), T2 FT50-75 (7:18), U4 SA612, U5 SA612, Y1 12 MHz, Y2 12 MHz, Y3 12 MHz, Y4 12 MHz

Commit message: Update 9Mar23
Parts:
- removed J10, J4, J6, J7, J8: TP, Connector_PinHeader_1.00mm:PinHeader_1x01_P1.00mm_Vertical, symbol Connector_Generic:Conn_01x01
- added C100: 100n, Capacitor_SMD:C_1206_3216Metric, symbol Device:C
- added J10: TP4, Connector_PinSocket_2.54mm:PinSocket_1x02_P2.54mm_Vertical, symbol Connector_Generic:Conn_01x02
- added J4: TP5, Connector_PinSocket_2.54mm:PinSocket_1x02_P2.54mm_Vertical, symbol Connector_Generic:Conn_01x02
- added J49: TP8, Connector_PinSocket_2.54mm:PinSocket_1x02_P2.54mm_Vertical, symbol Connector_Generic:Conn_01x02
- added J6: TP3, Connector_PinSocket_2.54mm:PinSocket_1x02_P2.54mm_Vertical, symbol Connector_Generic:Conn_01x02
- added J7: TP6, Connector_PinSocket_2.54mm:PinSocket_1x02_P2.54mm_Vertical, symbol Connector_Generic:Conn_01x02
- added J8: TP7, Connector_PinSocket_2.54mm:PinSocket_1x02_P2.54mm_Vertical, symbol Connector_Generic:Conn_01x02
- C26, C27, C28: footprint Capacitor_THT:C_Disc_D4.7mm_W2.5mm_P5.00mm -> Capacitor_SMD:C_1206_3216Metric
Connections:
- net GND: now also J10.1 (Pin_1), J4.2 (Pin_2), J49.2 (Pin_2), J6.2 (Pin_2), J7.2 (Pin_2), J8.2 (Pin_2)
- net at C19.2, U4.1 (IN_A): now also J6.1 (Pin_1)
- net at C15.2, U4.6 (OSC_B): now also J4.1 (Pin_1)
- net at C30.1, T2.4 (SB): now also J7.1 (Pin_1)
- net at K3.13, K3.4, U5.4 (OUT_A): now also C100.1
- net at C32.2, U5.6 (OSC_B): now also J8.1 (Pin_1)
- net at C29.2, T1.1 (AA): now also J10.2 (Pin_2)
- new net: C100.2, J49.1 (Pin_1)
Other:
- moved on the sheet: C29

Commit message: Update_17Mar23
Parts:
- C100: value 100n -> 10u
Changed lines of the file:
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@@
   (symbol (lib_id "Device:C") (at 198.12 140.335 0) (unit 1)
     (in_bom yes) (on_board yes)
-    (property "Reference" "C100" (id 0) (at 195.58 142.875 0)
+    (property "Reference" "C100" (id 0) (at 198.755 142.875 0)
       (effects (font (size 1.27 1.27)) (justify left))
     )
-    (property "Value" "100n" (id 1) (at 191.77 137.795 0)
+    (property "Value" "10u" (id 1) (at 198.755 137.795 0)
       (effects (font (size 1.27 1.27)) (justify left))
     )

Commit message: Update 17Mar23
Parts:
- renumbered C100 to C34, C34 to C35, J8 to J10, J9 to J11, J10 to J12, J49 to J13, J4 to J6, J5 to J7, J6 to J8, J7 to J9
Changed lines of the file:
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@@
   (symbol (lib_id "power:GND") (at 190.5 134.62 0) (unit 1)
     (in_bom yes) (on_board yes) (fields_autoplaced)
-    (property "Reference" "#PWR029" (id 0) (at 190.5 140.97 0)
+    (property "Reference" "#PWR045" (id 0) (at 190.5 140.97 0)
       (effects (font (size 1.27 1.27)) hide)
     )
@@
   (symbol (lib_id "power:GND") (at 93.98 81.28 0) (unit 1)
     (in_bom yes) (on_board yes)
-    (property "Reference" "#PWR019" (id 0) (at 93.98 87.63 0)
+    (property "Reference" "#PWR031" (id 0) (at 93.98 87.63 0)
       (effects (font (size 1.27 1.27)) hide)
     )
@@
   (symbol (lib_id "Device:C") (at 198.12 140.335 0) (unit 1)
     (in_bom yes) (on_board yes)
-    (property "Reference" "C100" (id 0) (at 198.755 142.875 0)
+    (property "Reference" "C34" (id 0) (at 198.755 142.875 0)
       (effects (font (size 1.27 1.27)) (justify left))
     )
@@
   (symbol (lib_id "power:GND") (at 208.915 146.685 0) (unit 1)
     (in_bom yes) (on_board yes)
-    (property "Reference" "#PWR0104" (id 0) (at 208.915 153.035 0)
+    (property "Reference" "#PWR047" (id 0) (at 208.915 153.035 0)
       (effects (font (size 1.27 1.27)) hide)
     )
@@
   (symbol (lib_id "Connector_Generic:Conn_01x02") (at 80.01 118.11 180) (unit 1)
     (in_bom yes) (on_board yes) (fields_autoplaced)
-    (property "Reference" "J10" (id 0) (at 80.01 109.22 0))
+    (property "Reference" "J12" (id 0) (at 80.01 109.22 0))
     (property "Value" "TP4" (id 1) (at 80.01 111.76 0))
     (property "Footprint" "Connector_PinSocket_2.54mm:PinSocket_1x02_P2.54mm_Vertical" (id 2) (at 80.01 118.11 0)
@@
   (symbol (lib_id "Connector_Generic:Conn_01x02") (at 220.345 106.045 90) (unit 1)
     (in_bom yes) (on_board yes) (fields_autoplaced)
-    (property "Reference" "J8" (id 0) (at 226.06 104.7749 90)
+    (property "Reference" "J10" (id 0) (at 226.06 104.7749 90)
       (effects (font (size 1.27 1.27)) (justify right))
     )
@@
   (symbol (lib_id "Device:C") (at 260.35 148.59 180) (unit 1)
     (in_bom yes) (on_board yes)
-    (property "Reference" "C34" (id 0) (at 259.08 146.05 90))
+    (property "Reference" "C35" (id 0) (at 259.08 146.05 90))
     (property "Value" "100n" (id 1) (at 262.89 144.78 90))
     (property "Footprint" "Capacitor_SMD:C_1206_3216Metric" (id 2) (at 259.3848 144.78 0)
@@
   (symbol (lib_id "power:GND") (at 191.77 100.965 0) (unit 1)
     (in_bom yes) (on_board yes)
-    (property "Reference" "#PWR099" (id 0) (at 191.77 107.315 0)
+    (property "Reference" "#PWR034" (id 0) (at 191.77 107.315 0)
       (effects (font (size 1.27 1.27)) hide)
     )
@@
   (symbol (lib_id "power:GND") (at 118.11 116.84 0) (unit 1)
     (in_bom yes) (on_board yes) (fields_autoplaced)
-    (property "Reference" "#PWR024" (id 0) (at 118.11 123.19 0)
+    (property "Reference" "#PWR039" (id 0) (at 118.11 123.19 0)
       (effects (font (size 1.27 1.27)) hide)
     )
@@
   (symbol (lib_id "Connector_Generic:Conn_01x02") (at 206.375 141.605 90) (unit 1)
     (in_bom yes) (on_board yes) (fields_autoplaced)
-    (property "Reference" "J49" (id 0) (at 212.09 140.3349 90)
+    (property "Reference" "J13" (id 0) (at 212.09 140.3349 90)
       (effects (font (size 1.27 1.27)) (justify right))
     )
@@
   (symbol (lib_id "power:PWR_FLAG") (at 93.98 68.58 0) (unit 1)
     (in_bom yes) (on_board yes) (fields_autoplaced)
-    (property "Reference" "#FLG06" (id 0) (at 93.98 66.675 0)
+    (property "Reference" "#FLG07" (id 0) (at 93.98 66.675 0)
       (effects (font (size 1.27 1.27)) hide)
     )
@@
   (symbol (lib_id "power:GND") (at 256.54 137.16 90) (unit 1)
     (in_bom yes) (on_board yes) (fields_autoplaced)
-    (property "Reference" "#PWR030" (id 0) (at 262.89 137.16 0)
+    (property "Reference" "#PWR046" (id 0) (at 262.89 137.16 0)
       (effects (font (size 1.27 1.27)) hide)
     )
@@
   (symbol (lib_id "power:GND") (at 57.15 106.68 0) (unit 1)
     (in_bom yes) (on_board yes) (fields_autoplaced)
-    (property "Reference" "#PWR022" (id 0) (at 57.15 113.03 0)
+    (property "Reference" "#PWR036" (id 0) (at 57.15 113.03 0)
       (effects (font (size 1.27 1.27)) hide)
     )
@@
   (symbol (lib_id "power:GND") (at 86.995 118.11 0) (unit 1)
     (in_bom yes) (on_board yes)
-    (property "Reference" "#PWR0102" (id 0) (at 86.995 124.46 0)
+    (property "Reference" "#PWR041" (id 0) (at 86.995 124.46 0)
       (effects (font (size 1.27 1.27)) hide)
     )
@@
   (symbol (lib_id "Connector_Generic:Conn_01x02") (at 57.15 76.835 90) (unit 1)
     (in_bom yes) (on_board yes) (fields_autoplaced)
-    (property "Reference" "J6" (id 0) (at 62.23 75.5649 90)
+    (property "Reference" "J8" (id 0) (at 62.23 75.5649 90)
       (effects (font (size 1.27 1.27)) (justify right))
     )
@@
   (symbol (lib_id "Connector_Generic:Conn_01x02") (at 109.22 62.23 90) (unit 1)
     (in_bom yes) (on_board yes) (fields_autoplaced)
-    (property "Reference" "J4" (id 0) (at 114.3 60.9599 90)
+    (property "Reference" "J6" (id 0) (at 114.3 60.9599 90)
       (effects (font (size 1.27 1.27)) (justify right))
     )
@@
   (symbol (lib_id "Connector:Conn_Coaxial") (at 164.465 72.39 0) (unit 1)
     (in_bom yes) (on_board yes) (fields_autoplaced)
-    (property "Reference" "J5" (id 0) (at 167.64 71.4131 0)
+    (property "Reference" "J7" (id 0) (at 167.64 71.4131 0)
       (effects (font (size 1.27 1.27)) (justify left))
     )
@@
   (symbol (lib_id "power:GND") (at 111.76 66.675 0) (unit 1)
     (in_bom yes) (on_board yes)
-    (property "Reference" "#PWR097" (id 0) (at 111.76 73.025 0)
+    (property "Reference" "#PWR029" (id 0) (at 111.76 73.025 0)
       (effects (font (size 1.27 1.27)) hide)
     )
@@
   (symbol (lib_id "Connector_Generic:Conn_01x02") (at 189.23 95.885 90) (unit 1)
     (in_bom yes) (on_board yes) (fields_autoplaced)
-    (property "Reference" "J7" (id 0) (at 194.31 94.6149 90)
+    (property "Reference" "J9" (id 0) (at 194.31 94.6149 90)
       (effects (font (size 1.27 1.27)) (justify right))
     )
@@
   (symbol (lib_id "power:PWR_FLAG") (at 231.14 89.535 0) (unit 1)
     (in_bom yes) (on_board yes) (fields_autoplaced)
-    (property "Reference" "#FLG07" (id 0) (at 231.14 87.63 0)
+    (property "Reference" "#FLG08" (id 0) (at 231.14 87.63 0)
       (effects (font (size 1.27 1.27)) hide)
     )
@@
   (symbol (lib_id "power:GND") (at 254 118.11 0) (unit 1)
     (in_bom yes) (on_board yes)
-    (property "Reference" "#PWR026" (id 0) (at 254 124.46 0)
+    (property "Reference" "#PWR042" (id 0) (at 254 124.46 0)
       (effects (font (size 1.27 1.27)) hide)
     )
@@
   (symbol (lib_id "power:GND") (at 238.76 120.65 0) (unit 1)
     (in_bom yes) (on_board yes)
-    (property "Reference" "#PWR027" (id 0) (at 238.76 127 0)
+    (property "Reference" "#PWR043" (id 0) (at 238.76 127 0)
       (effects (font (size 1.27 1.27)) hide)
     )
@@
   (symbol (lib_id "Connector:Conn_Coaxial") (at 254 110.49 0) (unit 1)
     (in_bom yes) (on_board yes) (fields_autoplaced)
-    (property "Reference" "J9" (id 0) (at 256.54 109.5131 0)
+    (property "Reference" "J11" (id 0) (at 256.54 109.5131 0)
       (effects (font (size 1.27 1.27)) (justify left))
     )
@@
   (symbol (lib_id "power:GND") (at 222.885 111.125 0) (unit 1)
     (in_bom yes) (on_board yes)
-    (property "Reference" "#PWR0100" (id 0) (at 222.885 117.475 0)
+    (property "Reference" "#PWR037" (id 0) (at 222.885 117.475 0)
       (effects (font (size 1.27 1.27)) hide)
     )
@@
   (symbol (lib_id "power:GND") (at 147.32 113.03 0) (unit 1)
     (in_bom yes) (on_board yes) (fields_autoplaced)
-    (property "Reference" "#PWR023" (id 0) (at 147.32 119.38 0)
+    (property "Reference" "#PWR038" (id 0) (at 147.32 119.38 0)
       (effects (font (size 1.27 1.27)) hide)
     )
@@
   (symbol (lib_id "power:GND") (at 164.465 80.01 0) (unit 1)
     (in_bom yes) (on_board yes)
-    (property "Reference" "#PWR018" (id 0) (at 164.465 86.36 0)
+    (property "Reference" "#PWR030" (id 0) (at 164.465 86.36 0)
       (effects (font (size 1.27 1.27)) hide)
     )
@@
   (symbol (lib_id "power:GND") (at 161.29 129.54 0) (unit 1)
     (in_bom yes) (on_board yes) (fields_autoplaced)
-    (property "Reference" "#PWR028" (id 0) (at 161.29 135.89 0)
+    (property "Reference" "#PWR044" (id 0) (at 161.29 135.89 0)
       (effects (font (size 1.27 1.27)) hide)
     )
@@
   (symbol (lib_id "power:GND") (at 59.69 81.915 0) (unit 1)
     (in_bom yes) (on_board yes)
-    (property "Reference" "#PWR098" (id 0) (at 59.69 88.265 0)
+    (property "Reference" "#PWR032" (id 0) (at 59.69 88.265 0)
       (effects (font (size 1.27 1.27)) hide)
     )
@@
   (symbol (lib_id "power:GND") (at 136.525 82.55 0) (unit 1)
     (in_bom yes) (on_board yes)
-    (property "Reference" "#PWR020" (id 0) (at 136.525 88.9 0)
+    (property "Reference" "#PWR033" (id 0) (at 136.525 88.9 0)
       (effects (font (size 1.27 1.27)) hide)
     )
@@
   (symbol (lib_id "power:GND") (at 231.14 102.235 0) (unit 1)
     (in_bom yes) (on_board yes)
-    (property "Reference" "#PWR021" (id 0) (at 231.14 108.585 0)
+    (property "Reference" "#PWR035" (id 0) (at 231.14 108.585 0)
       (effects (font (size 1.27 1.27)) hide)
     )
@@
   (symbol (lib_id "power:GND") (at 48.26 118.11 0) (unit 1)
     (in_bom yes) (on_board yes) (fields_autoplaced)
-    (property "Reference" "#PWR025" (id 0) (at 48.26 124.46 0)
-      (effects (font (size 1.27 1.27)) hide)
-    )
+    (property "Reference" "#PWR040" (id 0) (at 48.26 124.46 0)
+      (effects (font (size 1.27 1.27)) hide)
+    )

Commit message: Update 24Mar23
Parts:
- added R77, R78: 50, Resistor_SMD:R_1206_3216Metric, symbol Device:R_US
Connections:
- net GND: now also R77.2, R78.2
- net at C32.1, R21.1, R22.1: now also R78.1
- net at C15.1, R17.1, R18.1: now also R77.1
Other:
- moved on the sheet: J11, R21, R22, R23

Commit message: Cleanup 8May23
Parts:
- R24: value 100R -> 100
- R77, R78: value 50 -> 51
- T1: value FT50-75 (18:7) -> FT50-43 (18:7)
- T2: value FT50-75 (7:18) -> FT50-43 (7:18)
Changed lines of the file:
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@@
       (effects (font (size 1.27 1.27)) (justify left))
     )
-    (property "Value" "50" (id 1) (at 233.68 115.5699 0)
+    (property "Value" "51" (id 1) (at 233.68 115.5699 0)
       (effects (font (size 1.27 1.27)) (justify left))
     )
@@
     (in_bom yes) (on_board yes) (fields_autoplaced)
     (property "Reference" "T1" (id 0) (at 106.6927 100.33 0))
-    (property "Value" "FT50-75 (18:7)" (id 1) (at 106.6927 102.87 0))
+    (property "Value" "FT50-43 (18:7)" (id 1) (at 106.6927 102.87 0))
     (property "Footprint" "Transformer_THT:Transformer_Toroid_Horizontal_D14.0mm_Amidon-T50" (id 2) (at 106.68 110.49 0)
       (effects (font (size 1.27 1.27)) hide)
@@
       (effects (font (size 1.27 1.27)) (justify left))
     )
-    (property "Value" "50" (id 1) (at 124.46 77.4699 0)
+    (property "Value" "51" (id 1) (at 124.46 77.4699 0)
       (effects (font (size 1.27 1.27)) (justify left))
     )
@@
     (in_bom yes) (on_board yes) (fields_autoplaced)
     (property "Reference" "T2" (id 0) (at 174.0027 111.76 0))
-    (property "Value" "FT50-75 (7:18)" (id 1) (at 174.0027 114.3 0))
+    (property "Value" "FT50-43 (7:18)" (id 1) (at 174.0027 114.3 0))
     (property "Footprint" "Transformer_THT:Transformer_Toroid_Horizontal_D14.0mm_Amidon-T50" (id 2) (at 173.99 121.92 0)
       (effects (font (size 1.27 1.27)) hide)
@@
       (effects (font (size 1.27 1.27)) (justify left))
     )
-    (property "Value" "100R" (id 1) (at 22.86 120.6499 0)
-      (effects (font (size 1.27 1.27)) (justify left))
-    )
+    (property "Value" "100" (id 1) (at 22.86 120.6499 0)
+      (effects (font (size 1.27 1.27)) (justify left))
+    )
