File: Phoenix612 Complete/Version 1.1/MicPreamp.kicad_sch (KiCad schematic)
At the start: 18 parts, among them J13 MICIN, Q2 2N3904

Commit message: Update 9Mar23
Parts:
- removed R40: 10K, Resistor_SMD:R_1206_3216Metric, symbol Device:R_US
- added J50: TP10, Connector_PinSocket_2.54mm:PinSocket_1x02_P2.54mm_Vertical, symbol Connector_Generic:Conn_01x02
Connections:
- net GND: now also J50.2 (Pin_2)
- net IFMICIN: now also J50.1 (Pin_1)
Changed lines of the file:
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@@
+    (stroke (width 0) (type default) (color 0 0 0 0))
+  )
+  (wire (pts (xy 150.495 83.82) (xy 150.495 92.075))
     (stroke (width 0) (type default) (color 0 0 0 0))
   )
@@
     (stroke (width 0) (type default) (color 0 0 0 0))
   )
-  (wire (pts (xy 90.17 114.935) (xy 90.17 112.395))
-    (stroke (width 0) (type default) (color 0 0 0 0))
-  )
   (wire (pts (xy 75.565 102.235) (xy 79.375 102.235))
     (stroke (width 0) (type default) (color 0 0 0 0))
@@
   )
   (wire (pts (xy 113.03 95.885) (xy 120.65 95.885))
-    (stroke (width 0) (type default) (color 0 0 0 0))
-  )
-  (wire (pts (xy 90.17 102.235) (xy 90.17 104.775))
     (stroke (width 0) (type default) (color 0 0 0 0))
   )
@@
     (pin "2")
   )
-  (symbol (lib_id "Device:R_US") (at 90.17 108.585 0) (unit 1)
-    (in_bom yes) (on_board yes) (fields_autoplaced)
-    (property "Reference" "R40" (id 0) (at 92.71 107.3149 0)
-      (effects (font (size 1.27 1.27)) (justify left))
-    )
-    (property "Value" "10K" (id 1) (at 92.71 109.8549 0)
-      (effects (font (size 1.27 1.27)) (justify left))
-    )
-    (property "Footprint" "Resistor_SMD:R_1206_3216Metric" (id 2) (at 91.186 108.839 90)
-      (effects (font (size 1.27 1.27)) hide)
-    )
-    (property "Datasheet" "~" (id 3) (at 90.17 108.585 0)
-      (effects (font (size 1.27 1.27)) hide)
-    )
-    (pin "1")
-    (pin "2")
-  )
   (symbol (lib_id "power:GND") (at 76.2 83.185 0) (unit 1)
     (in_bom yes) (on_board yes)
@@
     (pin "2")
   )
-  (symbol (lib_id "power:GND") (at 90.17 114.935 0) (unit 1)
-    (in_bom yes) (on_board yes)
-    (property "Reference" "#PWR050" (id 0) (at 90.17 121.285 0)
-      (effects (font (size 1.27 1.27)) hide)
-    )
-    (property "Value" "GND" (id 1) (at 90.17 118.745 0))
-    (property "Footprint" "" (id 2) (at 90.17 114.935 0)
-      (effects (font (size 1.27 1.27)) hide)
-    )
-    (property "Datasheet" "" (id 3) (at 90.17 114.935 0)
+  (symbol (lib_id "power:GND") (at 153.035 83.82 0) (unit 1)
+    (in_bom yes) (on_board yes)
+    (property "Reference" "#PWR0105" (id 0) (at 153.035 90.17 0)
+      (effects (font (size 1.27 1.27)) hide)
+    )
+    (property "Value" "GND" (id 1) (at 153.035 87.63 0))
+    (property "Footprint" "" (id 2) (at 153.035 83.82 0)
+      (effects (font (size 1.27 1.27)) hide)
+    )
+    (property "Datasheet" "" (id 3) (at 153.035 83.82 0)
       (effects (font (size 1.27 1.27)) hide)
     )
@@
     (pin "1")
   )
+  (symbol (lib_id "Connector_Generic:Conn_01x02") (at 150.495 78.74 90) (unit 1)
+    (in_bom yes) (on_board yes) (fields_autoplaced)
+    (property "Reference" "J50" (id 0) (at 156.21 77.4699 90)
+      (effects (font (size 1.27 1.27)) (justify right))
+    )
+    (property "Value" "TP10" (id 1) (at 156.21 80.0099 90)
+      (effects (font (size 1.27 1.27)) (justify right))
+    )
+    (property "Footprint" "Connector_PinSocket_2.54mm:PinSocket_1x02_P2.54mm_Vertical" (id 2) (at 150.495 78.74 0)
+      (effects (font (size 1.27 1.27)) hide)
+    )
+    (property "Datasheet" "~" (id 3) (at 150.495 78.74 0)
+      (effects (font (size 1.27 1.27)) hide)
+    )
+    (pin "1")
+    (pin "2")
+  )
   (symbol (lib_id "Device:C") (at 76.2 76.835 0) (unit 1)

Commit message: Update 17Mar23
Parts:
- renumbered C48 to C49, C49 to C50, C50 to C51, C51 to C52, C52 to C53, C53 to C54, C54 to C55, J50 to J16, J13 to J17
Changed lines of the file:
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@@
   (symbol (lib_id "Connector_Generic:Conn_01x02") (at 62.23 104.775 180) (unit 1)
     (in_bom yes) (on_board yes) (fields_autoplaced)
-    (property "Reference" "J13" (id 0) (at 62.23 95.25 0))
+    (property "Reference" "J17" (id 0) (at 62.23 95.25 0))
     (property "Value" "MICIN" (id 1) (at 62.23 97.79 0))
     (property "Footprint" "Connector_PinHeader_2.54mm:PinHeader_1x02_P2.54mm_Vertical" (id 2) (at 62.23 104.775 0)
@@
   (symbol (lib_id "power:GND") (at 67.31 107.315 0) (unit 1)
     (in_bom yes) (on_board yes)
-    (property "Reference" "#PWR047" (id 0) (at 67.31 113.665 0)
+    (property "Reference" "#PWR066" (id 0) (at 67.31 113.665 0)
       (effects (font (size 1.27 1.27)) hide)
     )
@@
   (symbol (lib_id "Device:C") (at 75.565 108.585 0) (unit 1)
     (in_bom yes) (on_board yes)
-    (property "Reference" "C54" (id 0) (at 76.835 111.125 90))
+    (property "Reference" "C55" (id 0) (at 76.835 111.125 90))
     (property "Value" "10n" (id 1) (at 73.66 111.76 90))
     (property "Footprint" "Capacitor_SMD:C_1206_3216Metric" (id 2) (at 76.5302 112.395 0)
@@
   (symbol (lib_id "power:GND") (at 76.2 83.185 0) (unit 1)
     (in_bom yes) (on_board yes)
-    (property "Reference" "#PWR045" (id 0) (at 76.2 89.535 0)
+    (property "Reference" "#PWR063" (id 0) (at 76.2 89.535 0)
       (effects (font (size 1.27 1.27)) hide)
     )
@@
   (symbol (lib_id "Device:C") (at 150.495 97.155 0) (unit 1)
     (in_bom yes) (on_board yes) (fields_autoplaced)
-    (property "Reference" "C52" (id 0) (at 153.67 95.8849 0)
+    (property "Reference" "C53" (id 0) (at 153.67 95.8849 0)
       (effects (font (size 1.27 1.27)) (justify left))
     )
@@
   (symbol (lib_id "power:GND") (at 153.035 83.82 0) (unit 1)
     (in_bom yes) (on_board yes)
-    (property "Reference" "#PWR0105" (id 0) (at 153.035 90.17 0)
+    (property "Reference" "#PWR064" (id 0) (at 153.035 90.17 0)
       (effects (font (size 1.27 1.27)) hide)
     )
@@
   (symbol (lib_id "Device:C_Polarized") (at 96.52 102.235 90) (unit 1)
     (in_bom yes) (on_board yes)
-    (property "Reference" "C53" (id 0) (at 93.98 99.695 0)
+    (property "Reference" "C54" (id 0) (at 93.98 99.695 0)
       (effects (font (size 1.27 1.27)) (justify left))
     )
@@
   (symbol (lib_id "power:GND") (at 142.24 99.06 0) (unit 1)
     (in_bom yes) (on_board yes)
-    (property "Reference" "#PWR046" (id 0) (at 142.24 105.41 0)
+    (property "Reference" "#PWR065" (id 0) (at 142.24 105.41 0)
       (effects (font (size 1.27 1.27)) hide)
     )
@@
   (symbol (lib_id "power:PWR_FLAG") (at 76.2 69.215 0) (unit 1)
     (in_bom yes) (on_board yes)
-    (property "Reference" "#FLG010" (id 0) (at 76.2 67.31 0)
+    (property "Reference" "#FLG011" (id 0) (at 76.2 67.31 0)
       (effects (font (size 1.27 1.27)) hide)
     )
@@
   (symbol (lib_id "Device:C_Polarized") (at 82.55 76.835 0) (unit 1)
     (in_bom yes) (on_board yes)
-    (property "Reference" "C50" (id 0) (at 85.09 74.295 0)
+    (property "Reference" "C51" (id 0) (at 85.09 74.295 0)
       (effects (font (size 1.27 1.27)) (justify left))
     )
@@
   (symbol (lib_id "power:GND") (at 150.495 112.395 0) (unit 1)
     (in_bom yes) (on_board yes) (fields_autoplaced)
-    (property "Reference" "#PWR049" (id 0) (at 150.495 118.745 0)
+    (property "Reference" "#PWR068" (id 0) (at 150.495 118.745 0)
       (effects (font (size 1.27 1.27)) hide)
     )
@@
   (symbol (lib_id "power:GND") (at 113.03 111.125 0) (unit 1)
     (in_bom yes) (on_board yes)
-    (property "Reference" "#PWR048" (id 0) (at 113.03 117.475 0)
+    (property "Reference" "#PWR067" (id 0) (at 113.03 117.475 0)
       (effects (font (size 1.27 1.27)) hide)
     )
@@
   (symbol (lib_id "Device:C") (at 69.85 76.835 0) (unit 1)
     (in_bom yes) (on_board yes)
-    (property "Reference" "C48" (id 0) (at 71.12 74.295 0)
+    (property "Reference" "C49" (id 0) (at 71.12 74.295 0)
       (effects (font (size 1.27 1.27)) (justify left))
     )
@@
   (symbol (lib_id "power:GND") (at 75.565 115.57 0) (unit 1)
     (in_bom yes) (on_board yes)
-    (property "Reference" "#PWR051" (id 0) (at 75.565 121.92 0)
+    (property "Reference" "#PWR069" (id 0) (at 75.565 121.92 0)
       (effects (font (size 1.27 1.27)) hide)
     )
@@
   (symbol (lib_id "Connector_Generic:Conn_01x02") (at 150.495 78.74 90) (unit 1)
     (in_bom yes) (on_board yes) (fields_autoplaced)
-    (property "Reference" "J50" (id 0) (at 156.21 77.4699 90)
+    (property "Reference" "J16" (id 0) (at 156.21 77.4699 90)
       (effects (font (size 1.27 1.27)) (justify right))
     )
@@
   (symbol (lib_id "Device:C") (at 76.2 76.835 0) (unit 1)
     (in_bom yes) (on_board yes)
-    (property "Reference" "C49" (id 0) (at 77.47 74.295 0)
+    (property "Reference" "C50" (id 0) (at 77.47 74.295 0)
       (effects (font (size 1.27 1.27)) (justify left))
     )
@@
   (symbol (lib_id "Device:C_Polarized") (at 124.46 95.885 90) (unit 1)
     (in_bom yes) (on_board yes)
-    (property "Reference" "C51" (id 0) (at 121.92 93.345 0)
-      (effects (font (size 1.27 1.27)) (justify left))
-    )
+    (property "Reference" "C52" (id 0) (at 121.92 93.345 0)
+      (effects (font (size 1.27 1.27)) (justify left))
+    )

Commit message: Update 24Mar23
Parts:
- renumbered RV4 to MG1
Connections:
- net GND: now also MG1.1; no longer MG1.3
- net at C52.2: now also MG1.3; no longer MG1.1
Other:
- moved on the sheet: MG1
Changed lines of the file:
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@@
   (junction (at 82.55 71.755) (diameter 0) (color 0 0 0 0)
   )
+  (junction (at 142.24 95.885) (diameter 0) (color 0 0 0 0)
+  )
   (junction (at 76.2 81.915) (diameter 0) (color 0 0 0 0)
   )
@@
     (stroke (width 0) (type default) (color 0 0 0 0))
   )
-  (wire (pts (xy 134.62 92.075) (xy 150.495 92.075))
-    (stroke (width 0) (type default) (color 0 0 0 0))
-  )
   (wire (pts (xy 76.2 71.755) (xy 76.2 73.025))
     (stroke (width 0) (type default) (color 0 0 0 0))
@@
     (stroke (width 0) (type default) (color 0 0 0 0))
   )
+  (wire (pts (xy 142.24 95.885) (xy 142.875 95.885))
+    (stroke (width 0) (type default) (color 0 0 0 0))
+  )
   (wire (pts (xy 67.31 102.235) (xy 75.565 102.235))
     (stroke (width 0) (type default) (color 0 0 0 0))
@@
     (stroke (width 0) (type default) (color 0 0 0 0))
   )
+  (wire (pts (xy 75.565 102.235) (xy 79.375 102.235))
+    (stroke (width 0) (type default) (color 0 0 0 0))
+  )
+  (wire (pts (xy 105.41 102.235) (xy 103.505 102.235))
+    (stroke (width 0) (type default) (color 0 0 0 0))
+  )
+  (wire (pts (xy 69.85 80.645) (xy 69.85 81.915))
+    (stroke (width 0) (type default) (color 0 0 0 0))
+  )
+  (wire (pts (xy 76.2 81.915) (xy 76.2 80.645))
+    (stroke (width 0) (type default) (color 0 0 0 0))
+  )
+  (wire (pts (xy 113.03 95.885) (xy 113.03 97.155))
+    (stroke (width 0) (type default) (color 0 0 0 0))
+  )
+  (wire (pts (xy 76.2 81.915) (xy 82.55 81.915))
+    (stroke (width 0) (type default) (color 0 0 0 0))
+  )
+  (wire (pts (xy 67.31 107.315) (xy 67.31 104.775))
+    (stroke (width 0) (type default) (color 0 0 0 0))
+  )
+  (wire (pts (xy 75.565 102.235) (xy 75.565 104.775))
+    (stroke (width 0) (type default) (color 0 0 0 0))
+  )
+  (wire (pts (xy 113.03 85.09) (xy 113.03 95.885))
+    (stroke (width 0) (type default) (color 0 0 0 0))
+  )
+  (wire (pts (xy 90.17 71.755) (xy 90.17 76.835))
+    (stroke (width 0) (type default) (color 0 0 0 0))
+  )
+  (wire (pts (xy 90.17 84.455) (xy 90.17 102.235))
+    (stroke (width 0) (type default) (color 0 0 0 0))
+  )
+  (wire (pts (xy 76.2 69.215) (xy 76.2 71.755))
+    (stroke (width 0) (type default) (color 0 0 0 0))
+  )
+  (wire (pts (xy 90.17 71.755) (xy 113.03 71.755))
+    (stroke (width 0) (type default) (color 0 0 0 0))
+  )
+  (wire (pts (xy 113.03 95.885) (xy 120.65 95.885))
+    (stroke (width 0) (type default) (color 0 0 0 0))
+  )
+  (wire (pts (xy 136.525 92.075) (xy 150.495 92.075))
+    (stroke (width 0) (type default) (color 0 0 0 0))
+  )
+  (wire (pts (xy 82.55 71.755) (xy 82.55 73.025))
+    (stroke (width 0) (type default) (color 0 0 0 0))
+  )
+  (wire (pts (xy 134.62 99.695) (xy 136.525 99.695))
+    (stroke (width 0) (type default) (color 0 0 0 0))
+  )
+  (wire (pts (xy 103.505 95.885) (xy 103.505 102.235))
+    (stroke (width 0) (type default) (color 0 0 0 0))
+  )
+  (wire (pts (xy 86.995 102.235) (xy 90.17 102.235))
+    (stroke (width 0) (type default) (color 0 0 0 0))
+  )
+  (wire (pts (xy 92.71 102.235) (xy 90.17 102.235))
+    (stroke (width 0) (type default) (color 0 0 0 0))
+  )
+  (wire (pts (xy 69.85 71.755) (xy 76.2 71.755))
+    (stroke (width 0) (type default) (color 0 0 0 0))
+  )
+  (wire (pts (xy 150.495 92.075) (xy 166.37 92.075))
+    (stroke (width 0) (type default) (color 0 0 0 0))
+  )
+  (wire (pts (xy 75.565 115.57) (xy 75.565 112.395))
+    (stroke (width 0) (type default) (color 0 0 0 0))
+  )
+  (wire (pts (xy 69.85 81.915) (xy 76.2 81.915))
+    (stroke (width 0) (type default) (color 0 0 0 0))
+  )
+  (wire (pts (xy 136.525 99.695) (xy 136.525 92.075))
+    (stroke (width 0) (type default) (color 0 0 0 0))
+  )
   (wire (pts (xy 138.43 95.885) (xy 142.24 95.885))
     (stroke (width 0) (type default) (color 0 0 0 0))
   )
-  (wire (pts (xy 75.565 102.235) (xy 79.375 102.235))
-    (stroke (width 0) (type default) (color 0 0 0 0))
-  )
-  (wire (pts (xy 105.41 102.235) (xy 103.505 102.235))
-    (stroke (width 0) (type default) (color 0 0 0 0))
-  )
-  (wire (pts (xy 69.85 80.645) (xy 69.85 81.915))
-    (stroke (width 0) (type default) (color 0 0 0 0))
-  )
-  (wire (pts (xy 76.2 81.915) (xy 76.2 80.645))
-    (stroke (width 0) (type default) (color 0 0 0 0))
-  )
-  (wire (pts (xy 113.03 95.885) (xy 113.03 97.155))
-    (stroke (width 0) (type default) (color 0 0 0 0))
-  )
-  (wire (pts (xy 76.2 81.915) (xy 82.55 81.915))
-    (stroke (width 0) (type default) (color 0 0 0 0))
-  )
-  (wire (pts (xy 67.31 107.315) (xy 67.31 104.775))
-    (stroke (width 0) (type default) (color 0 0 0 0))
-  )
-  (wire (pts (xy 75.565 102.235) (xy 75.565 104.775))
-    (stroke (width 0) (type default) (color 0 0 0 0))
-  )
-  (wire (pts (xy 113.03 85.09) (xy 113.03 95.885))
-    (stroke (width 0) (type default) (color 0 0 0 0))
-  )
-  (wire (pts (xy 90.17 71.755) (xy 90.17 76.835))
-    (stroke (width 0) (type default) (color 0 0 0 0))
-  )
-  (wire (pts (xy 90.17 84.455) (xy 90.17 102.235))
-    (stroke (width 0) (type default) (color 0 0 0 0))
-  )
-  (wire (pts (xy 76.2 69.215) (xy 76.2 71.755))
-    (stroke (width 0) (type default) (color 0 0 0 0))
-  )
-  (wire (pts (xy 90.17 71.755) (xy 113.03 71.755))
-    (stroke (width 0) (type default) (color 0 0 0 0))
-  )
-  (wire (pts (xy 113.03 95.885) (xy 120.65 95.885))
-    (stroke (width 0) (type default) (color 0 0 0 0))
-  )
-  (wire (pts (xy 82.55 71.755) (xy 82.55 73.025))
-    (stroke (width 0) (type default) (color 0 0 0 0))
-  )
-  (wire (pts (xy 103.505 95.885) (xy 103.505 102.235))
-    (stroke (width 0) (type default) (color 0 0 0 0))
-  )
-  (wire (pts (xy 86.995 102.235) (xy 90.17 102.235))
-    (stroke (width 0) (type default) (color 0 0 0 0))
-  )
-  (wire (pts (xy 92.71 102.235) (xy 90.17 102.235))
-    (stroke (width 0) (type default) (color 0 0 0 0))
-  )
-  (wire (pts (xy 69.85 71.755) (xy 76.2 71.755))
-    (stroke (width 0) (type default) (color 0 0 0 0))
-  )
-  (wire (pts (xy 130.81 95.885) (xy 128.27 95.885))
-    (stroke (width 0) (type default) (color 0 0 0 0))
-  )
-  (wire (pts (xy 150.495 92.075) (xy 166.37 92.075))
-    (stroke (width 0) (type default) (color 0 0 0 0))
-  )
-  (wire (pts (xy 75.565 115.57) (xy 75.565 112.395))
-    (stroke (width 0) (type default) (color 0 0 0 0))
-  )
-  (wire (pts (xy 69.85 81.915) (xy 76.2 81.915))
-    (stroke (width 0) (type default) (color 0 0 0 0))
-  )
   (wire (pts (xy 76.2 81.915) (xy 76.2 83.185))
     (stroke (width 0) (type default) (color 0 0 0 0))
   )
   (wire (pts (xy 105.41 95.885) (xy 103.505 95.885))
+    (stroke (width 0) (type default) (color 0 0 0 0))
+  )
+  (wire (pts (xy 128.27 95.885) (xy 130.81 95.885))
     (stroke (width 0) (type default) (color 0 0 0 0))
   )
@@
     (pin "2")
   )
-  (symbol (lib_id "Device:R_Potentiometer_Trim") (at 134.62 95.885 90) (unit 1)
-    (in_bom yes) (on_board yes) (fields_autoplaced)
-    (property "Reference" "RV4" (id 0) (at 134.62 99.06 90))
-    (property "Value" "10K" (id 1) (at 134.62 101.6 90))
+  (symbol (lib_id "Device:R_Potentiometer_Trim") (at 134.62 95.885 270) (unit 1)
+    (in_bom yes) (on_board yes) (fields_autoplaced)
+    (property "Reference" "MG1" (id 0) (at 134.62 90.17 90))
+    (property "Value" "10K" (id 1) (at 134.62 92.71 90))
     (property "Footprint" "Potentiometer_THT:Potentiometer_Bourns_3296W_Vertical" (id 2) (at 134.62 95.885 0)
       (effects (font (size 1.27 1.27)) hide)

Commit message: Cleanup 8May23
Parts:
- R38: value 220 -> 220K
- R39: value 10R -> 10
Changed lines of the file:
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@@
     (in_bom yes) (on_board yes) (fields_autoplaced)
     (property "Reference" "R38" (id 0) (at 109.22 90.17 90))
-    (property "Value" "220" (id 1) (at 109.22 92.71 90))
+    (property "Value" "220K" (id 1) (at 109.22 92.71 90))
     (property "Footprint" "Resistor_SMD:R_1206_3216Metric" (id 2) (at 109.474 94.869 90)
       (effects (font (size 1.27 1.27)) hide)
@@
       (effects (font (size 1.27 1.27)) (justify right))
     )
-    (property "Value" "10R" (id 1) (at 152.4 107.9499 0)
+    (property "Value" "10" (id 1) (at 152.4 107.9499 0)
       (effects (font (size 1.27 1.27)) (justify right))
     )
