File: Phoenix612 Complete/Version 1.1/PA_Driver.kicad_sch (KiCad schematic)
At the start: 23 parts, among them J16 TP, J17 TP, U10 OPA2674

Commit message: Update 9Mar23
Parts:
- removed J16, J17: TP, Connector_PinHeader_1.00mm:PinHeader_1x01_P1.00mm_Vertical, symbol Connector_Generic:Conn_01x01
- added J16: TP13, Connector_PinSocket_2.54mm:PinSocket_1x02_P2.54mm_Vertical, symbol Connector_Generic:Conn_01x02
- added J17: TP14, Connector_PinSocket_2.54mm:PinSocket_1x02_P2.54mm_Vertical, symbol Connector_Generic:Conn_01x02
- R54, R55: value 10K -> 1K
Connections:
- net GND: now also J16.2 (Pin_2), J17.2 (Pin_2)
- net PA_IN: now also J17.1 (Pin_1)
- net at C63.2, R49.1: now also J16.1 (Pin_1)
Changed lines of the file:
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@@
   (junction (at 216.535 105.41) (diameter 0) (color 0 0 0 0)
   )
+  (junction (at 127 60.96) (diameter 0) (color 0 0 0 0)
+  )
   (junction (at 171.45 62.865) (diameter 0) (color 0 0 0 0)
   )
@@
   )
   (junction (at 174.625 106.68) (diameter 0) (color 0 0 0 0)
-  )
-  (junction (at 127 60.96) (diameter 0) (color 0 0 0 0)
   )
   (no_connect (at 105.0178 69.2257))
@@
     (stroke (width 0) (type default) (color 0 0 0 0))
   )
+  (wire (pts (xy 127 44.45) (xy 127 60.96))
+    (stroke (width 0) (type default) (color 0 0 0 0))
+  )
   (wire (pts (xy 198.755 99.06) (xy 198.755 105.41))
     (stroke (width 0) (type default) (color 0 0 0 0))
@@
   )
   (wire (pts (xy 187.96 128.905) (xy 175.26 128.905))
+    (stroke (width 0) (type default) (color 0 0 0 0))
+  )
+  (wire (pts (xy 171.45 47.625) (xy 171.45 62.865))
     (stroke (width 0) (type default) (color 0 0 0 0))
   )
@@
       (effects (font (size 1.27 1.27)) (justify left))
     )
-    (property "Value" "10K" (id 1) (at 167.64 95.8849 0)
+    (property "Value" "1K" (id 1) (at 167.64 95.8849 0)
       (effects (font (size 1.27 1.27)) (justify left))
     )
@@
     (pin "2")
   )
+  (symbol (lib_id "power:GND") (at 173.99 47.625 0) (unit 1)
+    (in_bom yes) (on_board yes)
+    (property "Reference" "#PWR0109" (id 0) (at 173.99 53.975 0)
+      (effects (font (size 1.27 1.27)) hide)
+    )
+    (property "Value" "GND" (id 1) (at 173.99 51.435 0))
+    (property "Footprint" "" (id 2) (at 173.99 47.625 0)
+      (effects (font (size 1.27 1.27)) hide)
+    )
+    (property "Datasheet" "" (id 3) (at 173.99 47.625 0)
+      (effects (font (size 1.27 1.27)) hide)
+    )
+    (pin "1")
+  )
   (symbol (lib_id "Device:C_Polarized") (at 229.235 118.745 0) (unit 1)
     (in_bom yes) (on_board yes) (fields_autoplaced)
@@
     (pin "2")
   )
-  (symbol (lib_id "Connector_Generic:Conn_01x01") (at 127 55.88 90) (unit 1)
-    (in_bom yes) (on_board yes) (fields_autoplaced)
-    (property "Reference" "J16" (id 0) (at 129.54 54.6099 90)
-      (effects (font (size 1.27 1.27)) (justify right))
-    )
-    (property "Value" "TP" (id 1) (at 129.54 57.1499 90)
-      (effects (font (size 1.27 1.27)) (justify right))
-    )
-    (property "Footprint" "Connector_PinHeader_1.00mm:PinHeader_1x01_P1.00mm_Vertical" (id 2) (at 127 55.88 0)
-      (effects (font (size 1.27 1.27)) hide)
-    )
-    (property "Datasheet" "~" (id 3) (at 127 55.88 0)
-      (effects (font (size 1.27 1.27)) hide)
-    )
-    (pin "1")
-  )
   (symbol (lib_id "power:GND") (at 74.93 73.025 0) (unit 1)
     (in_bom yes) (on_board yes) (fields_autoplaced)
@@
     (pin "1")
   )
-  (symbol (lib_id "Connector_Generic:Conn_01x01") (at 171.45 57.785 90) (unit 1)
-    (in_bom yes) (on_board yes) (fields_autoplaced)
-    (property "Reference" "J17" (id 0) (at 173.99 56.5149 90)
+  (symbol (lib_id "Device:R_US") (at 207.01 93.345 0) (unit 1)
+    (in_bom yes) (on_board yes) (fields_autoplaced)
+    (property "Reference" "R53" (id 0) (at 209.55 92.0749 0)
+      (effects (font (size 1.27 1.27)) (justify left))
+    )
+    (property "Value" "5.6" (id 1) (at 209.55 94.6149 0)
+      (effects (font (size 1.27 1.27)) (justify left))
+    )
+    (property "Footprint" "Resistor_SMD:R_1206_3216Metric" (id 2) (at 208.026 93.599 90)
+      (effects (font (size 1.27 1.27)) hide)
+    )
+    (property "Datasheet" "~" (id 3) (at 207.01 93.345 0)
+      (effects (font (size 1.27 1.27)) hide)
+    )
+    (pin "1")
+    (pin "2")
+  )
+  (symbol (lib_id "Connector_Generic:Conn_01x02") (at 171.45 42.545 90) (unit 1)
+    (in_bom yes) (on_board yes) (fields_autoplaced)
+    (property "Reference" "J17" (id 0) (at 176.53 41.2749 90)
       (effects (font (size 1.27 1.27)) (justify right))
     )
-    (property "Value" "TP" (id 1) (at 173.99 59.0549 90)
+    (property "Value" "TP14" (id 1) (at 176.53 43.8149 90)
       (effects (font (size 1.27 1.27)) (justify right))
     )
-    (property "Footprint" "Connector_PinHeader_1.00mm:PinHeader_1x01_P1.00mm_Vertical" (id 2) (at 171.45 57.785 0)
-      (effects (font (size 1.27 1.27)) hide)
-    )
-    (property "Datasheet" "~" (id 3) (at 171.45 57.785 0)
-      (effects (font (size 1.27 1.27)) hide)
-    )
-    (pin "1")
-  )
-  (symbol (lib_id "Device:R_US") (at 207.01 93.345 0) (unit 1)
-    (in_bom yes) (on_board yes) (fields_autoplaced)
-    (property "Reference" "R53" (id 0) (at 209.55 92.0749 0)
-      (effects (font (size 1.27 1.27)) (justify left))
-    )
-    (property "Value" "5.6" (id 1) (at 209.55 94.6149 0)
-      (effects (font (size 1.27 1.27)) (justify left))
-    )
-    (property "Footprint" "Resistor_SMD:R_1206_3216Metric" (id 2) (at 208.026 93.599 90)
-      (effects (font (size 1.27 1.27)) hide)
-    )
-    (property "Datasheet" "~" (id 3) (at 207.01 93.345 0)
+    (property "Footprint" "Connector_PinSocket_2.54mm:PinSocket_1x02_P2.54mm_Vertical" (id 2) (at 171.45 42.545 0)
+      (effects (font (size 1.27 1.27)) hide)
+    )
+    (property "Datasheet" "~" (id 3) (at 171.45 42.545 0)
       (effects (font (size 1.27 1.27)) hide)
     )
@@
     (pin "2")
   )
+  (symbol (lib_id "Connector_Generic:Conn_01x02") (at 127 39.37 90) (unit 1)
+    (in_bom yes) (on_board yes) (fields_autoplaced)
+    (property "Reference" "J16" (id 0) (at 132.08 38.0999 90)
+      (effects (font (size 1.27 1.27)) (justify right))
+    )
+    (property "Value" "TP13" (id 1) (at 132.08 40.6399 90)
+      (effects (font (size 1.27 1.27)) (justify right))
+    )
+    (property "Footprint" "Connector_PinSocket_2.54mm:PinSocket_1x02_P2.54mm_Vertical" (id 2) (at 127 39.37 0)
+      (effects (font (size 1.27 1.27)) hide)
+    )
+    (property "Datasheet" "~" (id 3) (at 127 39.37 0)
+      (effects (font (size 1.27 1.27)) hide)
+    )
+    (pin "1")
+    (pin "2")
+  )
   (symbol (lib_id "Device:R_US") (at 157.48 118.745 0) (unit 1)
     (in_bom yes) (on_board yes) (fields_autoplaced)
@@
       (effects (font (size 1.27 1.27)) (justify left))
     )
-    (property "Value" "10K" (id 1) (at 160.02 120.0149 0)
+    (property "Value" "1K" (id 1) (at 160.02 120.0149 0)
       (effects (font (size 1.27 1.27)) (justify left))
     )
@@
       (effects (font (size 1.27 1.27)) hide)
     )
+    (pin "1")
+  )
+  (symbol (lib_id "power:GND") (at 129.54 44.45 0) (unit 1)
+    (in_bom yes) (on_board yes)
+    (property "Reference" "#PWR0108" (id 0) (at 129.54 50.8 0)
+      (effects (font (size 1.27 1.27)) hide)
+    )
+    (property "Value" "GND" (id 1) (at 129.54 48.26 0))
+    (property "Footprint" "" (id 2) (at 129.54 44.45 0)
+      (effects (font (size 1.27 1.27)) hide)
+    )
+    (property "Datasheet" "" (id 3) (at 129.54 44.45 0)
+      (effects (font (size 1.27 1.27)) hide)
+    )

Commit message: Update 17Mar23
Parts:
- renumbered C63 to C64, C64 to C65, C65 to C66, C66 to C67, C67 to C68, C68 to C69, C69 to C70, C70 to C71, C71 to C72, J16 to J20, J17 to J21, R47 to R46, R48 to R47, R49 to R48, R50 to R49, R51 to R50, R52 to R51, R53 to R52, R54 to R53, R55 to R54
Changed lines of the file:
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@@
   (symbol (lib_id "Device:C") (at 207.01 119.38 0) (unit 1)
     (in_bom yes) (on_board yes) (fields_autoplaced)
-    (property "Reference" "C67" (id 0) (at 210.82 118.1099 0)
+    (property "Reference" "C68" (id 0) (at 210.82 118.1099 0)
       (effects (font (size 1.27 1.27)) (justify left))
     )
@@
   (symbol (lib_id "Device:R_US") (at 165.735 94.615 0) (unit 1)
     (in_bom yes) (on_board yes) (fields_autoplaced)
-    (property "Reference" "R54" (id 0) (at 167.64 93.3449 0)
+    (property "Reference" "R53" (id 0) (at 167.64 93.3449 0)
       (effects (font (size 1.27 1.27)) (justify left))
     )
@@
   (symbol (lib_id "Device:C") (at 68.58 63.5 90) (unit 1)
     (in_bom yes) (on_board yes)
-    (property "Reference" "C64" (id 0) (at 66.04 62.23 0)
+    (property "Reference" "C65" (id 0) (at 66.04 62.23 0)
       (effects (font (size 1.27 1.27)) (justify left))
     )
@@
   (symbol (lib_id "Device:C") (at 165.735 120.65 0) (unit 1)
     (in_bom yes) (on_board yes) (fields_autoplaced)
-    (property "Reference" "C70" (id 0) (at 168.91 119.3799 0)
+    (property "Reference" "C71" (id 0) (at 168.91 119.3799 0)
       (effects (font (size 1.27 1.27)) (justify left))
     )
@@
   (symbol (lib_id "Device:R_US") (at 74.93 69.215 180) (unit 1)
     (in_bom yes) (on_board yes) (fields_autoplaced)
-    (property "Reference" "R50" (id 0) (at 76.835 67.9449 0)
+    (property "Reference" "R49" (id 0) (at 76.835 67.9449 0)
       (effects (font (size 1.27 1.27)) (justify right))
     )
@@
   (symbol (lib_id "Device:R_US") (at 102.235 74.93 90) (unit 1)
     (in_bom yes) (on_board yes)
-    (property "Reference" "R52" (id 0) (at 100.965 77.47 90))
+    (property "Reference" "R51" (id 0) (at 100.965 77.47 90))
     (property "Value" "1K" (id 1) (at 104.775 77.47 90))
     (property "Footprint" "Resistor_SMD:R_1206_3216Metric" (id 2) (at 102.489 73.914 90)
@@
   (symbol (lib_id "power:GND") (at 173.99 47.625 0) (unit 1)
     (in_bom yes) (on_board yes)
-    (property "Reference" "#PWR0109" (id 0) (at 173.99 53.975 0)
+    (property "Reference" "#PWR080" (id 0) (at 173.99 53.975 0)
       (effects (font (size 1.27 1.27)) hide)
     )
@@
   (symbol (lib_id "Device:C_Polarized") (at 229.235 118.745 0) (unit 1)
     (in_bom yes) (on_board yes) (fields_autoplaced)
-    (property "Reference" "C66" (id 0) (at 232.41 116.5859 0)
+    (property "Reference" "C67" (id 0) (at 232.41 116.5859 0)
       (effects (font (size 1.27 1.27)) (justify left))
     )
@@
   (symbol (lib_id "Device:C") (at 175.26 120.65 0) (unit 1)
     (in_bom yes) (on_board yes) (fields_autoplaced)
-    (property "Reference" "C71" (id 0) (at 179.07 119.3799 0)
+    (property "Reference" "C72" (id 0) (at 179.07 119.3799 0)
       (effects (font (size 1.27 1.27)) (justify left))
     )
@@
   (symbol (lib_id "Device:R_US") (at 134.62 65.405 90) (unit 1)
     (in_bom yes) (on_board yes)
-    (property "Reference" "R49" (id 0) (at 131.445 67.31 90))
+    (property "Reference" "R48" (id 0) (at 131.445 67.31 90))
     (property "Value" "100" (id 1) (at 137.795 67.31 90))
     (property "Footprint" "Resistor_SMD:R_1206_3216Metric" (id 2) (at 134.874 64.389 90)
@@
   (symbol (lib_id "Device:R_US") (at 88.9 63.5 90) (unit 1)
     (in_bom yes) (on_board yes) (fields_autoplaced)
-    (property "Reference" "R48" (id 0) (at 88.9 57.15 90))
+    (property "Reference" "R47" (id 0) (at 88.9 57.15 90))
     (property "Value" "100" (id 1) (at 88.9 59.69 90))
     (property "Footprint" "Resistor_SMD:R_1206_3216Metric" (id 2) (at 89.154 62.484 90)
@@
   (symbol (lib_id "power:GND") (at 165.735 141.605 0) (unit 1)
     (in_bom yes) (on_board yes) (fields_autoplaced)
-    (property "Reference" "#PWR062" (id 0) (at 165.735 147.955 0)
+    (property "Reference" "#PWR084" (id 0) (at 165.735 147.955 0)
       (effects (font (size 1.27 1.27)) hide)
     )
@@
   (symbol (lib_id "Device:C_Polarized") (at 187.96 120.015 0) (unit 1)
     (in_bom yes) (on_board yes) (fields_autoplaced)
-    (property "Reference" "C69" (id 0) (at 191.77 117.8559 0)
+    (property "Reference" "C70" (id 0) (at 191.77 117.8559 0)
       (effects (font (size 1.27 1.27)) (justify left))
     )
@@
   (symbol (lib_id "power:GND") (at 74.93 73.025 0) (unit 1)
     (in_bom yes) (on_board yes) (fields_autoplaced)
-    (property "Reference" "#PWR059" (id 0) (at 74.93 79.375 0)
+    (property "Reference" "#PWR081" (id 0) (at 74.93 79.375 0)
       (effects (font (size 1.27 1.27)) hide)
     )
@@
   (symbol (lib_id "Device:R_US") (at 207.01 93.345 0) (unit 1)
     (in_bom yes) (on_board yes) (fields_autoplaced)
-    (property "Reference" "R53" (id 0) (at 209.55 92.0749 0)
+    (property "Reference" "R52" (id 0) (at 209.55 92.0749 0)
       (effects (font (size 1.27 1.27)) (justify left))
     )
@@
   (symbol (lib_id "Connector_Generic:Conn_01x02") (at 171.45 42.545 90) (unit 1)
     (in_bom yes) (on_board yes) (fields_autoplaced)
-    (property "Reference" "J17" (id 0) (at 176.53 41.2749 90)
+    (property "Reference" "J21" (id 0) (at 176.53 41.2749 90)
       (effects (font (size 1.27 1.27)) (justify right))
     )
@@
   (symbol (lib_id "Device:C") (at 216.535 119.38 0) (unit 1)
     (in_bom yes) (on_board yes) (fields_autoplaced)
-    (property "Reference" "C68" (id 0) (at 220.345 118.1099 0)
+    (property "Reference" "C69" (id 0) (at 220.345 118.1099 0)
       (effects (font (size 1.27 1.27)) (justify left))
     )
@@
   (symbol (lib_id "Connector_Generic:Conn_01x02") (at 127 39.37 90) (unit 1)
     (in_bom yes) (on_board yes) (fields_autoplaced)
-    (property "Reference" "J16" (id 0) (at 132.08 38.0999 90)
+    (property "Reference" "J20" (id 0) (at 132.08 38.0999 90)
       (effects (font (size 1.27 1.27)) (justify right))
     )
@@
   (symbol (lib_id "Device:R_US") (at 157.48 118.745 0) (unit 1)
     (in_bom yes) (on_board yes) (fields_autoplaced)
-    (property "Reference" "R55" (id 0) (at 160.02 117.4749 0)
+    (property "Reference" "R54" (id 0) (at 160.02 117.4749 0)
       (effects (font (size 1.27 1.27)) (justify left))
     )
@@
   (symbol (lib_id "Device:C") (at 80.01 63.5 90) (unit 1)
     (in_bom yes) (on_board yes)
-    (property "Reference" "C65" (id 0) (at 77.47 62.23 0)
+    (property "Reference" "C66" (id 0) (at 77.47 62.23 0)
       (effects (font (size 1.27 1.27)) (justify left))
     )
@@
   (symbol (lib_id "power:GND") (at 248.92 127 0) (unit 1)
     (in_bom yes) (on_board yes) (fields_autoplaced)
-    (property "Reference" "#PWR060" (id 0) (at 248.92 133.35 0)
+    (property "Reference" "#PWR082" (id 0) (at 248.92 133.35 0)
       (effects (font (size 1.27 1.27)) hide)
     )
@@
   (symbol (lib_id "power:GND") (at 129.54 44.45 0) (unit 1)
     (in_bom yes) (on_board yes)
-    (property "Reference" "#PWR0108" (id 0) (at 129.54 50.8 0)
+    (property "Reference" "#PWR079" (id 0) (at 129.54 50.8 0)
       (effects (font (size 1.27 1.27)) hide)
     )
@@
   (symbol (lib_id "Device:R_US") (at 167.005 62.865 90) (unit 1)
     (in_bom yes) (on_board yes) (fields_autoplaced)
-    (property "Reference" "R47" (id 0) (at 167.005 56.515 90))
+    (property "Reference" "R46" (id 0) (at 167.005 56.515 90))
     (property "Value" "5.6R" (id 1) (at 167.005 59.055 90))
     (property "Footprint" "Resistor_SMD:R_1206_3216Metric" (id 2) (at 167.259 61.849 90)
@@
   (symbol (lib_id "Device:R_US") (at 149.86 73.66 90) (unit 1)
     (in_bom yes) (on_board yes)
-    (property "Reference" "R51" (id 0) (at 147.32 76.2 90))
+    (property "Reference" "R50" (id 0) (at 147.32 76.2 90))
     (property "Value" "1K" (id 1) (at 153.035 76.2 90))
     (property "Footprint" "Resistor_SMD:R_1206_3216Metric" (id 2) (at 150.114 72.644 90)
@@
   (symbol (lib_id "power:PWR_FLAG") (at 215.9 102.235 0) (unit 1)
     (in_bom yes) (on_board yes)
-    (property "Reference" "#FLG012" (id 0) (at 215.9 100.33 0)
+    (property "Reference" "#FLG013" (id 0) (at 215.9 100.33 0)
       (effects (font (size 1.27 1.27)) hide)
     )
@@
   (symbol (lib_id "Device:C") (at 120.65 60.96 90) (unit 1)
     (in_bom yes) (on_board yes)
-    (property "Reference" "C63" (id 0) (at 118.11 59.69 0)
+    (property "Reference" "C64" (id 0) (at 118.11 59.69 0)
       (effects (font (size 1.27 1.27)) (justify left))
     )
@@
   (symbol (lib_id "power:GND") (at 207.01 140.335 0) (unit 1)
     (in_bom yes) (on_board yes) (fields_autoplaced)
-    (property "Reference" "#PWR061" (id 0) (at 207.01 146.685 0)
+    (property "Reference" "#PWR083" (id 0) (at 207.01 146.685 0)
       (effects (font (size 1.27 1.27)) hide)
     )
@@
   (symbol (lib_id "power:PWR_FLAG") (at 174.625 103.505 0) (unit 1)
     (in_bom yes) (on_board yes)
-    (property "Reference" "#FLG013" (id 0) (at 174.625 101.6 0)
-      (effects (font (size 1.27 1.27)) hide)
-    )
+    (property "Reference" "#FLG014" (id 0) (at 174.625 101.6 0)
+      (effects (font (size 1.27 1.27)) hide)
+    )

Commit message: Cleanup 8May23
Parts:
- R46: value 5.6R -> 5.6
- R49: value 50 -> 51
Changed lines of the file:
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@@
   (symbol (lib_id "Device:R_US") (at 74.93 69.215 180) (unit 1)
     (in_bom yes) (on_board yes) (fields_autoplaced)
-    (property "Reference" "R49" (id 0) (at 76.835 67.9449 0)
-      (effects (font (size 1.27 1.27)) (justify right))
-    )
-    (property "Value" "50" (id 1) (at 76.835 70.4849 0)
+    (property "Reference" "R49" (id 0) (at 77.47 67.9449 0)
+      (effects (font (size 1.27 1.27)) (justify right))
+    )
+    (property "Value" "51" (id 1) (at 77.47 70.4849 0)
       (effects (font (size 1.27 1.27)) (justify right))
     )
@@
   (symbol (lib_id "Device:R_US") (at 167.005 62.865 90) (unit 1)
     (in_bom yes) (on_board yes) (fields_autoplaced)
-    (property "Reference" "R46" (id 0) (at 167.005 56.515 90))
-    (property "Value" "5.6R" (id 1) (at 167.005 59.055 90))
+    (property "Reference" "R46" (id 0) (at 167.005 57.15 90))
+    (property "Value" "5.6" (id 1) (at 167.005 59.69 90))
     (property "Footprint" "Resistor_SMD:R_1206_3216Metric" (id 2) (at 167.259 61.849 90)
       (effects (font (size 1.27 1.27)) hide)
