File: Phoenix612 Complete/Version 1.1/PA_Preamp.kicad_sch (KiCad schematic)
At the start: 28 parts, among them J18 TP11, J19 TP12, J58 JMP, U8 LT1253, U9 QPR_Filter

Commit message: Update 24Mar23
Parts:
- added L17: 20u, Inductor_SMD:L_1206_3216Metric, symbol Device:L
- renumbered RV5 to TXG1
Connections:
- net TX12V: now also L17.1; no longer R40.1
- net at R44.1, U8.2 (InA-): now also TXG1.3; no longer TXG1.1
- net at R45.1, TXG1.2: now also TXG1.1; no longer TXG1.3
- new net: L17.2, R40.1
Other:
- moved on the sheet: TXG1
Changed lines of the file:
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@@
   (junction (at 103.505 92.71) (diameter 0) (color 0 0 0 0)
   )
+  (junction (at 229.87 45.72) (diameter 0) (color 0 0 0 0)
+  )
+  (junction (at 154.94 123.19) (diameter 0) (color 0 0 0 0)
+  )
+  (junction (at 217.17 45.72) (diameter 0) (color 0 0 0 0)
+  )
   (junction (at 154.94 110.49) (diameter 0) (color 0 0 0 0)
   )
-  (junction (at 229.87 45.72) (diameter 0) (color 0 0 0 0)
-  )
-  (junction (at 217.17 45.72) (diameter 0) (color 0 0 0 0)
-  )
-  (junction (at 154.94 123.19) (diameter 0) (color 0 0 0 0)
-  )
   (junction (at 215.9 113.665) (diameter 0) (color 0 0 0 0)
   )
@@
     (stroke (width 0) (type default) (color 0 0 0 0))
   )
+  (wire (pts (xy 154.94 123.19) (xy 154.94 124.46))
+    (stroke (width 0) (type default) (color 0 0 0 0))
+  )
   (wire (pts (xy 152.4 60.96) (xy 161.29 60.96))
     (stroke (width 0) (type default) (color 0 0 0 0))
@@
     (stroke (width 0) (type default) (color 0 0 0 0))
   )
-  (wire (pts (xy 160.02 119.38) (xy 160.02 123.19))
-    (stroke (width 0) (type default) (color 0 0 0 0))
-  )
   (wire (pts (xy 208.28 99.06) (xy 208.28 111.125))
     (stroke (width 0) (type default) (color 0 0 0 0))
@@
     (stroke (width 0) (type default) (color 0 0 0 0))
   )
-  (wire (pts (xy 152.4 49.53) (xy 152.4 52.07))
+  (wire (pts (xy 152.4 34.29) (xy 152.4 40.005))
     (stroke (width 0) (type default) (color 0 0 0 0))
   )
@@
     (stroke (width 0) (type default) (color 0 0 0 0))
   )
+  (wire (pts (xy 152.4 47.625) (xy 152.4 52.07))
+    (stroke (width 0) (type default) (color 0 0 0 0))
+  )
   (wire (pts (xy 217.17 41.275) (xy 217.17 45.72))
     (stroke (width 0) (type default) (color 0 0 0 0))
@@
     (stroke (width 0) (type default) (color 0 0 0 0))
   )
+  (wire (pts (xy 149.225 123.19) (xy 149.225 118.11))
+    (stroke (width 0) (type default) (color 0 0 0 0))
+  )
   (wire (pts (xy 152.4 60.96) (xy 152.4 63.5))
     (stroke (width 0) (type default) (color 0 0 0 0))
@@
     (stroke (width 0) (type default) (color 0 0 0 0))
   )
-  (wire (pts (xy 158.75 119.38) (xy 160.02 119.38))
-    (stroke (width 0) (type default) (color 0 0 0 0))
-  )
   (wire (pts (xy 215.9 113.665) (xy 215.9 115.57))
     (stroke (width 0) (type default) (color 0 0 0 0))
@@
     (stroke (width 0) (type default) (color 0 0 0 0))
   )
+  (wire (pts (xy 154.94 110.49) (xy 154.94 114.3))
+    (stroke (width 0) (type default) (color 0 0 0 0))
+  )
   (wire (pts (xy 79.375 83.82) (xy 83.185 83.82))
     (stroke (width 0) (type default) (color 0 0 0 0))
@@
     (stroke (width 0) (type default) (color 0 0 0 0))
   )
-  (wire (pts (xy 154.94 123.19) (xy 160.02 123.19))
+  (wire (pts (xy 154.94 121.92) (xy 154.94 123.19))
     (stroke (width 0) (type default) (color 0 0 0 0))
   )
@@
     (stroke (width 0) (type default) (color 0 0 0 0))
   )
-  (wire (pts (xy 154.94 110.49) (xy 154.94 115.57))
+  (wire (pts (xy 149.225 118.11) (xy 151.13 118.11))
     (stroke (width 0) (type default) (color 0 0 0 0))
   )
@@
     (stroke (width 0) (type default) (color 0 0 0 0))
   )
-  (wire (pts (xy 154.94 123.19) (xy 154.94 124.46))
-    (stroke (width 0) (type default) (color 0 0 0 0))
-  )
   (wire (pts (xy 113.665 97.79) (xy 111.125 97.79))
     (stroke (width 0) (type default) (color 0 0 0 0))
@@
   )
   (wire (pts (xy 229.87 45.72) (xy 240.665 45.72))
+    (stroke (width 0) (type default) (color 0 0 0 0))
+  )
+  (wire (pts (xy 154.94 123.19) (xy 149.225 123.19))
     (stroke (width 0) (type default) (color 0 0 0 0))
   )
@@
     )
   )
-  (global_label "TX12V" (shape output) (at 152.4 49.53 90) (fields_autoplaced)
+  (global_label "TX12V" (shape output) (at 152.4 34.29 90) (fields_autoplaced)
     (effects (font (size 1.27 1.27)) (justify left))
-    (property "Intersheet References" "${INTERSHEET_REFS}" (id 0) (at 152.3206 41.4321 90)
+    (property "Intersheet References" "${INTERSHEET_REFS}" (id 0) (at 152.3206 26.1921 90)
       (effects (font (size 1.27 1.27)) (justify left) hide)
     )
@@
     (pin "1")
   )
-  (symbol (lib_id "Device:R_Potentiometer_Trim") (at 154.94 119.38 0) (unit 1)
-    (in_bom yes) (on_board yes) (fields_autoplaced)
-    (property "Reference" "RV5" (id 0) (at 152.4 118.1099 0)
+  (symbol (lib_id "Device:R_Potentiometer_Trim") (at 154.94 118.11 180) (unit 1)
+    (in_bom yes) (on_board yes) (fields_autoplaced)
+    (property "Reference" "TXG1" (id 0) (at 157.48 116.8399 0)
       (effects (font (size 1.27 1.27)) (justify right))
     )
-    (property "Value" "10K" (id 1) (at 152.4 120.6499 0)
+    (property "Value" "10K" (id 1) (at 157.48 119.3799 0)
       (effects (font (size 1.27 1.27)) (justify right))
     )
-    (property "Footprint" "Potentiometer_THT:Potentiometer_Bourns_3296W_Vertical" (id 2) (at 154.94 119.38 0)
-      (effects (font (size 1.27 1.27)) hide)
-    )
-    (property "Datasheet" "~" (id 3) (at 154.94 119.38 0)
+    (property "Footprint" "Potentiometer_THT:Potentiometer_Bourns_3296W_Vertical" (id 2) (at 154.94 118.11 0)
+      (effects (font (size 1.27 1.27)) hide)
+    )
+    (property "Datasheet" "~" (id 3) (at 154.94 118.11 0)
       (effects (font (size 1.27 1.27)) hide)
     )
@@
     (pin "3")
   )
+  (symbol (lib_id "Device:L") (at 152.4 43.815 0) (unit 1)
+    (in_bom yes) (on_board yes) (fields_autoplaced)
+    (property "Reference" "L17" (id 0) (at 153.67 42.5449 0)
+      (effects (font (size 1.27 1.27)) (justify left))
+    )
+    (property "Value" "20u" (id 1) (at 153.67 45.0849 0)
+      (effects (font (size 1.27 1.27)) (justify left))
+    )
+    (property "Footprint" "Inductor_SMD:L_1206_3216Metric" (id 2) (at 152.4 43.815 0)
+      (effects (font (size 1.27 1.27)) hide)
+    )
+    (property "Datasheet" "~" (id 3) (at 152.4 43.815 0)
+      (effects (font (size 1.27 1.27)) hide)
+    )
+    (pin "1")
+    (pin "2")
+  )
   (symbol (lib_id "Device:C") (at 146.05 92.71 90) (unit 1)

Commit message: Cleanup 8May23
Parts:
- R76: value 50R -> 51
- TR2: value T50-22:4 -> T50-43 (22:4)
- TXG1: value 10K -> 1K
Changed lines of the file:
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@@
       (effects (font (size 1.27 1.27)) (justify right))
     )
-    (property "Value" "10K" (id 1) (at 157.48 119.3799 0)
+    (property "Value" "1K" (id 1) (at 157.48 119.3799 0)
       (effects (font (size 1.27 1.27)) (justify right))
     )
@@
     (in_bom yes) (on_board yes)
     (property "Reference" "TR2" (id 0) (at 85.725 82.55 0))
-    (property "Value" "T50-22:4" (id 1) (at 85.725 80.01 0))
+    (property "Value" "T50-43 (22:4)" (id 1) (at 85.725 80.01 0))
     (property "Footprint" "Custom_RF:T50-1Tap-Close" (id 2) (at 90.805 80.01 0)
       (effects (font (size 1.27 1.27)) hide)
@@
     (in_bom yes) (on_board yes) (fields_autoplaced)
     (property "Reference" "R76" (id 0) (at 223.52 92.71 90))
-    (property "Value" "50R" (id 1) (at 223.52 95.25 90))
+    (property "Value" "51" (id 1) (at 223.52 95.25 90))
     (property "Footprint" "Resistor_SMD:R_1206_3216Metric" (id 2) (at 223.774 98.044 90)
       (effects (font (size 1.27 1.27)) hide)
