File: Phoenix612 Complete/Version 1.1/Phoenix612 Complete v1.1.kicad_sch (KiCad schematic)
At the start: 0 parts

Commit message: Update_17Mar23
Parts:
- added H1, H2, H3, H4: MountingHole, MountingHole:MountingHole_3.2mm_M3_ISO7380_Pad_TopBottom, symbol Mechanical:MountingHole
Connections:
- new net GND: H1.1, H2.1, H3.1, H4.1
Changed lines of the file:
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@@
     (company "DATER (Dave Peter)")
+  )
+  (symbol (lib_name "MountingHole_1") (lib_id "Mechanical:MountingHole") (at 139.065 38.735 0) (unit 1)
+    (in_bom no) (on_board yes) (fields_autoplaced)
+    (property "Reference" "H3" (id 0) (at 142.24 37.4649 0)
+      (effects (font (size 1.27 1.27)) (justify left) hide)
+    )
+    (property "Value" "MountingHole" (id 1) (at 142.24 40.0049 0)
+      (effects (font (size 1.27 1.27)) (justify left) hide)
+    )
+    (property "Footprint" "MountingHole:MountingHole_3.2mm_M3_ISO7380_Pad_TopBottom" (id 2) (at 139.065 38.735 0)
+      (effects (font (size 1.27 1.27)) hide)
+    )
+    (property "Datasheet" "~" (id 3) (at 139.065 38.735 0)
+      (effects (font (size 1.27 1.27)) hide)
+    )
+    (pin "1")
+  )
+  (symbol (lib_name "MountingHole_1") (lib_id "Mechanical:MountingHole") (at 128.905 38.735 0) (unit 1)
+    (in_bom no) (on_board yes) (fields_autoplaced)
+    (property "Reference" "H1" (id 0) (at 132.08 37.4649 0)
+      (effects (font (size 1.27 1.27)) (justify left) hide)
+    )
+    (property "Value" "MountingHole" (id 1) (at 132.08 40.0049 0)
+      (effects (font (size 1.27 1.27)) (justify left) hide)
+    )
+    (property "Footprint" "MountingHole:MountingHole_3.2mm_M3_ISO7380_Pad_TopBottom" (id 2) (at 128.905 38.735 0)
+      (effects (font (size 1.27 1.27)) hide)
+    )
+    (property "Datasheet" "~" (id 3) (at 128.905 38.735 0)
+      (effects (font (size 1.27 1.27)) hide)
+    )
+    (pin "1")
+  )
+  (symbol (lib_id "power:GND") (at 128.905 42.545 0) (unit 1)
+    (in_bom yes) (on_board yes)
+    (property "Reference" "#PWR0114" (id 0) (at 128.905 48.895 0)
+      (effects (font (size 1.27 1.27)) hide)
+    )
+    (property "Value" "GND" (id 1) (at 128.905 46.355 0))
+    (property "Footprint" "" (id 2) (at 128.905 42.545 0)
+      (effects (font (size 1.27 1.27)) hide)
+    )
+    (property "Datasheet" "" (id 3) (at 128.905 42.545 0)
+      (effects (font (size 1.27 1.27)) hide)
+    )
+    (pin "1")
+  )
+  (symbol (lib_id "power:GND") (at 133.985 42.545 0) (unit 1)
+    (in_bom yes) (on_board yes)
+    (property "Reference" "#PWR0115" (id 0) (at 133.985 48.895 0)
+      (effects (font (size 1.27 1.27)) hide)
+    )
+    (property "Value" "GND" (id 1) (at 133.985 46.355 0))
+    (property "Footprint" "" (id 2) (at 133.985 42.545 0)
+      (effects (font (size 1.27 1.27)) hide)
+    )
+    (property "Datasheet" "" (id 3) (at 133.985 42.545 0)
+      (effects (font (size 1.27 1.27)) hide)
+    )
+    (pin "1")
+  )
+  (symbol (lib_id "power:GND") (at 139.065 42.545 0) (unit 1)
+    (in_bom yes) (on_board yes)
+    (property "Reference" "#PWR0116" (id 0) (at 139.065 48.895 0)
+      (effects (font (size 1.27 1.27)) hide)
+    )
+    (property "Value" "GND" (id 1) (at 139.065 46.355 0))
+    (property "Footprint" "" (id 2) (at 139.065 42.545 0)
+      (effects (font (size 1.27 1.27)) hide)
+    )
+    (property "Datasheet" "" (id 3) (at 139.065 42.545 0)
+      (effects (font (size 1.27 1.27)) hide)
+    )
+    (pin "1")
+  )
+  (symbol (lib_name "MountingHole_1") (lib_id "Mechanical:MountingHole") (at 133.985 38.735 0) (unit 1)
+    (in_bom no) (on_board yes) (fields_autoplaced)
+    (property "Reference" "H2" (id 0) (at 137.16 37.4649 0)
+      (effects (font (size 1.27 1.27)) (justify left) hide)
+    )
+    (property "Value" "MountingHole" (id 1) (at 137.16 40.0049 0)
+      (effects (font (size 1.27 1.27)) (justify left) hide)
+    )
+    (property "Footprint" "MountingHole:MountingHole_3.2mm_M3_ISO7380_Pad_TopBottom" (id 2) (at 133.985 38.735 0)
+      (effects (font (size 1.27 1.27)) hide)
+    )
+    (property "Datasheet" "~" (id 3) (at 133.985 38.735 0)
+      (effects (font (size 1.27 1.27)) hide)
+    )
+    (pin "1")
+  )
+  (symbol (lib_id "power:GND") (at 124.46 42.545 0) (unit 1)
+    (in_bom yes) (on_board yes)
+    (property "Reference" "#PWR0113" (id 0) (at 124.46 48.895 0)
+      (effects (font (size 1.27 1.27)) hide)
+    )
+    (property "Value" "GND" (id 1) (at 124.46 46.355 0))
+    (property "Footprint" "" (id 2) (at 124.46 42.545 0)
+      (effects (font (size 1.27 1.27)) hide)
+    )
+    (property "Datasheet" "" (id 3) (at 124.46 42.545 0)
+      (effects (font (size 1.27 1.27)) hide)
+    )
+    (pin "1")
+  )
+  (symbol (lib_name "MountingHole_1") (lib_id "Mechanical:MountingHole") (at 124.46 38.735 0) (unit 1)
+    (in_bom no) (on_board yes) (fields_autoplaced)
+    (property "Reference" "H4" (id 0) (at 127.635 37.4649 0)
+      (effects (font (size 1.27 1.27)) (justify left) hide)
+    )
+    (property "Value" "MountingHole" (id 1) (at 127.635 40.0049 0)
+      (effects (font (size 1.27 1.27)) (justify left) hide)
+    )
+    (property "Footprint" "MountingHole:MountingHole_3.2mm_M3_ISO7380_Pad_TopBottom" (id 2) (at 124.46 38.735 0)
+      (effects (font (size 1.27 1.27)) hide)
+    )
+    (property "Datasheet" "~" (id 3) (at 124.46 38.735 0)
+      (effects (font (size 1.27 1.27)) hide)
+    )
+    (pin "1")
   )
   (sheet (at 114.3 95.25) (size 26.035 25.4) (fields_autoplaced)
@@
       (reference "#FLG015") (unit 1) (value "PWR_FLAG") (footprint "")
     )
+    (path "/f41cfc14-3798-49af-aac9-12db59c92150/5b2b98df-baf9-417d-889d-f4e3fc6eefb6"
+      (reference "#FLG016") (unit 1) (value "PWR_FLAG") (footprint "")
+    )
     (path "/7d624223-b511-4648-87bb-11892eb59d0f/d75a90ae-ed96-4fbe-996a-da4f16a54bf5"
       (reference "#PWR01") (unit 1) (value "GND") (footprint "")
@@
       (reference "#PWR09") (unit 1) (value "GND") (footprint "")
     )
-    (path "/f41cfc14-3798-49af-aac9-12db59c92150/236f5b18-23b0-474a-87e3-df8f656a853f"
+    (path "/f41cfc14-3798-49af-aac9-12db59c92150/7938c5f4-a303-4487-bf65-bbc6d79847be"
       (reference "#PWR010") (unit 1) (value "GND") (footprint "")
     )
@@
       (reference "#PWR0111") (unit 1) (value "GND") (footprint "")
     )
+    (path "/f41cfc14-3798-49af-aac9-12db59c92150/cf73ad07-6350-49c6-a0da-cdcb2d76db36"
+      (reference "#PWR0112") (unit 1) (value "GND") (footprint "")
+    )
+    (path "/dfac9206-b3b5-4114-ba6e-5710a8071b72"
+      (reference "#PWR0113") (unit 1) (value "GND") (footprint "")
+    )
+    (path "/9998bb65-79dd-47af-854e-962db52c0ea8"
+      (reference "#PWR0114") (unit 1) (value "GND") (footprint "")
+    )
+    (path "/a304b2df-b9c5-4a7f-8af3-dbd8c93a3761"
+      (reference "#PWR0115") (unit 1) (value "GND") (footprint "")
+    )
+    (path "/ac8a7885-58a6-40ec-97a9-0456b7806cc0"
+      (reference "#PWR0116") (unit 1) (value "GND") (footprint "")
+    )
     (path "/7d624223-b511-4648-87bb-11892eb59d0f/0c9f0e84-c3db-485c-a06a-351786b5713d"
       (reference "C1") (unit 1) (value "10n") (footprint "Capacitor_SMD:C_1206_3216Metric")
@@
     )
     (path "/d0cc8f58-fbb9-405a-9672-436f64e1806a/30fe963b-31d3-4c63-89f1-29a29457ecbe"
-      (reference "C100") (unit 1) (value "100n") (footprint "Capacitor_SMD:C_1206_3216Metric")
+      (reference "C100") (unit 1) (value "10u") (footprint "Capacitor_SMD:C_1206_3216Metric")
     )
     (path "/f41cfc14-3798-49af-aac9-12db59c92150/e90351f7-3590-4b89-b864-4af65324d423"
-      (reference "D1") (unit 1) (value "1N4001") (footprint "Diode_THT:D_DO-41_SOD81_P10.16mm_Horizontal")
+      (reference "D1") (unit 1) (value "1N5817") (footprint "Diode_THT:D_DO-41_SOD81_P10.16mm_Horizontal")
     )
     (path "/f41cfc14-3798-49af-aac9-12db59c92150/fdede4dc-8ffa-4dbd-a8d3-046e7b9a25c4"
@@
       (reference "D12") (unit 1) (value "1N4148") (footprint "Diode_THT:D_DO-35_SOD27_P7.62mm_Horizontal")
     )
+    (path "/5d612b1f-03db-4104-aadc-f417809bf5bc"
+      (reference "H1") (unit 1) (value "MountingHole") (footprint "MountingHole:MountingHole_3.2mm_M3_ISO7380_Pad_TopBottom")
+    )
+    (path "/b58c70b2-e05b-4e26-93b4-8eada62f0e62"
+      (reference "H2") (unit 1) (value "MountingHole") (footprint "MountingHole:MountingHole_3.2mm_M3_ISO7380_Pad_TopBottom")
+    )
+    (path "/0952cdc8-120b-4a57-9ea5-969be49a0604"
+      (reference "H3") (unit 1) (value "MountingHole") (footprint "MountingHole:MountingHole_3.2mm_M3_ISO7380_Pad_TopBottom")
+    )
+    (path "/e0d6b27c-82b6-42bc-bdf8-c695d85ac920"
+      (reference "H4") (unit 1) (value "MountingHole") (footprint "MountingHole:MountingHole_3.2mm_M3_ISO7380_Pad_TopBottom")
+    )
     (path "/7d624223-b511-4648-87bb-11892eb59d0f/e5454615-aa92-4770-a749-925acdc333a4"
       (reference "J1") (unit 1) (value "TP1") (footprint "Connector_PinSocket_2.54mm:PinSocket_1x02_P2.54mm_Vertical")
     )
-    (path "/f41cfc14-3798-49af-aac9-12db59c92150/bc58939b-737d-4ae0-a0a5-42f7139961ab"
+    (path "/f41cfc14-3798-49af-aac9-12db59c92150/2456f523-372c-4c6b-823b-d6932b042407"
       (reference "J2") (unit 1) (value "PWR") (footprint "Connector_PinHeader_2.54mm:PinHeader_1x03_P2.54mm_Vertical")
     )
@@
       (reference "J50") (unit 1) (value "TP10") (footprint "Connector_PinSocket_2.54mm:PinSocket_1x02_P2.54mm_Vertical")
     )
+    (path "/f41cfc14-3798-49af-aac9-12db59c92150/333b52e8-096f-4d03-8ac3-0a8b9628c70b"
+      (reference "J51") (unit 1) (value "VCC") (footprint "Connector_BarrelJack:BarrelJack_GCT_DCJ200-10-A_Horizontal")
+    )
     (path "/f41cfc14-3798-49af-aac9-12db59c92150/00db175b-0fe8-4dd7-a896-7872ad3e4927"

Commit message: Update 17Mar23
Parts:
- added H5, H6, H7, H8: MountingHole, MountingHole:MountingHole_3.2mm_M3_ISO7380_Pad_TopBottom, symbol Mechanical:MountingHole
- renumbered H4 to H1, H1 to H2, H2 to H3, H3 to H4
Connections:
- net GND: now also H5.1, H6.1, H7.1, H8.1
