File: Phoenix612 Complete/Version 1.1/RF_amp.kicad_sch (KiCad schematic)
At the start: 27 parts, among them J1 TP, U1 LT1253, U2 QPR_Filter

Commit message: Update 9Mar23
Parts:
- removed J1: TP, Connector_PinHeader_1.00mm:PinHeader_1x01_P1.00mm_Vertical, symbol Connector_Generic:Conn_01x01
- added J1: TP1, Connector_PinSocket_2.54mm:PinSocket_1x02_P2.54mm_Vertical, symbol Connector_Generic:Conn_01x02
- added J48: TP2, Connector_PinSocket_2.54mm:PinSocket_1x02_P2.54mm_Vertical, symbol Connector_Generic:Conn_01x02
- RV1, RV2: value 10K -> 1K
Connections:
- net GND: now also J1.2 (Pin_2), J48.2 (Pin_2)
- net IFRFIN: now also J48.1 (Pin_1)
- net at R5.2, U1.5 (InB+): now also J1.1 (Pin_1)
Changed lines of the file:
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@@
   (junction (at 81.28 129.54) (diameter 0) (color 0 0 0 0)
   )
-  (junction (at 119.38 102.87) (diameter 0) (color 0 0 0 0)
-  )
   (junction (at 78.74 67.31) (diameter 0) (color 0 0 0 0)
   )
@@
   (junction (at 128.27 129.54) (diameter 0) (color 0 0 0 0)
   )
+  (junction (at 118.745 102.87) (diameter 0) (color 0 0 0 0)
+  )
   (junction (at 180.34 118.11) (diameter 0) (color 0 0 0 0)
   )
+  (junction (at 224.155 105.41) (diameter 0) (color 0 0 0 0)
+  )
   (junction (at 148.59 106.68) (diameter 0) (color 0 0 0 0)
   )
@@
     (stroke (width 0) (type default) (color 0 0 0 0))
   )
+  (wire (pts (xy 118.745 95.885) (xy 118.745 102.87))
+    (stroke (width 0) (type default) (color 0 0 0 0))
+  )
   (wire (pts (xy 118.11 81.28) (xy 143.51 81.28))
     (stroke (width 0) (type default) (color 0 0 0 0))
@@
     (stroke (width 0) (type default) (color 0 0 0 0))
   )
-  (wire (pts (xy 226.695 105.41) (xy 221.615 105.41))
+  (wire (pts (xy 234.95 105.41) (xy 224.155 105.41))
     (stroke (width 0) (type default) (color 0 0 0 0))
   )
@@
     (stroke (width 0) (type default) (color 0 0 0 0))
   )
+  (wire (pts (xy 224.155 105.41) (xy 221.615 105.41))
+    (stroke (width 0) (type default) (color 0 0 0 0))
+  )
   (wire (pts (xy 95.885 79.375) (xy 95.885 77.47))
     (stroke (width 0) (type default) (color 0 0 0 0))
   )
+  (wire (pts (xy 224.155 95.25) (xy 224.155 105.41))
+    (stroke (width 0) (type default) (color 0 0 0 0))
+  )
   (wire (pts (xy 86.36 125.73) (xy 86.36 129.54))
     (stroke (width 0) (type default) (color 0 0 0 0))
   )
-  (wire (pts (xy 119.38 102.87) (xy 129.54 102.87))
+  (wire (pts (xy 113.03 102.87) (xy 118.745 102.87))
     (stroke (width 0) (type default) (color 0 0 0 0))
   )
@@
     (stroke (width 0) (type default) (color 0 0 0 0))
   )
+  (wire (pts (xy 118.745 102.87) (xy 129.54 102.87))
+    (stroke (width 0) (type default) (color 0 0 0 0))
+  )
   (wire (pts (xy 180.34 115.57) (xy 180.34 118.11))
     (stroke (width 0) (type default) (color 0 0 0 0))
@@
   )
   (wire (pts (xy 67.31 67.31) (xy 67.31 70.485))
-    (stroke (width 0) (type default) (color 0 0 0 0))
-  )
-  (wire (pts (xy 113.03 102.87) (xy 119.38 102.87))
     (stroke (width 0) (type default) (color 0 0 0 0))
   )
@@
     (effects (font (size 1.27 1.27)) (justify left bottom))
   )
-  (global_label "IFRFIN" (shape input) (at 226.695 105.41 0) (fields_autoplaced)
+  (global_label "IFRFIN" (shape input) (at 234.95 105.41 0) (fields_autoplaced)
     (effects (font (size 1.27 1.27)) (justify left))
-    (property "Intersheet References" "${INTERSHEET_REFS}" (id 0) (at 235.0952 105.4894 0)
+    (property "Intersheet References" "${INTERSHEET_REFS}" (id 0) (at 243.3502 105.4894 0)
       (effects (font (size 1.27 1.27)) (justify left) hide)
     )
@@
       (effects (font (size 1.27 1.27)) (justify right))
     )
-    (property "Value" "10K" (id 1) (at 125.73 126.9999 0)
+    (property "Value" "1K" (id 1) (at 125.73 126.9999 0)
       (effects (font (size 1.27 1.27)) (justify right))
     )
@@
     (pin "3")
   )
-  (symbol (lib_id "Connector_Generic:Conn_01x01") (at 119.38 97.79 90) (unit 1)
-    (in_bom yes) (on_board yes) (fields_autoplaced)
-    (property "Reference" "J1" (id 0) (at 121.92 96.5199 90)
-      (effects (font (size 1.27 1.27)) (justify right))
-    )
-    (property "Value" "TP" (id 1) (at 121.92 99.0599 90)
-      (effects (font (size 1.27 1.27)) (justify right))
-    )
-    (property "Footprint" "Connector_PinHeader_1.00mm:PinHeader_1x01_P1.00mm_Vertical" (id 2) (at 119.38 97.79 0)
-      (effects (font (size 1.27 1.27)) hide)
-    )
-    (property "Datasheet" "~" (id 3) (at 119.38 97.79 0)
-      (effects (font (size 1.27 1.27)) hide)
-    )
-    (pin "1")
-  )
   (symbol (lib_id "Device:R_US") (at 78.74 73.66 0) (unit 1)
     (in_bom yes) (on_board yes) (fields_autoplaced)
@@
     (pin "1")
     (pin "2")
+  )
+  (symbol (lib_id "power:GND") (at 121.285 95.885 0) (unit 1)
+    (in_bom yes) (on_board yes) (fields_autoplaced)
+    (property "Reference" "#PWR0101" (id 0) (at 121.285 102.235 0)
+      (effects (font (size 1.27 1.27)) hide)
+    )
+    (property "Value" "GND" (id 1) (at 121.285 100.965 0))
+    (property "Footprint" "" (id 2) (at 121.285 95.885 0)
+      (effects (font (size 1.27 1.27)) hide)
+    )
+    (property "Datasheet" "" (id 3) (at 121.285 95.885 0)
+      (effects (font (size 1.27 1.27)) hide)
+    )
+    (pin "1")
   )
   (symbol (lib_id "Device:C") (at 167.64 106.68 90) (unit 1)
@@
     (pin "1")
   )
+  (symbol (lib_id "Connector_Generic:Conn_01x02") (at 224.155 90.17 90) (unit 1)
+    (in_bom yes) (on_board yes) (fields_autoplaced)
+    (property "Reference" "J48" (id 0) (at 229.87 88.8999 90)
+      (effects (font (size 1.27 1.27)) (justify right))
+    )
+    (property "Value" "TP2" (id 1) (at 229.87 91.4399 90)
+      (effects (font (size 1.27 1.27)) (justify right))
+    )
+    (property "Footprint" "Connector_PinSocket_2.54mm:PinSocket_1x02_P2.54mm_Vertical" (id 2) (at 224.155 90.17 0)
+      (effects (font (size 1.27 1.27)) hide)
+    )
+    (property "Datasheet" "~" (id 3) (at 224.155 90.17 0)
+      (effects (font (size 1.27 1.27)) hide)
+    )
+    (pin "1")
+    (pin "2")
+  )
   (symbol (lib_id "power:GND") (at 143.51 83.82 0) (unit 1)
     (in_bom yes) (on_board yes) (fields_autoplaced)
@@
       (effects (font (size 1.27 1.27)) (justify right))
     )
-    (property "Value" "10K" (id 1) (at 78.74 126.9999 0)
+    (property "Value" "1K" (id 1) (at 78.74 126.9999 0)
       (effects (font (size 1.27 1.27)) (justify right))
     )
@@
     (pin "1")
   )
+  (symbol (lib_id "Connector_Generic:Conn_01x02") (at 118.745 90.805 90) (unit 1)
+    (in_bom yes) (on_board yes) (fields_autoplaced)
+    (property "Reference" "J1" (id 0) (at 124.46 89.5349 90)
+      (effects (font (size 1.27 1.27)) (justify right))
+    )
+    (property "Value" "TP1" (id 1) (at 124.46 92.0749 90)
+      (effects (font (size 1.27 1.27)) (justify right))
+    )
+    (property "Footprint" "Connector_PinSocket_2.54mm:PinSocket_1x02_P2.54mm_Vertical" (id 2) (at 118.745 90.805 0)
+      (effects (font (size 1.27 1.27)) hide)
+    )
+    (property "Datasheet" "~" (id 3) (at 118.745 90.805 0)
+      (effects (font (size 1.27 1.27)) hide)
+    )
+    (pin "1")
+    (pin "2")
+  )
   (symbol (lib_id "power:GND") (at 221.615 119.38 0) (unit 1)
     (in_bom yes) (on_board yes) (fields_autoplaced)
@@
     (pin "2")
   )
+  (symbol (lib_id "power:GND") (at 226.695 95.25 0) (unit 1)
+    (in_bom yes) (on_board yes)
+    (property "Reference" "#PWR050" (id 0) (at 226.695 101.6 0)
+      (effects (font (size 1.27 1.27)) hide)
+    )
+    (property "Value" "GND" (id 1) (at 226.695 99.06 0))
+    (property "Footprint" "" (id 2) (at 226.695 95.25 0)
+      (effects (font (size 1.27 1.27)) hide)
+    )
+    (property "Datasheet" "" (id 3) (at 226.695 95.25 0)
+      (effects (font (size 1.27 1.27)) hide)
+    )
+    (pin "1")
+  )
   (symbol (lib_id "Custom_RF:T50 ") (at 216.535 110.49 180) (unit 1)

Commit message: Update 17Mar23
Parts:
- renumbered J48 to J1, J1 to J2
Changed lines of the file:
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@@
   (symbol (lib_id "power:GND") (at 190.5 125.73 0) (unit 1)
     (in_bom yes) (on_board yes) (fields_autoplaced)
-    (property "Reference" "#PWR06" (id 0) (at 190.5 132.08 0)
+    (property "Reference" "#PWR016" (id 0) (at 190.5 132.08 0)
       (effects (font (size 1.27 1.27)) hide)
     )
@@
   (symbol (lib_id "power:GND") (at 128.27 148.59 0) (unit 1)
     (in_bom yes) (on_board yes) (fields_autoplaced)
-    (property "Reference" "#PWR08" (id 0) (at 128.27 154.94 0)
+    (property "Reference" "#PWR018" (id 0) (at 128.27 154.94 0)
       (effects (font (size 1.27 1.27)) hide)
     )
@@
   (symbol (lib_id "power:GND") (at 81.28 148.59 0) (unit 1)
     (in_bom yes) (on_board yes) (fields_autoplaced)
-    (property "Reference" "#PWR07" (id 0) (at 81.28 154.94 0)
+    (property "Reference" "#PWR017" (id 0) (at 81.28 154.94 0)
       (effects (font (size 1.27 1.27)) hide)
     )
@@
   (symbol (lib_id "power:GND") (at 121.285 95.885 0) (unit 1)
     (in_bom yes) (on_board yes) (fields_autoplaced)
-    (property "Reference" "#PWR0101" (id 0) (at 121.285 102.235 0)
+    (property "Reference" "#PWR014" (id 0) (at 121.285 102.235 0)
       (effects (font (size 1.27 1.27)) hide)
     )
@@
   (symbol (lib_id "power:GND") (at 78.74 80.01 0) (unit 1)
     (in_bom yes) (on_board yes) (fields_autoplaced)
-    (property "Reference" "#PWR03" (id 0) (at 78.74 86.36 0)
+    (property "Reference" "#PWR011" (id 0) (at 78.74 86.36 0)
       (effects (font (size 1.27 1.27)) hide)
     )
@@
   (symbol (lib_id "Connector_Generic:Conn_01x02") (at 224.155 90.17 90) (unit 1)
     (in_bom yes) (on_board yes) (fields_autoplaced)
-    (property "Reference" "J48" (id 0) (at 229.87 88.8999 90)
+    (property "Reference" "J1" (id 0) (at 229.87 88.8999 90)
       (effects (font (size 1.27 1.27)) (justify right))
     )
@@
   (symbol (lib_id "power:GND") (at 143.51 83.82 0) (unit 1)
     (in_bom yes) (on_board yes) (fields_autoplaced)
-    (property "Reference" "#PWR04" (id 0) (at 143.51 90.17 0)
+    (property "Reference" "#PWR012" (id 0) (at 143.51 90.17 0)
       (effects (font (size 1.27 1.27)) hide)
     )
@@
   (symbol (lib_id "power:GND") (at 67.31 80.01 0) (unit 1)
     (in_bom yes) (on_board yes) (fields_autoplaced)
-    (property "Reference" "#PWR02" (id 0) (at 67.31 86.36 0)
+    (property "Reference" "#PWR010" (id 0) (at 67.31 86.36 0)
       (effects (font (size 1.27 1.27)) hide)
     )
@@
   (symbol (lib_id "power:GND") (at 95.885 79.375 0) (unit 1)
     (in_bom yes) (on_board yes) (fields_autoplaced)
-    (property "Reference" "#PWR01" (id 0) (at 95.885 85.725 0)
+    (property "Reference" "#PWR09" (id 0) (at 95.885 85.725 0)
       (effects (font (size 1.27 1.27)) hide)
     )
@@
   (symbol (lib_id "Connector_Generic:Conn_01x02") (at 118.745 90.805 90) (unit 1)
     (in_bom yes) (on_board yes) (fields_autoplaced)
-    (property "Reference" "J1" (id 0) (at 124.46 89.5349 90)
+    (property "Reference" "J2" (id 0) (at 124.46 89.5349 90)
       (effects (font (size 1.27 1.27)) (justify right))
     )
@@
   (symbol (lib_id "power:GND") (at 221.615 119.38 0) (unit 1)
     (in_bom yes) (on_board yes) (fields_autoplaced)
-    (property "Reference" "#PWR05" (id 0) (at 221.615 125.73 0)
+    (property "Reference" "#PWR015" (id 0) (at 221.615 125.73 0)
       (effects (font (size 1.27 1.27)) hide)
     )
@@
   (symbol (lib_id "power:GND") (at 226.695 95.25 0) (unit 1)
     (in_bom yes) (on_board yes)
-    (property "Reference" "#PWR050" (id 0) (at 226.695 101.6 0)
-      (effects (font (size 1.27 1.27)) hide)
-    )
+    (property "Reference" "#PWR013" (id 0) (at 226.695 101.6 0)
+      (effects (font (size 1.27 1.27)) hide)
+    )

Commit message: Update 24Mar23
Parts:
- renumbered RV1 to RFG1, RV2 to RFG2
Connections:
- net at R7.1, U1.2 (InA-): now also RFG1.3; no longer RFG1.1
- net at R10.1, RFG2.2: now also RFG2.1; no longer RFG2.3
- net at R8.2, U1.6 (InB-): now also RFG2.3; no longer RFG2.1
- net at R9.1, RFG1.2: now also RFG1.1; no longer RFG1.3
Other:
- moved on the sheet: RFG1, RFG2

Commit message: Cleanup 8May23
Parts:
- R3: value 51R -> 51
- R4, R5: value 200R -> 200
- R6: value 50 -> 51
- TR1: value T50-22:4 -> T50-75 (22:4)
Changed lines of the file:
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@@
       (effects (font (size 1.27 1.27)) (justify right))
     )
-    (property "Value" "51R" (id 1) (at 89.535 78.74 0)
+    (property "Value" "51" (id 1) (at 89.535 78.74 0)
       (effects (font (size 1.27 1.27)) (justify right))
     )
@@
     (in_bom yes) (on_board yes)
     (property "Reference" "R6" (id 0) (at 156.21 110.49 90))
-    (property "Value" "50" (id 1) (at 156.21 104.14 90))
+    (property "Value" "51" (id 1) (at 156.21 104.14 90))
     (property "Footprint" "Resistor_SMD:R_1206_3216Metric" (id 2) (at 156.464 105.664 90)
       (effects (font (size 1.27 1.27)) hide)
@@
     (in_bom yes) (on_board yes) (fields_autoplaced)
     (property "Reference" "R4" (id 0) (at 76.835 92.71 90))
-    (property "Value" "200R" (id 1) (at 76.835 95.25 90))
+    (property "Value" "200" (id 1) (at 76.835 95.25 90))
     (property "Footprint" "Resistor_SMD:R_1206_3216Metric" (id 2) (at 77.089 98.044 90)
       (effects (font (size 1.27 1.27)) hide)
@@
     (in_bom yes) (on_board yes) (fields_autoplaced)
     (property "Reference" "R5" (id 0) (at 109.22 96.52 90))
-    (property "Value" "200R" (id 1) (at 109.22 99.06 90))
+    (property "Value" "200" (id 1) (at 109.22 99.06 90))
     (property "Footprint" "Resistor_SMD:R_1206_3216Metric" (id 2) (at 109.474 101.854 90)
       (effects (font (size 1.27 1.27)) hide)
@@
     (in_bom yes) (on_board yes) (fields_autoplaced)
     (property "Reference" "TR1" (id 0) (at 217.2081 100.33 0))
-    (property "Value" "T50-22:4" (id 1) (at 217.2081 102.87 0))
+    (property "Value" "T50-75 (22:4)" (id 1) (at 217.2081 102.87 0))
     (property "Footprint" "Custom_RF:T50-1Tap-Close" (id 2) (at 213.995 119.38 0)
       (effects (font (size 1.27 1.27)) hide)
