File: Phoenix612 Complete/Version 1.1/Smeter.kicad_sch (KiCad schematic)
At the start: 28 parts, among them J47 Smeter, U12 NE5532

Commit message: Update 17Mar23
Parts:
- renumbered C99 to C100, C88 to C89, C89 to C90, C90 to C91, C91 to C92, C92 to C93, C93 to C94, C94 to C95, C95 to C96, C96 to C97, C97 to C98, C98 to C99, J47 to J56, R65 to R64, R66 to R65, R67 to R66, R68 to R67, R69 to R68, R70 to R69, R71 to R70, R72 to R71, R73 to R72, R74 to R73

Commit message: Update 24Mar23
Parts:
- renumbered RV7 to SMC1
Connections:
- net GND: now also SMC1.1; no longer SMC1.3
- net at C89.2: now also SMC1.3; no longer SMC1.1
Other:
- moved on the sheet: SMC1
Changed lines of the file:
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@@
+    (stroke (width 0) (type default) (color 0 0 0 0))
+  )
+  (wire (pts (xy 39.37 87.63) (xy 39.37 91.44))
     (stroke (width 0) (type default) (color 0 0 0 0))
   )
@@
     (stroke (width 0) (type default) (color 0 0 0 0))
   )
+  (wire (pts (xy 47.625 85.09) (xy 35.56 85.09))
+    (stroke (width 0) (type default) (color 0 0 0 0))
+  )
   (wire (pts (xy 66.675 83.185) (xy 66.675 92.075))
     (stroke (width 0) (type default) (color 0 0 0 0))
@@
     (stroke (width 0) (type default) (color 0 0 0 0))
   )
+  (wire (pts (xy 35.56 85.09) (xy 35.56 83.82))
+    (stroke (width 0) (type default) (color 0 0 0 0))
+  )
   (wire (pts (xy 91.44 163.195) (xy 93.98 163.195))
     (stroke (width 0) (type default) (color 0 0 0 0))
@@
     (stroke (width 0) (type default) (color 0 0 0 0))
   )
+  (wire (pts (xy 83.185 92.075) (xy 84.455 92.075))
+    (stroke (width 0) (type default) (color 0 0 0 0))
+  )
+  (wire (pts (xy 58.42 161.925) (xy 58.42 164.465))
+    (stroke (width 0) (type default) (color 0 0 0 0))
+  )
+  (wire (pts (xy 74.295 97.155) (xy 74.295 92.075))
+    (stroke (width 0) (type default) (color 0 0 0 0))
+  )
+  (wire (pts (xy 156.845 83.185) (xy 165.735 83.185))
+    (stroke (width 0) (type default) (color 0 0 0 0))
+  )
+  (wire (pts (xy 46.99 164.465) (xy 58.42 164.465))
+    (stroke (width 0) (type default) (color 0 0 0 0))
+  )
+  (wire (pts (xy 83.82 163.195) (xy 79.375 163.195))
+    (stroke (width 0) (type default) (color 0 0 0 0))
+  )
+  (wire (pts (xy 76.835 97.155) (xy 74.295 97.155))
+    (stroke (width 0) (type default) (color 0 0 0 0))
+  )
+  (wire (pts (xy 109.22 163.195) (xy 99.06 163.195))
+    (stroke (width 0) (type default) (color 0 0 0 0))
+  )
+  (wire (pts (xy 36.195 77.47) (xy 39.37 77.47))
+    (stroke (width 0) (type default) (color 0 0 0 0))
+  )
+  (wire (pts (xy 75.565 92.075) (xy 74.295 92.075))
+    (stroke (width 0) (type default) (color 0 0 0 0))
+  )
+  (wire (pts (xy 46.99 165.735) (xy 46.99 164.465))
+    (stroke (width 0) (type default) (color 0 0 0 0))
+  )
+  (wire (pts (xy 99.06 172.085) (xy 99.06 170.18))
+    (stroke (width 0) (type default) (color 0 0 0 0))
+  )
+  (wire (pts (xy 139.7 83.185) (xy 144.145 83.185))
+    (stroke (width 0) (type default) (color 0 0 0 0))
+  )
+  (wire (pts (xy 109.22 163.195) (xy 109.22 164.465))
+    (stroke (width 0) (type default) (color 0 0 0 0))
+  )
+  (wire (pts (xy 69.215 83.185) (xy 66.675 83.185))
+    (stroke (width 0) (type default) (color 0 0 0 0))
+  )
+  (wire (pts (xy 139.7 95.885) (xy 139.7 92.71))
+    (stroke (width 0) (type default) (color 0 0 0 0))
+  )
+  (wire (pts (xy 81.915 97.155) (xy 84.455 97.155))
+    (stroke (width 0) (type default) (color 0 0 0 0))
+  )
+  (wire (pts (xy 74.295 92.075) (xy 66.675 92.075))
+    (stroke (width 0) (type default) (color 0 0 0 0))
+  )
+  (wire (pts (xy 104.775 85.725) (xy 104.775 93.345))
+    (stroke (width 0) (type default) (color 0 0 0 0))
+  )
+  (wire (pts (xy 79.375 163.195) (xy 79.375 164.465))
+    (stroke (width 0) (type default) (color 0 0 0 0))
+  )
+  (wire (pts (xy 100.965 80.645) (xy 106.68 80.645))
+    (stroke (width 0) (type default) (color 0 0 0 0))
+  )
+  (wire (pts (xy 165.735 85.725) (xy 165.735 89.535))
+    (stroke (width 0) (type default) (color 0 0 0 0))
+  )
+  (wire (pts (xy 46.99 164.465) (xy 39.37 164.465))
+    (stroke (width 0) (type default) (color 0 0 0 0))
+  )
+  (wire (pts (xy 156.845 83.185) (xy 156.845 84.455))
+    (stroke (width 0) (type default) (color 0 0 0 0))
+  )
+  (wire (pts (xy 122.555 98.425) (xy 122.555 93.345))
+    (stroke (width 0) (type default) (color 0 0 0 0))
+  )
+  (wire (pts (xy 113.665 93.345) (xy 112.395 93.345))
+    (stroke (width 0) (type default) (color 0 0 0 0))
+  )
+  (wire (pts (xy 156.845 92.075) (xy 156.845 95.25))
+    (stroke (width 0) (type default) (color 0 0 0 0))
+  )
+  (wire (pts (xy 151.765 83.185) (xy 156.845 83.185))
+    (stroke (width 0) (type default) (color 0 0 0 0))
+  )
+  (wire (pts (xy 139.7 83.185) (xy 139.7 85.09))
+    (stroke (width 0) (type default) (color 0 0 0 0))
+  )
+  (wire (pts (xy 58.42 164.465) (xy 58.42 165.735))
+    (stroke (width 0) (type default) (color 0 0 0 0))
+  )
+  (wire (pts (xy 39.37 164.465) (xy 39.37 163.195))
+    (stroke (width 0) (type default) (color 0 0 0 0))
+  )
+  (wire (pts (xy 59.055 78.105) (xy 69.215 78.105))
+    (stroke (width 0) (type default) (color 0 0 0 0))
+  )
+  (wire (pts (xy 109.22 172.085) (xy 109.22 169.545))
+    (stroke (width 0) (type default) (color 0 0 0 0))
+  )
+  (wire (pts (xy 112.395 93.345) (xy 104.775 93.345))
+    (stroke (width 0) (type default) (color 0 0 0 0))
+  )
   (wire (pts (xy 39.37 77.47) (xy 39.37 80.01))
     (stroke (width 0) (type default) (color 0 0 0 0))
   )
-  (wire (pts (xy 83.185 92.075) (xy 84.455 92.075))
-    (stroke (width 0) (type default) (color 0 0 0 0))
-  )
-  (wire (pts (xy 58.42 161.925) (xy 58.42 164.465))
-    (stroke (width 0) (type default) (color 0 0 0 0))
-  )
-  (wire (pts (xy 74.295 97.155) (xy 74.295 92.075))
-    (stroke (width 0) (type default) (color 0 0 0 0))
-  )
-  (wire (pts (xy 156.845 83.185) (xy 165.735 83.185))
-    (stroke (width 0) (type default) (color 0 0 0 0))
-  )
-  (wire (pts (xy 46.99 164.465) (xy 58.42 164.465))
-    (stroke (width 0) (type default) (color 0 0 0 0))
-  )
-  (wire (pts (xy 83.82 163.195) (xy 79.375 163.195))
-    (stroke (width 0) (type default) (color 0 0 0 0))
-  )
-  (wire (pts (xy 76.835 97.155) (xy 74.295 97.155))
-    (stroke (width 0) (type default) (color 0 0 0 0))
-  )
-  (wire (pts (xy 109.22 163.195) (xy 99.06 163.195))
-    (stroke (width 0) (type default) (color 0 0 0 0))
-  )
-  (wire (pts (xy 36.195 77.47) (xy 39.37 77.47))
-    (stroke (width 0) (type default) (color 0 0 0 0))
-  )
-  (wire (pts (xy 75.565 92.075) (xy 74.295 92.075))
-    (stroke (width 0) (type default) (color 0 0 0 0))
-  )
-  (wire (pts (xy 46.99 165.735) (xy 46.99 164.465))
-    (stroke (width 0) (type default) (color 0 0 0 0))
-  )
-  (wire (pts (xy 99.06 172.085) (xy 99.06 170.18))
-    (stroke (width 0) (type default) (color 0 0 0 0))
-  )
-  (wire (pts (xy 139.7 83.185) (xy 144.145 83.185))
-    (stroke (width 0) (type default) (color 0 0 0 0))
-  )
-  (wire (pts (xy 109.22 163.195) (xy 109.22 164.465))
-    (stroke (width 0) (type default) (color 0 0 0 0))
-  )
-  (wire (pts (xy 69.215 83.185) (xy 66.675 83.185))
-    (stroke (width 0) (type default) (color 0 0 0 0))
-  )
-  (wire (pts (xy 139.7 95.885) (xy 139.7 92.71))
-    (stroke (width 0) (type default) (color 0 0 0 0))
-  )
-  (wire (pts (xy 81.915 97.155) (xy 84.455 97.155))
-    (stroke (width 0) (type default) (color 0 0 0 0))
-  )
-  (wire (pts (xy 74.295 92.075) (xy 66.675 92.075))
-    (stroke (width 0) (type default) (color 0 0 0 0))
-  )
-  (wire (pts (xy 104.775 85.725) (xy 104.775 93.345))
-    (stroke (width 0) (type default) (color 0 0 0 0))
-  )
-  (wire (pts (xy 79.375 163.195) (xy 79.375 164.465))
-    (stroke (width 0) (type default) (color 0 0 0 0))
-  )
-  (wire (pts (xy 100.965 80.645) (xy 106.68 80.645))
-    (stroke (width 0) (type default) (color 0 0 0 0))
-  )
-  (wire (pts (xy 165.735 85.725) (xy 165.735 89.535))
-    (stroke (width 0) (type default) (color 0 0 0 0))
-  )
-  (wire (pts (xy 46.99 164.465) (xy 39.37 164.465))
-    (stroke (width 0) (type default) (color 0 0 0 0))
-  )
-  (wire (pts (xy 156.845 83.185) (xy 156.845 84.455))
-    (stroke (width 0) (type default) (color 0 0 0 0))
-  )
-  (wire (pts (xy 122.555 98.425) (xy 122.555 93.345))
-    (stroke (width 0) (type default) (color 0 0 0 0))
-  )
-  (wire (pts (xy 113.665 93.345) (xy 112.395 93.345))
-    (stroke (width 0) (type default) (color 0 0 0 0))
-  )
-  (wire (pts (xy 156.845 92.075) (xy 156.845 95.25))
-    (stroke (width 0) (type default) (color 0 0 0 0))
-  )
-  (wire (pts (xy 151.765 83.185) (xy 156.845 83.185))
-    (stroke (width 0) (type default) (color 0 0 0 0))
-  )
-  (wire (pts (xy 139.7 83.185) (xy 139.7 85.09))
-    (stroke (width 0) (type default) (color 0 0 0 0))
-  )
-  (wire (pts (xy 58.42 164.465) (xy 58.42 165.735))
-    (stroke (width 0) (type default) (color 0 0 0 0))
-  )
-  (wire (pts (xy 39.37 164.465) (xy 39.37 163.195))
-    (stroke (width 0) (type default) (color 0 0 0 0))
-  )
-  (wire (pts (xy 59.055 78.105) (xy 69.215 78.105))
-    (stroke (width 0) (type default) (color 0 0 0 0))
-  )
-  (wire (pts (xy 39.37 87.63) (xy 39.37 91.44))
-    (stroke (width 0) (type default) (color 0 0 0 0))
-  )
-  (wire (pts (xy 47.625 83.82) (xy 43.18 83.82))
-    (stroke (width 0) (type default) (color 0 0 0 0))
-  )
-  (wire (pts (xy 109.22 172.085) (xy 109.22 169.545))
-    (stroke (width 0) (type default) (color 0 0 0 0))
-  )
-  (wire (pts (xy 112.395 93.345) (xy 104.775 93.345))
-    (stroke (width 0) (type default) (color 0 0 0 0))
-  )
   (wire (pts (xy 88.265 80.645) (xy 93.345 80.645))
     (stroke (width 0) (type default) (color 0 0 0 0))
@@
     (stroke (width 0) (type default) (color 0 0 0 0))
   )
-  (wire (pts (xy 47.625 78.105) (xy 47.625 83.82))
+  (wire (pts (xy 47.625 78.105) (xy 47.625 85.09))
     (stroke (width 0) (type default) (color 0 0 0 0))
   )
@@
     (pin "2")
   )
-  (symbol (lib_id "Device:R_Potentiometer_Trim") (at 39.37 83.82 0) (unit 1)
-    (in_bom yes) (on_board yes) (fields_autoplaced)
-    (property "Reference" "RV7" (id 0) (at 36.83 82.5499 0)
+  (symbol (lib_id "Device:R_Potentiometer_Trim") (at 39.37 83.82 180) (unit 1)
+    (in_bom yes) (on_board yes) (fields_autoplaced)
+    (property "Reference" "SMC1" (id 0) (at 41.91 82.5499 0)
       (effects (font (size 1.27 1.27)) (justify right))
     )
-    (property "Value" "10K" (id 1) (at 36.83 85.0899 0)
+    (property "Value" "10K" (id 1) (at 41.91 85.0899 0)
       (effects (font (size 1.27 1.27)) (justify right))
     )

Commit message: Cleanup 8May23
Parts:
- D12: value 1N4148 -> 1N914
Other:
- note added: "Need to change U12B to a peak detector with negative voltage supply"
- note added: "R65 is not needed"
Changed lines of the file:
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@@
     (stroke (width 0) (type default) (color 0 0 0 0))
+  )
+  (text "R65 is not needed" (at 134.62 106.68 0)
+    (effects (font (size 1.27 1.27)) (justify left bottom))
+  )
+  (text "Need to change U12B to a peak detector with negative voltage supply"
+    (at 110.49 67.31 0)
+    (effects (font (size 1.27 1.27)) (justify left bottom))
   )
   (global_label "SM_BIAS" (shape bidirectional) (at 79.375 163.195 90) (fields_autoplaced)
@@
     (in_bom yes) (on_board yes)
     (property "Reference" "D12" (id 0) (at 147.955 86.995 0))
-    (property "Value" "1N4148" (id 1) (at 146.685 80.645 0))
+    (property "Value" "1N914" (id 1) (at 146.685 80.645 0))
     (property "Footprint" "Diode_THT:D_DO-35_SOD27_P7.62mm_Horizontal" (id 2) (at 147.955 78.74 0)
       (effects (font (size 1.27 1.27)) hide)
